File: hardware/kicad/emg-filter/notch.sch (KiCad schematic (older format))
At the start: 88 parts, among them U11 LM4565, U12 LM4565, U13 LM4565, U14 LM4565, U15 LM4565, U16 LM4565, U17 LM4565, U18 LM4565

Commit message: pcb
Parts:
- U11, U12, U13, U14, U15, U16, U17, U18: footprint (none) -> emg-filter:LM4565
Changed lines of the file:
@@
 F 0 "U11" H 3625 1450 50  0000 C CNN
 F 1 "LM4565" H 3975 1450 50  0000 C CNN
-F 2 "" H 4825 1150 50  0001 C CNN
+F 2 "emg-filter:LM4565" H 4825 1150 50  0001 C CNN
 F 3 "" H 4825 1150 50  0001 C CNN
 	1    3825 1150
@@
 F 0 "U12" H 3650 2875 50  0000 C CNN
 F 1 "LM4565" H 4000 2875 50  0000 C CNN
-F 2 "" H 4850 2575 50  0001 C CNN
+F 2 "emg-filter:LM4565" H 4850 2575 50  0001 C CNN
 F 3 "" H 4850 2575 50  0001 C CNN
 	1    3850 2575
@@
 F 0 "U13" H 3650 4250 50  0000 C CNN
 F 1 "LM4565" H 4000 4250 50  0000 C CNN
-F 2 "" H 4850 3950 50  0001 C CNN
+F 2 "emg-filter:LM4565" H 4850 3950 50  0001 C CNN
 F 3 "" H 4850 3950 50  0001 C CNN
 	1    3850 3950
@@
 F 0 "U14" H 3675 5675 50  0000 C CNN
 F 1 "LM4565" H 4025 5675 50  0000 C CNN
-F 2 "" H 4875 5375 50  0001 C CNN
+F 2 "emg-filter:LM4565" H 4875 5375 50  0001 C CNN
 F 3 "" H 4875 5375 50  0001 C CNN
 	1    3875 5375
@@
 F 0 "U15" H 8525 1450 50  0000 C CNN
 F 1 "LM4565" H 8875 1450 50  0000 C CNN
-F 2 "" H 9725 1150 50  0001 C CNN
+F 2 "emg-filter:LM4565" H 9725 1150 50  0001 C CNN
 F 3 "" H 9725 1150 50  0001 C CNN
 	1    8725 1150
@@
 F 0 "U16" H 8550 2875 50  0000 C CNN
 F 1 "LM4565" H 8900 2875 50  0000 C CNN
-F 2 "" H 9750 2575 50  0001 C CNN
+F 2 "emg-filter:LM4565" H 9750 2575 50  0001 C CNN
 F 3 "" H 9750 2575 50  0001 C CNN
 	1    8750 2575
@@
 F 0 "U17" H 8550 4250 50  0000 C CNN
 F 1 "LM4565" H 8900 4250 50  0000 C CNN
-F 2 "" H 9750 3950 50  0001 C CNN
+F 2 "emg-filter:LM4565" H 9750 3950 50  0001 C CNN
 F 3 "" H 9750 3950 50  0001 C CNN
 	1    8750 3950
@@
 F 0 "U18" H 8575 5675 50  0000 C CNN
 F 1 "LM4565" H 8925 5675 50  0000 C CNN
-F 2 "" H 9775 5375 50  0001 C CNN
+F 2 "emg-filter:LM4565" H 9775 5375 50  0001 C CNN
 F 3 "" H 9775 5375 50  0001 C CNN
 	1    8775 5375
