File: hardware/kicad/emg-filter/rectifier.sch (KiCad schematic (older format))
At the start: 0 parts

Commit message: Initial branch commit
Parts:
- added D? (x2): 1N4148, symbol Device:D
- added R1, R? (x3): 10k, symbol Device:R
- added R?: 5k, symbol Device:R
- added U1: LM4565, symbol emg-filter:LM4565
Changed lines of the file:
@@
 $Descr A4 11693 8268
 encoding utf-8
-Sheet 1 9
+Sheet 6 9
 Title ""
 Date ""
@@
 Comment4 ""
 $EndDescr
+$Comp
+L emg-filter:LM4565 U1
+U 1 1 61C39F82
+P 7050 2900
+F 0 "U1" H 7050 3431 50  0000 C CNN
+F 1 "LM4565" H 7050 3340 50  0000 C CNN
+F 2 "" H 8050 2900 50  0001 C CNN
+F 3 "" H 8050 2900 50  0001 C CNN
+	1    7050 2900
+	1    0    0    -1
+$EndComp
+$Comp
+L Device:R R1
+U 1 1 61C3AD78
+P 6000 2700
+F 0 "R1" V 6207 2700 50  0000 C CNN
+F 1 "10k" V 6116 2700 50  0000 C CNN
+F 2 "" V 5930 2700 50  0001 C CNN
+F 3 "~" H 6000 2700 50  0001 C CNN
+	1    6000 2700
+	0    -1   -1   0
+$EndComp
+$Comp
+L Device:R R?
+U 1 1 61C4805B
+P 6000 3150
+F 0 "R?" V 6207 3150 50  0000 C CNN
+F 1 "10k" V 6116 3150 50  0000 C CNN
+F 2 "" V 5930 3150 50  0001 C CNN
+F 3 "~" H 6000 3150 50  0001 C CNN
+	1    6000 3150
+	0    -1   -1   0
+$EndComp
+$Comp
+L Device:R R?
+U 1 1 61C4A9A1
+P 6000 2250
+F 0 "R?" V 5793 2250 50  0000 C CNN
+F 1 "5k" V 5884 2250 50  0000 C CNN
+F 2 "" V 5930 2250 50  0001 C CNN
+F 3 "~" H 6000 2250 50  0001 C CNN
+	1    6000 2250
+	0    1    1    0
+$EndComp
+$Comp
+L Device:R R?
+U 1 1 61C4B3BB
+P 6000 3500
+F 0 "R?" V 6207 3500 50  0000 C CNN
+F 1 "10k" V 6116 3500 50  0000 C CNN
+F 2 "" V 5930 3500 50  0001 C CNN
+F 3 "~" H 6000 3500 50  0001 C CNN
+	1    6000 3500
+	0    -1   -1   0
+$EndComp
+$Comp
+L Device:R R?
+U 1 1 61C4B97C
+P 6000 3800
+F 0 "R?" V 6207 3800 50  0000 C CNN
+F 1 "10k" V 6116 3800 50  0000 C CNN
+F 2 "" V 5930 3800 50  0001 C CNN
+F 3 "~" H 6000 3800 50  0001 C CNN
+	1    6000 3800
+	0    -1   -1   0
+$EndComp
+$Comp
+L Device:D D?
+U 1 1 61C4C7DA
+P 5450 2550
+F 0 "D?" H 5450 2767 50  0000 C CNN
+F 1 "1N4148" H 5450 2676 50  0000 C CNN
+F 2 "" H 5450 2550 50  0001 C CNN
+F 3 "~" H 5450 2550 50  0001 C CNN
+	1    5450 2550
+	1    0    0    -1
+$EndComp
+$Comp
+L Device:D D?
+U 1 1 61C4C9DB
+P 5400 2850
+F 0 "D?" H 5400 3067 50  0000 C CNN
+F 1 "1N4148" H 5400 2976 50  0000 C CNN
+F 2 "" H 5400 2850 50  0001 C CNN
+F 3 "~" H 5400 2850 50  0001 C CNN
+	1    5400 2850
+	1    0    0    -1
+$EndComp
 $EndSCHEMATC
