File: hardware/kicad/emg-filter/rectifier.sch (KiCad schematic (older format))
At the start: 128 parts, among them U1 LM4565, U10 LM4565, U11 LM4565, U12 LM4565, U13 LM4565, U14 LM4565, U15 LM4565, U16 LM4565, U2 LM4565, U3 LM4565, U4 LM4565, U5 LM4565, U6 LM4565, U7 LM4565, U8 LM4565, U9 LM4565

Commit message: annotation
Parts:
- renumbered D5 to D10, D6 to D11, D7 to D12, D8 to D13, D9 to D14, D2 to D15, D10 to D16, D11 to D17, D12 to D18, D13 to D19, D14 to D20, D15 to D21, D16 to D22, D17 to D23, D18 to D24, D19 to D25, D20 to D26, D21 to D27, D22 to D28, D23 to D29, D24 to D30, D25 to D31, D26 to D32, D27 to D33, D28 to D34, D29 to D35, D30 to D36, D31 to D37, D32 to D38, D1 to D7, D3 to D8, D4 to D9, R1 to R155, R6 to R156, R7 to R157, R8 to R158, R9 to R159, R10 to R160, R11 to R161, R12 to R162, R2 to R163, R13 to R164, R14 to R165, R15 to R166, R16 to R167, R17 to R168, R18 to R169, R19 to R170, R3 to R171, R4 to R172, R20 to R173, R21 to R174, R22 to R175, R23 to R176, R24 to R177, R25 to R178, R26 to R179, R27 to R180, R28 to R181, R29 to R182, R30 to R183, R31 to R184, R32 to R185, R33 to R186, R5 to R187, R34 to R188, R35 to R189, R36 to R190, R37 to R191, R38 to R192, R39 to R193, R40 to R194, R41 to R195, R42 to R196, R43 to R197, R44 to R198, R45 to R199, R46 to R200, R47 to R201, R48 to R202, R49 to R203, R50 to R204, R51 to R205, R52 to R206, R53 to R207, R54 to R208, R55 to R209, R56 to R210, R57 to R211, R58 to R212, R59 to R213, R60 to R214, R61 to R215, R62 to R216, R63 to R217, R64 to R218, R65 to R219, R66 to R220, R67 to R221, R68 to R222, R69 to R223, R70 to R224, R71 to R225, R72 to R226, R73 to R227, R74 to R228, R75 to R229, R76 to R230, R77 to R231, R78 to R232, R79 to R233, R80 to R234, U1 to U36, U2 to U37, U3 to U38, U4 to U39, U5 to U40, U6 to U41, U7 to U42, U8 to U43, U9 to U44, U10 to U45, U11 to U46, U12 to U47, U13 to U48, U14 to U49, U15 to U50, U16 to U51

Commit message: linked stages by renaming labels
Connections:
- net INPUT_10_RECTIFIER renamed NOTCH_RECT_10
- net INPUT_11_RECTIFIER renamed NOTCH_RECT_11
- net INPUT_12_RECTIFIER renamed NOTCH_RECT_12
- net INPUT_13_RECTIFIER renamed NOTCH_RECT_13
- net INPUT_14_RECTIFIER renamed NOTCH_RECT_14
- net INPUT_15_RECTIFIER renamed NOTCH_RECT_15
- net INPUT_16_RECTIFIER renamed NOTCH_RECT_16
- net INPUT_1_RECTIFIER renamed NOTCH_RECT_1
- net INPUT_2_RECTIFIER renamed NOTCH_RECT_2
- net INPUT_3_RECTIFIER renamed NOTCH_RECT_3
- net INPUT_4_RECTIFIER renamed NOTCH_RECT_4
- net INPUT_5_RECTIFIER renamed NOTCH_RECT_5
- net INPUT_6_RECTIFIER renamed NOTCH_RECT_6
- net INPUT_7_RECTIFIER renamed NOTCH_RECT_7
- net INPUT_8_RECTIFIER renamed NOTCH_RECT_8
- net INPUT_9_RECTIFIER renamed NOTCH_RECT_9
Changed lines of the file:
@@
 $Descr A2 23386 16535
 encoding utf-8
-Sheet 1 10
+Sheet 7 10
 Title ""
 Date ""
@@
 Wire Wire Line
 	7250 1150 7100 1150
-Text GLabel 1700 1550 0    50   Input ~ 0
-INPUT_1_RECTIFIER
 Wire Wire Line
 	1800 1550 1700 1550
 Connection ~ 1800 1550
-Text GLabel 5400 1350 2    50   Input ~ 0
-OUTPUT_1_RECTIFIER
 Wire Wire Line
 	5400 1350 5300 1350
@@
 Wire Wire Line
 	7300 3000 7150 3000
-Text GLabel 1750 3400 0    50   Input ~ 0
-INPUT_2_RECTIFIER
 Wire Wire Line
 	1850 3400 1750 3400
 Connection ~ 1850 3400
-Text GLabel 5450 3200 2    50   Input ~ 0
-OUTPUT_2_RECTIFIER
 Wire Wire Line
 	5450 3200 5350 3200
@@
 Wire Wire Line
 	7350 4900 7200 4900
-Text GLabel 1800 5300 0    50   Input ~ 0
-INPUT_3_RECTIFIER
 Wire Wire Line
 	1900 5300 1800 5300
 Connection ~ 1900 5300
-Text GLabel 5500 5100 2    50   Input ~ 0
-OUTPUT_3_RECTIFIER
 Wire Wire Line
 	5500 5100 5400 5100
@@
 Wire Wire Line
 	7450 6850 7300 6850
-Text GLabel 1900 7250 0    50   Input ~ 0
-INPUT_4_RECTIFIER
 Wire Wire Line
 	2000 7250 1900 7250
 Connection ~ 2000 7250
-Text GLabel 5600 7050 2    50   Input ~ 0
-OUTPUT_4_RECTIFIER
 Wire Wire Line
 	5600 7050 5500 7050
@@
 Wire Wire Line
 	7450 8850 7300 8850
-Text GLabel 1900 9250 0    50   Input ~ 0
-INPUT_5_RECTIFIER
 Wire Wire Line
 	2000 9250 1900 9250
 Connection ~ 2000 9250
-Text GLabel 5600 9050 2    50   Input ~ 0
-OUTPUT_5_RECTIFIER
 Wire Wire Line
 	5600 9050 5500 9050
@@
 Wire Wire Line
 	7450 10950 7300 10950
-Text GLabel 1900 11350 0    50   Input ~ 0
-INPUT_6_RECTIFIER
 Wire Wire Line
 	2000 11350 1900 11350
 Connection ~ 2000 11350
-Text GLabel 5600 11150 2    50   Input ~ 0
-OUTPUT_6_RECTIFIER
 Wire Wire Line
 	5600 11150 5500 11150
@@
 Wire Wire Line
 	7450 12650 7300 12650
-Text GLabel 1900 13050 0    50   Input ~ 0
-INPUT_7_RECTIFIER
 Wire Wire Line
 	2000 13050 1900 13050
 Connection ~ 2000 13050
-Text GLabel 5600 12850 2    50   Input ~ 0
-OUTPUT_7_RECTIFIER
 Wire Wire Line
 	5600 12850 5500 12850
@@
 Wire Wire Line
 	7450 14500 7300 14500
-Text GLabel 1900 14900 0    50   Input ~ 0
-INPUT_8_RECTIFIER
 Wire Wire Line
 	2000 14900 1900 14900
 Connection ~ 2000 14900
-Text GLabel 5600 14700 2    50   Input ~ 0
-OUTPUT_8_RECTIFIER
 Wire Wire Line
 	5600 14700 5500 14700
@@
 Wire Wire Line
 	16250 1150 16100 1150
-Text GLabel 10700 1550 0    50   Input ~ 0
-INPUT_9_RECTIFIER
 Wire Wire Line
 	10800 1550 10700 1550
 Connection ~ 10800 1550
-Text GLabel 14400 1350 2    50   Input ~ 0
-OUTPUT_9_RECTIFIER
 Wire Wire Line
 	14400 1350 14300 1350
@@
 Wire Wire Line
 	16150 2800 16000 2800
-Text GLabel 10600 3200 0    50   Input ~ 0
-INPUT_10_RECTIFIER
 Wire Wire Line
 	10700 3200 10600 3200
 Connection ~ 10700 3200
-Text GLabel 14300 3000 2    50   Input ~ 0
-OUTPUT_10_RECTIFIER
 Wire Wire Line
 	14300 3000 14200 3000
@@
 Wire Wire Line
 	16150 4750 16000 4750
-Text GLabel 10600 5150 0    50   Input ~ 0
-INPUT_11_RECTIFIER
 Wire Wire Line
 	10700 5150 10600 5150
 Connection ~ 10700 5150
-Text GLabel 14300 4950 2    50   Input ~ 0
-OUTPUT_11_RECTIFIER
 Wire Wire Line
 	14300 4950 14200 4950
@@
 Wire Wire Line
 	16200 6700 16050 6700
-Text GLabel 10650 7100 0    50   Input ~ 0
-INPUT_12_RECTIFIER
 Wire Wire Line
 	10750 7100 10650 7100
 Connection ~ 10750 7100
-Text GLabel 14350 6900 2    50   Input ~ 0
-OUTPUT_12_RECTIFIER
 Wire Wire Line
 	14350 6900 14250 6900
@@
 Wire Wire Line
 	16100 8550 15950 8550
-Text GLabel 10550 8950 0    50   Input ~ 0
-INPUT_13_RECTIFIER
 Wire Wire Line
 	10650 8950 10550 8950
 Connection ~ 10650 8950
-Text GLabel 14250 8750 2    50   Input ~ 0
-OUTPUT_13_RECTIFIER
 Wire Wire Line
 	14250 8750 14150 8750
@@
 Wire Wire Line
 	16300 10700 16150 10700
-Text GLabel 10750 11100 0    50   Input ~ 0
-INPUT_14_RECTIFIER
 Wire Wire Line
 	10850 11100 10750 11100
 Connection ~ 10850 11100
-Text GLabel 14450 10900 2    50   Input ~ 0
-OUTPUT_14_RECTIFIER
 Wire Wire Line
 	14450 10900 14350 10900
@@
 Wire Wire Line
 	16300 12400 16150 12400
-Text GLabel 10750 12800 0    50   Input ~ 0
-INPUT_15_RECTIFIER
 Wire Wire Line
 	10850 12800 10750 12800
 Connection ~ 10850 12800
-Text GLabel 14450 12600 2    50   Input ~ 0
-OUTPUT_15_RECTIFIER
 Wire Wire Line
 	14450 12600 14350 12600
@@
 Wire Wire Line
 	16250 14250 16100 14250
-Text GLabel 10700 14650 0    50   Input ~ 0
-INPUT_16_RECTIFIER
 Wire Wire Line
 	10800 14650 10700 14650
 Connection ~ 10800 14650
-Text GLabel 14400 14450 2    50   Input ~ 0
-OUTPUT_16_RECTIFIER
 Wire Wire Line
 	14400 14450 14300 14450
@@
 	-1   0    0    1
 $EndComp
+Text GLabel 1750 3400 0    50   Input ~ 0
+NOTCH_RECT_2
+Text GLabel 1800 5300 0    50   Input ~ 0
+NOTCH_RECT_3
+Text GLabel 1700 1550 0    50   Input ~ 0
+NOTCH_RECT_1
+Text GLabel 10700 14650 0    50   Input ~ 0
+NOTCH_RECT_16
+Text GLabel 10750 12800 0    50   Input ~ 0
+NOTCH_RECT_15
+Text GLabel 10750 11100 0    50   Input ~ 0
+NOTCH_RECT_14
+Text GLabel 10550 8950 0    50   Input ~ 0
+NOTCH_RECT_13
+Text GLabel 10650 7100 0    50   Input ~ 0
+NOTCH_RECT_12
+Text GLabel 10600 5150 0    50   Input ~ 0
+NOTCH_RECT_11
+Text GLabel 10600 3200 0    50   Input ~ 0
+NOTCH_RECT_10
+Text GLabel 10700 1550 0    50   Input ~ 0
+NOTCH_RECT_9
+Text GLabel 1900 14900 0    50   Input ~ 0
+NOTCH_RECT_8
+Text GLabel 1900 13050 0    50   Input ~ 0
+NOTCH_RECT_7
+Text GLabel 1900 11350 0    50   Input ~ 0
+NOTCH_RECT_6
+Text GLabel 1900 9250 0    50   Input ~ 0
+NOTCH_RECT_5
+Text GLabel 1900 7250 0    50   Input ~ 0
+NOTCH_RECT_4
+Text GLabel 5400 1350 2    50   Input ~ 0
+RECT_AMP_1
+Text GLabel 5450 3200 2    50   Input ~ 0
+RECT_AMP_2
+Text GLabel 5500 5100 2    50   Input ~ 0
+RECT_AMP_3
+Text GLabel 5600 7050 2    50   Input ~ 0
+RECT_AMP_4
+Text GLabel 5600 9050 2    50   Input ~ 0
+RECT_AMP_5
+Text GLabel 5600 11150 2    50   Input ~ 0
+RECT_AMP_6
+Text GLabel 5600 12850 2    50   Input ~ 0
+RECT_AMP_7
+Text GLabel 5600 14700 2    50   Input ~ 0
+RECT_AMP_8
+Text GLabel 14400 1350 2    50   Input ~ 0
+RECT_AMP_9
+Text GLabel 14300 3000 2    50   Input ~ 0
+RECT_AMP_10
+Text GLabel 14300 4950 2    50   Input ~ 0
+RECT_AMP_11
+Text GLabel 14350 6900 2    50   Input ~ 0
+RECT_AMP_12
+Text GLabel 14250 8750 2    50   Input ~ 0
+RECT_AMP_13
+Text GLabel 14450 10900 2    50   Input ~ 0
+RECT_AMP_14
+Text GLabel 14450 12600 2    50   Input ~ 0
+RECT_AMP_15
+Text GLabel 14400 14450 2    50   Input ~ 0
+RECT_AMP_16
 $EndSCHEMATC
