File: hardware/kicad/emg-filter/instrumentation.sch (KiCad schematic (older format))
At the start: 5 parts, among them U1 INA2332

Commit message: instrumentation x16
Parts:
- added R10, R11, R12, R19, R20, R21, R22, R23, R24, R29, R30, R31, R32, R9: 10k, symbol Device:R
- added R13, R14, R15, R16, R17, R18, R25, R26, R27, R28, R3, R4, R5, R6: 191k, symbol Device:R
- added U2, U3, U4, U5, U6, U7, U8: INA2332, symbol emg-filter:INA2332
- renumbered R3 to R7, R4 to R8
Connections:
- net labels added: +VINA_11_INA, +VINA_13_INA, +VINA_15_INA, +VINA_3_INA, +VINA_5_INA, +VINA_7_INA, +VINA_9_INA, +VINB_10_INA, +VINB_12_INA, +VINB_14_INA, +VINB_16_INA, +VINB_4_INA, +VINB_6_INA, +VINB_8_INA, -VINA_11_INA, -VINA_13_INA, -VINA_15_INA, -VINA_3_INA, -VINA_5_INA, -VINA_7_INA, -VINA_9_INA, -VINB_10_INA, -VINB_12_INA, -VINB_14_INA, -VINB_16_INA, -VINB_4_INA, -VINB_6_INA, -VINB_8_INA, REFA_11_INA, REFA_13_INA, REFA_15_INA, REFA_3_INA, REFA_5_INA, REFA_7_INA, REFA_9_INA, REFB_10_INA, REFB_12_INA, REFB_14_INA, REFB_16_INA, REFB_4_INA, REFB_6_INA, REFB_8_INA, VOUTA_11_INA, VOUTA_13_INA, VOUTA_15_INA, VOUTA_3_INA, VOUTA_5_INA, VOUTA_7_INA, VOUTA_9_INA, VOUTB_10_INA, VOUTB_12_INA, VOUTB_14_INA, VOUTB_16_INA, VOUTB_4_INA, VOUTB_6_INA, VOUTB_8_INA
- wire segments 36 -> 288
Other:
- moved on the sheet: R1, R2, R7, R8

Commit message: fixed incorrect SHTDWN pin connection
Connections:
- net labels added: SHTDWN_INA
- wire segments 288 -> 280
Changed lines of the file:
@@
 $EndComp
-Wire Wire Line
-	2100 6400 2100 6450
-Wire Wire Line
-	2100 6450 2700 6450
-Wire Wire Line
-	2700 6450 2700 6200
 Wire Wire Line
 	2700 6200 2650 6200
-Wire Wire Line
-	2100 6450 2100 6500
-Connection ~ 2100 6450
 Wire Wire Line
 	2650 6100 2800 6100
@@
 Wire Wire Line
 	2650 2200 2800 2200
-Connection ~ 2100 2550
-Wire Wire Line
-	2100 2550 2100 2600
 Wire Wire Line
 	2700 2300 2650 2300
-Wire Wire Line
-	2700 2550 2700 2300
-Wire Wire Line
-	2100 2550 2700 2550
-Wire Wire Line
-	2100 2500 2100 2550
 $Comp
 L Device:R R8
@@
 Wire Wire Line
 	2650 4150 2800 4150
-Connection ~ 2100 4500
-Wire Wire Line
-	2100 4500 2100 4550
 Wire Wire Line
 	2700 4250 2650 4250
-Wire Wire Line
-	2700 4500 2700 4250
-Wire Wire Line
-	2100 4500 2700 4500
-Wire Wire Line
-	2100 4450 2100 4500
 $Comp
 L Device:R R10
@@
 $EndComp
 Wire Wire Line
-	5400 6400 5400 6450
-Wire Wire Line
-	5400 6450 6000 6450
-Wire Wire Line
-	6000 6450 6000 6200
-Wire Wire Line
 	6000 6200 5950 6200
-Wire Wire Line
-	5400 6450 5400 6500
-Connection ~ 5400 6450
 Wire Wire Line
 	5950 6100 6100 6100
@@
 Wire Wire Line
 	5950 2200 6100 2200
-Connection ~ 5400 2550
-Wire Wire Line
-	5400 2550 5400 2600
 Wire Wire Line
 	6000 2300 5950 2300
-Wire Wire Line
-	6000 2550 6000 2300
-Wire Wire Line
-	5400 2550 6000 2550
-Wire Wire Line
-	5400 2500 5400 2550
 $Comp
 L Device:R R20
@@
 Wire Wire Line
 	5950 4150 6100 4150
-Connection ~ 5400 4500
-Wire Wire Line
-	5400 4500 5400 4550
 Wire Wire Line
 	6000 4250 5950 4250
-Wire Wire Line
-	6000 4500 6000 4250
-Wire Wire Line
-	5400 4500 6000 4500
-Wire Wire Line
-	5400 4450 5400 4500
 $Comp
 L Device:R R22
@@
 $EndComp
 Wire Wire Line
-	8700 4450 8700 4500
-Wire Wire Line
-	8700 4500 9300 4500
-Wire Wire Line
-	9300 4500 9300 4250
-Wire Wire Line
 	9300 4250 9250 4250
-Wire Wire Line
-	8700 4500 8700 4550
-Connection ~ 8700 4500
 Wire Wire Line
 	9250 4150 9400 4150
@@
 $EndComp
 Wire Wire Line
-	8700 2500 8700 2550
-Wire Wire Line
-	8700 2550 9300 2550
-Wire Wire Line
-	9300 2550 9300 2300
-Wire Wire Line
 	9300 2300 9250 2300
-Wire Wire Line
-	8700 2550 8700 2600
-Connection ~ 8700 2550
 Wire Wire Line
 	9250 2200 9400 2200
@@
 Text GLabel 8150 4050 0    50   Input ~ 0
 +VINB_16_INA
+Wire Wire Line
+	2100 2500 2100 2600
+Text GLabel 2700 2350 3    50   Input ~ 0
+SHTDWN_INA
+Wire Wire Line
+	2700 2300 2700 2350
+Text GLabel 2050 1450 0    50   Input ~ 0
+SHTDWN_INA
+Wire Wire Line
+	2050 1450 2100 1450
+Text GLabel 5350 1450 0    50   Input ~ 0
+SHTDWN_INA
+Wire Wire Line
+	5350 1450 5400 1450
+Text GLabel 8650 1450 0    50   Input ~ 0
+SHTDWN_INA
+Wire Wire Line
+	8650 1450 8700 1450
+Text GLabel 8650 3400 0    50   Input ~ 0
+SHTDWN_INA
+Wire Wire Line
+	8650 3400 8700 3400
+Text GLabel 5350 3400 0    50   Input ~ 0
+SHTDWN_INA
+Wire Wire Line
+	5350 3400 5400 3400
+Text GLabel 2050 3400 0    50   Input ~ 0
+SHTDWN_INA
+Wire Wire Line
+	2050 3400 2100 3400
+Text GLabel 2050 5350 0    50   Input ~ 0
+SHTDWN_INA
+Wire Wire Line
+	2050 5350 2100 5350
+Text GLabel 5350 5350 0    50   Input ~ 0
+SHTDWN_INA
+Wire Wire Line
+	5350 5350 5400 5350
+Wire Wire Line
+	5400 2500 5400 2600
+Wire Wire Line
+	2100 4450 2100 4550
+Wire Wire Line
+	2100 6400 2100 6500
+Wire Wire Line
+	5400 6400 5400 6500
+Wire Wire Line
+	5400 4450 5400 4550
+Wire Wire Line
+	8700 4450 8700 4550
+Wire Wire Line
+	8700 2500 8700 2600
+Text GLabel 6000 2350 3    50   Input ~ 0
+SHTDWN_INA
+Wire Wire Line
+	6000 2300 6000 2350
+Text GLabel 9300 2350 3    50   Input ~ 0
+SHTDWN_INA
+Wire Wire Line
+	9300 2300 9300 2350
+Text GLabel 9300 4300 3    50   Input ~ 0
+SHTDWN_INA
+Wire Wire Line
+	9300 4250 9300 4300
+Text GLabel 6000 4300 3    50   Input ~ 0
+SHTDWN_INA
+Wire Wire Line
+	6000 4250 6000 4300
+Text GLabel 2700 4300 3    50   Input ~ 0
+SHTDWN_INA
+Wire Wire Line
+	2700 4250 2700 4300
+Text GLabel 2700 6250 3    50   Input ~ 0
+SHTDWN_INA
+Wire Wire Line
+	2700 6200 2700 6250
+Text GLabel 6000 6250 3    50   Input ~ 0
+SHTDWN_INA
+Wire Wire Line
+	6000 6200 6000 6250
 $EndSCHEMATC
