File: hardware/kicad/emg-filter/instrumentation.sch (KiCad schematic (older format))
At the start: 40 parts, among them U1 INA2332, U2 INA2332, U3 INA2332, U4 INA2332, U5 INA2332, U6 INA2332, U7 INA2332, U8 INA2332

Commit message: annotation
Parts:
- renumbered R1 to R11, R2 to R12, R3 to R13, R4 to R14, R5 to R15, R6 to R16, R7 to R17, R8 to R18, R9 to R19, R10 to R20, R11 to R21, R12 to R22, R13 to R23, R14 to R24, R15 to R25, R16 to R26, R17 to R27, R18 to R28, R19 to R29, R20 to R30, R21 to R31, R22 to R32, R23 to R33, R24 to R34, R25 to R35, R26 to R36, R27 to R37, R28 to R38, R29 to R39, R30 to R40, R31 to R41, R32 to R42, U7 to U10, U8 to U11, U1 to U4, U2 to U5, U3 to U6, U4 to U7, U5 to U8, U6 to U9

Commit message: linked stages by renaming labels
Connections:
- net labels added: INA_BP_1, INA_BP_10, INA_BP_11, INA_BP_12, INA_BP_13, INA_BP_14, INA_BP_15, INA_BP_16, INA_BP_2, INA_BP_3, INA_BP_4, INA_BP_5, INA_BP_6, INA_BP_7, INA_BP_8, INA_BP_9
- net labels removed: VOUTA_11_INA, VOUTA_13_INA, VOUTA_15_INA, VOUTA_1_INA, VOUTA_3_INA, VOUTA_5_INA, VOUTA_7_INA, VOUTA_9_INA, VOUTB_10_INA, VOUTB_12_INA, VOUTB_14_INA, VOUTB_16_INA, VOUTB_2_INA, VOUTB_4_INA, VOUTB_6_INA, VOUTB_8_INA
Changed lines of the file:
@@
 $Descr A4 11693 8268
 encoding utf-8
-Sheet 1 10
+Sheet 3 10
 Title ""
 Date ""
@@
 Wire Wire Line
 	2650 5700 2800 5700
-Text GLabel 2800 5650 1    50   Input ~ 0
-VOUTA_5_INA
 Wire Wire Line
 	2800 5700 2800 5650
@@
 Wire Wire Line
 	2650 6100 2800 6100
-Text GLabel 2800 6150 3    50   Input ~ 0
-VOUTB_6_INA
 Wire Wire Line
 	2800 6100 2800 6150
@@
 Wire Wire Line
 	2800 2200 2800 2250
-Text GLabel 2800 2250 3    50   Input ~ 0
-VOUTB_2_INA
 Wire Wire Line
 	2650 2200 2800 2200
@@
 Wire Wire Line
 	2800 1800 2800 1750
-Text GLabel 2800 1750 1    50   Input ~ 0
-VOUTA_1_INA
 Wire Wire Line
 	2650 1800 2800 1800
@@
 Wire Wire Line
 	2800 4150 2800 4200
-Text GLabel 2800 4200 3    50   Input ~ 0
-VOUTB_4_INA
 Wire Wire Line
 	2650 4150 2800 4150
@@
 Wire Wire Line
 	2800 3750 2800 3700
-Text GLabel 2800 3700 1    50   Input ~ 0
-VOUTA_3_INA
 Wire Wire Line
 	2650 3750 2800 3750
@@
 Wire Wire Line
 	5950 5700 6100 5700
-Text GLabel 6100 5650 1    50   Input ~ 0
-VOUTA_11_INA
 Wire Wire Line
 	6100 5700 6100 5650
@@
 Wire Wire Line
 	5950 6100 6100 6100
-Text GLabel 6100 6150 3    50   Input ~ 0
-VOUTB_12_INA
 Wire Wire Line
 	6100 6100 6100 6150
@@
 Wire Wire Line
 	6100 2200 6100 2250
-Text GLabel 6100 2250 3    50   Input ~ 0
-VOUTB_8_INA
 Wire Wire Line
 	5950 2200 6100 2200
@@
 Wire Wire Line
 	6100 1800 6100 1750
-Text GLabel 6100 1750 1    50   Input ~ 0
-VOUTA_7_INA
 Wire Wire Line
 	5950 1800 6100 1800
@@
 Wire Wire Line
 	6100 4150 6100 4200
-Text GLabel 6100 4200 3    50   Input ~ 0
-VOUTB_10_INA
 Wire Wire Line
 	5950 4150 6100 4150
@@
 Wire Wire Line
 	6100 3750 6100 3700
-Text GLabel 6100 3700 1    50   Input ~ 0
-VOUTA_9_INA
 Wire Wire Line
 	5950 3750 6100 3750
@@
 Wire Wire Line
 	9250 3750 9400 3750
-Text GLabel 9400 3700 1    50   Input ~ 0
-VOUTA_15_INA
 Wire Wire Line
 	9400 3750 9400 3700
@@
 Wire Wire Line
 	9250 1800 9400 1800
-Text GLabel 9400 1750 1    50   Input ~ 0
-VOUTA_13_INA
 Wire Wire Line
 	9400 1800 9400 1750
@@
 Wire Wire Line
 	9250 2200 9400 2200
-Text GLabel 9400 2250 3    50   Input ~ 0
-VOUTB_14_INA
 Wire Wire Line
 	9400 2200 9400 2250
@@
 Text GLabel 10250 4050 2    50   Input ~ 0
 REFB_16_INA
-Text GLabel 9400 4200 3    50   Input ~ 0
-VOUTB_16_INA
 Text GLabel 8150 4150 0    50   Input ~ 0
 -VINB_16_INA
@@
 Wire Wire Line
 	6000 6200 6000 6250
+Text GLabel 2800 1750 1    50   Input ~ 0
+INA_BP_1
+Text GLabel 2800 2250 3    50   Input ~ 0
+INA_BP_2
+Text GLabel 2800 3700 1    50   Input ~ 0
+INA_BP_3
+Text GLabel 2800 4200 3    50   Input ~ 0
+INA_BP_4
+Text GLabel 2800 5650 1    50   Input ~ 0
+INA_BP_5
+Text GLabel 2800 6150 3    50   Input ~ 0
+INA_BP_6
+Text GLabel 6100 1750 1    50   Input ~ 0
+INA_BP_7
+Text GLabel 6100 2250 3    50   Input ~ 0
+INA_BP_8
+Text GLabel 6100 3700 1    50   Input ~ 0
+INA_BP_9
+Text GLabel 6100 4200 3    50   Input ~ 0
+INA_BP_10
+Text GLabel 6100 5650 1    50   Input ~ 0
+INA_BP_11
+Text GLabel 6100 6150 3    50   Input ~ 0
+INA_BP_12
+Text GLabel 9400 1750 1    50   Input ~ 0
+INA_BP_13
+Text GLabel 9400 2250 3    50   Input ~ 0
+INA_BP_14
+Text GLabel 9400 3700 1    50   Input ~ 0
+INA_BP_15
+Text GLabel 9400 4200 3    50   Input ~ 0
+INA_BP_16
 $EndSCHEMATC

Commit message: notes from review with Dmitry, 01-06-22
Other:
- note added: "Add caps near pwr pins\n"
Changed lines of the file:
@@
 Text GLabel 9400 4200 3    50   Input ~ 0
 INA_BP_16
+Text Notes 2150 1400 0    50   ~ 0
+Add caps near pwr pins\n
 $EndSCHEMATC
