File: hardware/kicad/emg-filter/instrumentation.sch (KiCad schematic (older format))
At the start: 40 parts, among them U10 INA2332, U11 INA2332, U4 INA2332, U5 INA2332, U6 INA2332, U7 INA2332, U8 INA2332, U9 INA2332

Commit message: pi connector and adc
Other:
- moved on the sheet: R11, R12, R13, R14, R15, R16, R17, R18, R19, R20, R21, R22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

Commit message: fixed rect labels
Parts:
- renumbered R13 to R10, R14 to R11, R15 to R12, R16 to R13, R17 to R14, R18 to R15, R19 to R16, R20 to R17, R21 to R18, R22 to R19, R23 to R20, R24 to R21, R25 to R22, R26 to R23, R27 to R24, R28 to R25, R29 to R26, R30 to R27, R31 to R28, R32 to R29, R33 to R30, R34 to R31, R35 to R32, R36 to R33, R37 to R34, R38 to R35, R39 to R36, R40 to R37, R41 to R38, R42 to R39, R11 to R8, R12 to R9, U11 to U10, U4 to U3, U5 to U4, U6 to U5, U7 to U6, U8 to U7, U9 to U8, U10 to U9

Commit message: footprint association
Parts:
- R262: renamed from R8; footprint (none) -> Resistor_SMD:R_0805_2012Metric
- R263: renamed from R9; footprint (none) -> Resistor_SMD:R_0805_2012Metric
- R264: renamed from R10; footprint (none) -> Resistor_SMD:R_0805_2012Metric
- R265: renamed from R11; footprint (none) -> Resistor_SMD:R_0805_2012Metric
- R266: renamed from R12; footprint (none) -> Resistor_SMD:R_0805_2012Metric
- R267: renamed from R13; footprint (none) -> Resistor_SMD:R_0805_2012Metric
- R268: renamed from R14; footprint (none) -> Resistor_SMD:R_0805_2012Metric
- R269: renamed from R15; footprint (none) -> Resistor_SMD:R_0805_2012Metric
- R270: renamed from R16; footprint (none) -> Resistor_SMD:R_0805_2012Metric
- R271: renamed from R17; footprint (none) -> Resistor_SMD:R_0805_2012Metric
- R272: renamed from R18; footprint (none) -> Resistor_SMD:R_0805_2012Metric
- R273: renamed from R19; footprint (none) -> Resistor_SMD:R_0805_2012Metric
- R274: renamed from R20; footprint (none) -> Resistor_SMD:R_0805_2012Metric
- R275: renamed from R21; footprint (none) -> Resistor_SMD:R_0805_2012Metric
- R276: renamed from R22; footprint (none) -> Resistor_SMD:R_0805_2012Metric
- R277: renamed from R23; footprint (none) -> Resistor_SMD:R_0805_2012Metric
- R278: renamed from R24; footprint (none) -> Resistor_SMD:R_0805_2012Metric
- R279: renamed from R25; footprint (none) -> Resistor_SMD:R_0805_2012Metric
- R280: renamed from R26; footprint (none) -> Resistor_SMD:R_0805_2012Metric
- R281: renamed from R27; footprint (none) -> Resistor_SMD:R_0805_2012Metric
- R282: renamed from R28; footprint (none) -> Resistor_SMD:R_0805_2012Metric
- R283: renamed from R29; footprint (none) -> Resistor_SMD:R_0805_2012Metric
- R284: renamed from R30; footprint (none) -> Resistor_SMD:R_0805_2012Metric
- R285: renamed from R31; footprint (none) -> Resistor_SMD:R_0805_2012Metric
- R286: renamed from R32; footprint (none) -> Resistor_SMD:R_0805_2012Metric
- R287: renamed from R33; footprint (none) -> Resistor_SMD:R_0805_2012Metric
- R288: renamed from R34; footprint (none) -> Resistor_SMD:R_0805_2012Metric
- R289: renamed from R35; footprint (none) -> Resistor_SMD:R_0805_2012Metric
- R290: renamed from R36; footprint (none) -> Resistor_SMD:R_0805_2012Metric
- R291: renamed from R37; footprint (none) -> Resistor_SMD:R_0805_2012Metric
- R292: renamed from R38; footprint (none) -> Resistor_SMD:R_0805_2012Metric
- R293: renamed from R39; footprint (none) -> Resistor_SMD:R_0805_2012Metric
- U53: renamed from U3; footprint (none) -> Package_SO:TSSOP-14_4.4x5mm_P0.65mm
- U54: renamed from U4; footprint (none) -> Package_SO:TSSOP-14_4.4x5mm_P0.65mm
- U55: renamed from U5; footprint (none) -> Package_SO:TSSOP-14_4.4x5mm_P0.65mm
- U56: renamed from U6; footprint (none) -> Package_SO:TSSOP-14_4.4x5mm_P0.65mm
- U57: renamed from U7; footprint (none) -> Package_SO:TSSOP-14_4.4x5mm_P0.65mm
- U58: renamed from U8; footprint (none) -> Package_SO:TSSOP-14_4.4x5mm_P0.65mm
- U59: renamed from U9; footprint (none) -> Package_SO:TSSOP-14_4.4x5mm_P0.65mm
- U60: renamed from U10; footprint (none) -> Package_SO:TSSOP-14_4.4x5mm_P0.65mm

Commit message: Solving Stuff for Free
Parts:
- renumbered R262 to R294, R263 to R295, R264 to R296, R265 to R297, R266 to R298, R267 to R299, R268 to R300, R269 to R301, R270 to R302, R271 to R303, R272 to R304, R273 to R305, R274 to R306, R275 to R307, R276 to R308, R277 to R309, R278 to R310, R279 to R311, R280 to R312, R281 to R313, R282 to R314, R283 to R315, R284 to R316, R285 to R317, R286 to R318, R287 to R319, R288 to R320, R289 to R321, R290 to R322, R291 to R323, R292 to R324, R293 to R325

Commit message: Block implementation
Parts:
- removed R294, R295, R296, R297: 191k, Resistor_SMD:R_0805_2012Metric, symbol Device:R
- removed R300, R301, R302, R303: 10k, Resistor_SMD:R_0805_2012Metric, symbol Device:R
- removed U53, U54: INA2332, Package_SO:TSSOP-14_4.4x5mm_P0.65mm, symbol emg-filter:INA2332
Connections:
- net labels removed: +VINA_1_INA, +VINA_3_INA, +VINB_2_INA, +VINB_4_INA, -VINA_1_INA, -VINA_3_INA, -VINB_2_INA, -VINB_4_INA, INA_BP_1, INA_BP_2, INA_BP_3, INA_BP_4, REFA_1_INA, REFA_3_INA, REFB_2_INA, REFB_4_INA
- wire segments 280 -> 210
