File: hardware/kicad/emg-filter/notch2.sch (KiCad schematic (older format))
At the start: 72 parts

Commit message: annotation
Parts:
- gave numbers to parts that had none: 72

Commit message: linked stages by renaming labels
Connections:
- net INPUT_10_NOTCH renamed BP_NOTCH_10
- net INPUT_11_NOTCH renamed BP_NOTCH_11
- net INPUT_12_NOTCH renamed BP_NOTCH_12
- net INPUT_13_NOTCH renamed BP_NOTCH_13
- net INPUT_14_NOTCH renamed BP_NOTCH_14
- net INPUT_15_NOTCH renamed BP_NOTCH_15
- net INPUT_16_NOTCH renamed BP_NOTCH_16
- net INPUT_9_NOTCH renamed BP_NOTCH_9
- net OUTPUT_10_NOTCH renamed NOTCH_RECT_10
- net OUTPUT_11_NOTCH renamed NOTCH_RECT_11
- net OUTPUT_12_NOTCH renamed NOTCH_RECT_12
- net OUTPUT_13_NOTCH renamed NOTCH_RECT_13
- net OUTPUT_14_NOTCH renamed NOTCH_RECT_14
- net OUTPUT_15_NOTCH renamed NOTCH_RECT_15
- net OUTPUT_16_NOTCH renamed NOTCH_RECT_16
- net OUTPUT_9_NOTCH renamed NOTCH_RECT_9
Changed lines of the file:
@@
 Wire Wire Line
 	2600 1850 2600 1800
-Text GLabel 1900 1000 0    50   Input ~ 0
-INPUT_9_NOTCH
 Wire Wire Line
 	1900 1000 1950 1000
@@
 Wire Wire Line
 	4900 1350 4900 1400
-Text GLabel 4950 1000 2    50   Input ~ 0
-OUTPUT_9_NOTCH
 $Comp
 L Device:R R?
@@
 	-1   0    0    1
 $EndComp
-Text GLabel 3850 1100 0    50   Input ~ 0
-OUTPUT_9_NOTCH
 Wire Wire Line
 	4700 1350 4700 1850
@@
 Wire Wire Line
 	2600 3250 2600 3200
-Text GLabel 1900 2400 0    50   Input ~ 0
-INPUT_10_NOTCH
 Wire Wire Line
 	1900 2400 1950 2400
@@
 Wire Wire Line
 	2600 4650 2600 4600
-Text GLabel 1900 3800 0    50   Input ~ 0
-INPUT_11_NOTCH
 Wire Wire Line
 	1900 3800 1950 3800
@@
 Wire Wire Line
 	4900 4150 4900 4200
-Text GLabel 4950 3800 2    50   Input ~ 0
-OUTPUT_11_NOTCH
 $Comp
 L Device:R R?
@@
 	-1   0    0    1
 $EndComp
-Text GLabel 3850 3900 0    50   Input ~ 0
-OUTPUT_11_NOTCH
 Wire Wire Line
 	4700 4150 4700 4650
@@
 Wire Wire Line
 	2550 6050 2550 6000
-Text GLabel 1850 5200 0    50   Input ~ 0
-INPUT_12_NOTCH
 Wire Wire Line
 	1850 5200 1900 5200
@@
 Wire Wire Line
 	4850 5550 4850 5600
-Text GLabel 4900 5200 2    50   Input ~ 0
-OUTPUT_12_NOTCH
 $Comp
 L Device:R R?
@@
 	-1   0    0    1
 $EndComp
-Text GLabel 3800 5300 0    50   Input ~ 0
-OUTPUT_12_NOTCH
 Wire Wire Line
 	4650 5550 4650 6050
@@
 Wire Wire Line
 	7500 1850 7500 1800
-Text GLabel 6800 1000 0    50   Input ~ 0
-INPUT_13_NOTCH
 Wire Wire Line
 	6800 1000 6850 1000
@@
 Wire Wire Line
 	9800 1350 9800 1400
-Text GLabel 9850 1000 2    50   Input ~ 0
-OUTPUT_13_NOTCH
 $Comp
 L Device:R R?
@@
 	-1   0    0    1
 $EndComp
-Text GLabel 8750 1100 0    50   Input ~ 0
-OUTPUT_13_NOTCH
 Wire Wire Line
 	9600 1350 9600 1850
@@
 Wire Wire Line
 	7500 3250 7500 3200
-Text GLabel 6800 2400 0    50   Input ~ 0
-INPUT_14_NOTCH
 Wire Wire Line
 	6800 2400 6850 2400
@@
 Wire Wire Line
 	9800 2750 9800 2800
-Text GLabel 9850 2400 2    50   Input ~ 0
-OUTPUT_14_NOTCH
 $Comp
 L Device:R R?
@@
 	-1   0    0    1
 $EndComp
-Text GLabel 8750 2500 0    50   Input ~ 0
-OUTPUT_14_NOTCH
 Wire Wire Line
 	9600 2750 9600 3250
@@
 Wire Wire Line
 	7500 4650 7500 4600
-Text GLabel 6800 3800 0    50   Input ~ 0
-INPUT_15_NOTCH
 Wire Wire Line
 	6800 3800 6850 3800
@@
 Wire Wire Line
 	9800 4150 9800 4200
-Text GLabel 9850 3800 2    50   Input ~ 0
-OUTPUT_15_NOTCH
 $Comp
 L Device:R R?
@@
 	-1   0    0    1
 $EndComp
-Text GLabel 8750 3900 0    50   Input ~ 0
-OUTPUT_15_NOTCH
 Wire Wire Line
 	9600 4150 9600 4650
@@
 Wire Wire Line
 	7450 6050 7450 6000
-Text GLabel 6750 5200 0    50   Input ~ 0
-INPUT_16_NOTCH
 Wire Wire Line
 	6750 5200 6800 5200
@@
 Wire Wire Line
 	9750 5550 9750 5600
-Text GLabel 9800 5200 2    50   Input ~ 0
-OUTPUT_16_NOTCH
 $Comp
 L Device:R R?
@@
 	-1   0    0    1
 $EndComp
-Text GLabel 8700 5300 0    50   Input ~ 0
-OUTPUT_16_NOTCH
 Wire Wire Line
 	9550 5550 9550 6050
@@
 Wire Wire Line
 	4900 2750 4900 2800
-Text GLabel 4950 2400 2    50   Input ~ 0
-OUTPUT_10_NOTCH
 $Comp
 L Device:R R?
@@
 	-1   0    0    1
 $EndComp
-Text GLabel 3850 2500 0    50   Input ~ 0
-OUTPUT_10_NOTCH
 Wire Wire Line
 	4700 2750 4700 3250
@@
 	2600 1850 3800 1850
 Connection ~ 2600 1850
+Text GLabel 1900 1000 0    50   Input ~ 0
+BP_NOTCH_9
+Text GLabel 1900 2400 0    50   Input ~ 0
+BP_NOTCH_10
+Text GLabel 1900 3800 0    50   Input ~ 0
+BP_NOTCH_11
+Text GLabel 6800 1000 0    50   Input ~ 0
+BP_NOTCH_13
+Text GLabel 6800 2400 0    50   Input ~ 0
+BP_NOTCH_14
+Text GLabel 6800 3800 0    50   Input ~ 0
+BP_NOTCH_15
+Text GLabel 6750 5200 0    50   Input ~ 0
+BP_NOTCH_16
+Text GLabel 1850 5200 0    50   Input ~ 0
+BP_NOTCH_12
+Text GLabel 4950 1000 2    50   Input ~ 0
+NOTCH_RECT_9
+Text GLabel 4950 2400 2    50   Input ~ 0
+NOTCH_RECT_10
+Text GLabel 4950 3800 2    50   Input ~ 0
+NOTCH_RECT_11
+Text GLabel 4900 5200 2    50   Input ~ 0
+NOTCH_RECT_12
+Text GLabel 9850 1000 2    50   Input ~ 0
+NOTCH_RECT_13
+Text GLabel 9850 2400 2    50   Input ~ 0
+NOTCH_RECT_14
+Text GLabel 9850 3800 2    50   Input ~ 0
+NOTCH_RECT_15
+Text GLabel 9800 5200 2    50   Input ~ 0
+NOTCH_RECT_16
+Text GLabel 3850 1100 0    50   Input ~ 0
+NOTCH_RECT_9
+Text GLabel 3850 2500 0    50   Input ~ 0
+NOTCH_RECT_10
+Text GLabel 3850 3900 0    50   Input ~ 0
+NOTCH_RECT_11
+Text GLabel 3800 5300 0    50   Input ~ 0
+NOTCH_RECT_12
+Text GLabel 8750 1100 0    50   Input ~ 0
+NOTCH_RECT_13
+Text GLabel 8750 2500 0    50   Input ~ 0
+NOTCH_RECT_14
+Text GLabel 8750 3900 0    50   Input ~ 0
+NOTCH_RECT_15
+Text GLabel 8700 5300 0    50   Input ~ 0
+NOTCH_RECT_16
 $EndSCHEMATC
