File: hardware/kicad/emg-filter/connectors.sch (KiCad schematic (older format))
At the start: 0 parts

Commit message: Update connectors.sch
Parts:
- added J? (x48): Conn_01x02, symbol Connector_Generic:Conn_01x02
- added R? (x30): 0, symbol Device:R
Connections:
- net labels added: +VINA_10_INA, +VINA_12_INA, +VINA_14_INA, +VINA_16_INA, +VINA_1_INA, +VINA_3_INA, +VINA_5_INA, +VINA_7_INA, +VINB_11_INA, +VINB_13_INA, +VINB_15_INA, +VINB_2_INA, +VINB_4_INA, +VINB_6_INA, +VINB_8_INA, +VINB_9_INA, -VINA_10_INA, -VINA_12_INA, -VINA_14_INA, -VINA_16_INA, -VINA_1_INA, -VINA_3_INA, -VINA_5_INA, -VINA_7_INA, -VINB_11_INA, -VINB_13_INA, -VINB_15_INA, -VINB_2_INA, -VINB_4_INA, -VINB_6_INA, -VINB_8_INA, -VINB_9_INA, GND, REFA_10_INA, REFA_12_INA, REFA_14_INA, REFA_16_INA, REFA_1_INA, REFA_3_INA, REFA_5_INA, REFA_7_INA, REFB_11_INA, REFB_13_INA, REFB_15_INA, REFB_2_INA, REFB_4_INA, REFB_6_INA, REFB_8_INA, REFB_9_INA
- wire segments 0 -> 252
