File: hardware/kicad/emg-filter/connectors.sch (KiCad schematic (older format))
At the start: 78 parts

Commit message: notes from review with Dmitry, 01-06-22
Other:
- note added: "Consider solder jumpers, associate R to JMP footprint"
Changed lines of the file:
@@
 Wire Wire Line
 	8250 1650 8700 1650
+Text Notes 4000 5850 0    50   ~ 0
+Consider solder jumpers, associate R to JMP footprint
 $EndSCHEMATC
