File: hardware/kicad/emg-filter/connectors.sch (KiCad schematic (older format))
At the start: 78 parts

Commit message: Rectifier Fit on US letter format
Parts:
- gave numbers to parts that had none: 78
