File: hardware/kicad/emg-filter/connectors.sch (KiCad schematic (older format))
At the start: 78 parts

Commit message: pi connector and adc
Parts:
- added J?: Conn_02x20_Odd_Even, symbol Connector_Generic:Conn_02x20_Odd_Even
Connections:
- net labels added: !CS_1_PI, !CS_2_PI, DGND, DIN_MOSI_PI, DOUT_MISO_PI, SCLK_CLK_PI, VD_3V3_PI
- no-connect marks 0 -> 2
Other:
- note added: "TX\nRX"
- moved on the sheet: R?
