File: hardware/kicad/emg-filter/adc.sch (KiCad schematic (older format))
At the start: 11 parts, among them U1 ADC108S102, U2 ADC108S102

Commit message: annotation
Parts:
- renumbered C2 to C100, C3 to C101, C4 to C102, C5 to C103, C6 to C104, C7 to C105, C8 to C106, C1 to C99, U1 to U60, U2 to U61
Changed lines of the file:
@@
 OUTPUT_6_AMPLFIER
 $Comp
-L Device:C C5
+L Device:C C103
 U 1 1 61C4C270
 P 7450 3600
-F 0 "C5" H 7450 3700 50  0000 L CNN
+F 0 "C103" H 7450 3700 50  0000 L CNN
 F 1 "0.1uF" H 7450 3500 50  0000 L CNN
 F 2 "" H 7488 3450 50  0001 C CNN
@@
 DGND
 $Comp
-L power:GND #PWR05
+L power:GND #PWR0205
 U 1 1 61C5013A
 P 3500 3650
-F 0 "#PWR05" H 3500 3400 50  0001 C CNN
+F 0 "#PWR0205" H 3500 3400 50  0001 C CNN
 F 1 "GND" H 3505 3477 50  0000 C CNN
 F 2 "" H 3500 3650 50  0001 C CNN
@@
 $EndComp
 $Comp
-L power:GND #PWR06
+L power:GND #PWR0206
 U 1 1 61C5028D
 P 3800 3650
-F 0 "#PWR06" H 3800 3400 50  0001 C CNN
+F 0 "#PWR0206" H 3800 3400 50  0001 C CNN
 F 1 "GND" H 3805 3477 50  0000 C CNN
 F 2 "" H 3800 3650 50  0001 C CNN
@@
 DGND
 $Comp
-L Device:C C7
+L Device:C C105
 U 1 1 61C50D59
 P 7700 3600
-F 0 "C7" H 7815 3646 50  0000 L CNN
+F 0 "C105" H 7815 3646 50  0000 L CNN
 F 1 "1.0uF" H 7815 3555 50  0000 L CNN
 F 2 "" H 7738 3450 50  0001 C CNN
@@
 $EndComp
 $Comp
-L power:+5V #PWR04
+L power:+5V #PWR0204
 U 1 1 61C654D9
 P 3500 3150
-F 0 "#PWR04" H 3500 3000 50  0001 C CNN
+F 0 "#PWR0204" H 3500 3000 50  0001 C CNN
 F 1 "+5V" H 3515 3323 50  0000 C CNN
 F 2 "" H 3500 3150 50  0001 C CNN
@@
 OUTPUT_14_AMPLFIER
 $Comp
-L Device:C C6
+L Device:C C104
 U 1 1 61C90C65
 P 7450 4750
-F 0 "C6" H 7450 4850 50  0000 L CNN
+F 0 "C104" H 7450 4850 50  0000 L CNN
 F 1 "0.1uF" H 7450 4650 50  0000 L CNN
 F 2 "" H 7488 4600 50  0001 C CNN
@@
 DGND
 $Comp
-L Device:C C8
+L Device:C C106
 U 1 1 61C90C6D
 P 7700 4750
-F 0 "C8" H 7815 4796 50  0000 L CNN
+F 0 "C106" H 7815 4796 50  0000 L CNN
 F 1 "1.0uF" H 7815 4705 50  0000 L CNN
 F 2 "" H 7738 4600 50  0001 C CNN
@@
 $EndComp
 $Comp
-L Device:C C2
+L Device:C C100
 U 1 1 61C90C73
 P 4450 4550
-F 0 "C2" H 4565 4596 50  0000 L CNN
+F 0 "C100" H 4565 4596 50  0000 L CNN
 F 1 "0.1uF" H 4565 4505 50  0000 L CNN
 F 2 "" H 4488 4400 50  0001 C CNN
@@
 SCLK_PI
 $Comp
-L emg-filter:ADC108S102 U1
+L emg-filter:ADC108S102 U60
 U 1 1 61C5454E
 P 6100 3450
-F 0 "U1" H 6100 4025 50  0000 C CNN
+F 0 "U60" H 6100 4025 50  0000 C CNN
 F 1 "ADC108S102" H 6100 3934 50  0000 C CNN
 F 2 "" H 6100 3975 50  0001 C CNN
@@
 $EndComp
 $Comp
-L emg-filter:ADC108S102 U2
+L emg-filter:ADC108S102 U61
 U 1 1 61C5515F
 P 6100 4600
-F 0 "U2" H 6100 5175 50  0000 C CNN
+F 0 "U61" H 6100 5175 50  0000 C CNN
 F 1 "ADC108S102" H 6100 5084 50  0000 C CNN
 F 2 "" H 6100 5125 50  0001 C CNN
@@
 $EndComp
 $Comp
-L power:+5V #PWR08
+L power:+5V #PWR0208
 U 1 1 61C598EB
 P 4450 4300
-F 0 "#PWR08" H 4450 4150 50  0001 C CNN
+F 0 "#PWR0208" H 4450 4150 50  0001 C CNN
 F 1 "+5V" H 4465 4473 50  0000 C CNN
 F 2 "" H 4450 4300 50  0001 C CNN
@@
 Connection ~ 4450 4350
 $Comp
-L Device:C C4
+L Device:C C102
 U 1 1 61CCDE4C
 P 4700 4550
-F 0 "C4" H 4750 4650 50  0000 L CNN
+F 0 "C102" H 4750 4650 50  0000 L CNN
 F 1 "1.0uF" H 4700 4450 50  0000 L CNN
 F 2 "" H 4738 4400 50  0001 C CNN
@@
 	4700 4350 4450 4350
 $Comp
-L Device:C C1
+L Device:C C99
 U 1 1 61CDD1F6
 P 4450 3400
-F 0 "C1" H 4565 3446 50  0000 L CNN
+F 0 "C99" H 4565 3446 50  0000 L CNN
 F 1 "0.1uF" H 4565 3355 50  0000 L CNN
 F 2 "" H 4488 3250 50  0001 C CNN
@@
 AGND
 $Comp
-L power:+5V #PWR07
+L power:+5V #PWR0207
 U 1 1 61CDD1FF
 P 4450 3150
-F 0 "#PWR07" H 4450 3000 50  0001 C CNN
+F 0 "#PWR0207" H 4450 3000 50  0001 C CNN
 F 1 "+5V" H 4465 3323 50  0000 C CNN
 F 2 "" H 4450 3150 50  0001 C CNN
@@
 Connection ~ 4450 3200
 $Comp
-L Device:C C3
+L Device:C C101
 U 1 1 61CDD207
 P 4700 3400
-F 0 "C3" H 4750 3500 50  0000 L CNN
+F 0 "C101" H 4750 3500 50  0000 L CNN
 F 1 "1.0uF" H 4700 3300 50  0000 L CNN
 F 2 "" H 4738 3250 50  0001 C CNN

Commit message: linked stages by renaming labels
Connections:
- net labels added: OUT_AMP_1, OUT_AMP_10, OUT_AMP_11, OUT_AMP_12, OUT_AMP_13, OUT_AMP_14, OUT_AMP_15, OUT_AMP_16, OUT_AMP_2, OUT_AMP_3, OUT_AMP_4, OUT_AMP_5, OUT_AMP_6, OUT_AMP_7, OUT_AMP_8, OUT_AMP_9
- net labels removed: OUTPUT_10_AMPLFIER, OUTPUT_11_AMPLFIER, OUTPUT_12_AMPLFIER, OUTPUT_13_AMPLFIER, OUTPUT_14_AMPLFIER, OUTPUT_15_AMPLFIER, OUTPUT_16_AMPLFIER, OUTPUT_1_AMPLFIER, OUTPUT_2_AMPLFIER, OUTPUT_3_AMPLFIER, OUTPUT_4_AMPLFIER, OUTPUT_5_AMPLFIER, OUTPUT_6_AMPLFIER, OUTPUT_7_AMPLFIER, OUTPUT_8_AMPLFIER, OUTPUT_9_AMPLFIER
Changed lines of the file:
@@
 $Descr A4 11693 8268
 encoding utf-8
-Sheet 1 10
+Sheet 9 10
 Title ""
 Date ""
@@
 Comment4 ""
 $EndDescr
-Text GLabel 5750 3400 0    50   Input ~ 0
-OUTPUT_1_AMPLFIER
-Text GLabel 5750 3500 0    50   Input ~ 0
-OUTPUT_2_AMPLFIER
-Text GLabel 5750 3600 0    50   Input ~ 0
-OUTPUT_3_AMPLFIER
-Text GLabel 5750 3700 0    50   Input ~ 0
-OUTPUT_4_AMPLFIER
-Text GLabel 5750 3800 0    50   Input ~ 0
-OUTPUT_5_AMPLFIER
-Text GLabel 6450 3700 2    50   Input ~ 0
-OUTPUT_7_AMPLFIER
-Text GLabel 6450 3600 2    50   Input ~ 0
-OUTPUT_8_AMPLFIER
-Text GLabel 6450 3800 2    50   Input ~ 0
-OUTPUT_6_AMPLFIER
 $Comp
 L Device:C C103
@@
 Text GLabel 6450 3100 2    50   Input ~ 0
 SCLK_PI
-Text GLabel 5750 4550 0    50   Input ~ 0
-OUTPUT_9_AMPLFIER
-Text GLabel 5750 4650 0    50   Input ~ 0
-OUTPUT_10_AMPLFIER
-Text GLabel 5750 4750 0    50   Input ~ 0
-OUTPUT_11_AMPLFIER
-Text GLabel 5750 4850 0    50   Input ~ 0
-OUTPUT_12_AMPLFIER
-Text GLabel 5750 4950 0    50   Input ~ 0
-OUTPUT_13_AMPLFIER
-Text GLabel 6450 4850 2    50   Input ~ 0
-OUTPUT_15_AMPLFIER
-Text GLabel 6450 4750 2    50   Input ~ 0
-OUTPUT_16_AMPLFIER
-Text GLabel 6450 4950 2    50   Input ~ 0
-OUTPUT_14_AMPLFIER
 $Comp
 L Device:C C104
@@
 Wire Wire Line
 	4700 3200 4450 3200
+Text GLabel 5750 3400 0    50   Input ~ 0
+OUT_AMP_1
+Text GLabel 5750 3500 0    50   Input ~ 0
+OUT_AMP_2
+Text GLabel 5750 3600 0    50   Input ~ 0
+OUT_AMP_3
+Text GLabel 5750 3700 0    50   Input ~ 0
+OUT_AMP_4
+Text GLabel 5750 3800 0    50   Input ~ 0
+OUT_AMP_5
+Text GLabel 5750 4850 0    50   Input ~ 0
+OUT_AMP_12
+Text GLabel 5750 4950 0    50   Input ~ 0
+OUT_AMP_13
+Text GLabel 6450 4950 2    50   Input ~ 0
+OUT_AMP_14
+Text GLabel 6450 4850 2    50   Input ~ 0
+OUT_AMP_15
+Text GLabel 6450 4750 2    50   Input ~ 0
+OUT_AMP_16
+Text GLabel 5750 4750 0    50   Input ~ 0
+OUT_AMP_11
+Text GLabel 6450 3800 2    50   Input ~ 0
+OUT_AMP_6
+Text GLabel 6450 3700 2    50   Input ~ 0
+OUT_AMP_7
+Text GLabel 6450 3600 2    50   Input ~ 0
+OUT_AMP_8
+Text GLabel 5750 4550 0    50   Input ~ 0
+OUT_AMP_9
+Text GLabel 5750 4650 0    50   Input ~ 0
+OUT_AMP_10
 $EndSCHEMATC

Commit message: notes from review with Dmitry, 01-06-22
Connections:
- net labels added: DGND_PI, VD_3V3_PI
Other:
- note added: "1.\nrun analog and digital gnd seperatly. 4 layer pc, 1 gnd plane for both analog and digital."
- note added: "Bead used for EMI, use LC filter"
- note added: "Can therefor get rid of LC filter\n"
- note added: "Connect VD to 3.3V of Pi\n"
- note added: "DOUT (adc) = MISO, DOUT should connect to DIN of Pi"
- note added: "VD should match logic level of Pi"
Changed lines of the file:
@@
 L power:GND #PWR0206
 U 1 1 61C5028D
-P 3800 3650
-F 0 "#PWR0206" H 3800 3400 50  0001 C CNN
-F 1 "GND" H 3805 3477 50  0000 C CNN
-F 2 "" H 3800 3650 50  0001 C CNN
-F 3 "" H 3800 3650 50  0001 C CNN
-	1    3800 3650
+P 3800 3750
+F 0 "#PWR0206" H 3800 3500 50  0001 C CNN
+F 1 "GND" H 3805 3577 50  0000 C CNN
+F 2 "" H 3800 3750 50  0001 C CNN
+F 3 "" H 3800 3750 50  0001 C CNN
+	1    3800 3750
 	1    0    0    -1
 $EndComp
 Text GLabel 3500 3650 1    50   Input ~ 0
 AGND
-Text GLabel 3800 3650 1    50   Input ~ 0
-DGND
+Text GLabel 3800 3750 1    50   Input ~ 0
+DGND_PI
 $Comp
 L Device:C C105
@@
 Connection ~ 7450 3400
 Text GLabel 7750 3400 2    50   Input ~ 0
-VD
+VD_3V3_PI
 Wire Wire Line
 	7700 3400 7750 3400
@@
 Text GLabel 5750 4650 0    50   Input ~ 0
 OUT_AMP_10
+Text Notes 7500 2950 0    50   ~ 0
+1.\nrun analog and digital gnd seperatly. 4 layer pc, 1 gnd plane for both analog and digital.
+Text Notes 6900 2650 0    50   ~ 0
+Bead used for EMI, use LC filter
+Text Notes 5350 3950 0    50   ~ 0
+DOUT (adc) = MISO, DOUT should connect to DIN of Pi
+Text Notes 7250 4400 0    50   ~ 0
+VD should match logic level of Pi
+Text Notes 7300 4500 0    50   ~ 0
+Connect VD to 3.3V of Pi\n
+Text Notes 8050 4600 0    50   ~ 0
+Can therefor get rid of LC filter\n
 $EndSCHEMATC
