File: hardware/kicad/emg-filter/adc.sch (KiCad schematic (older format))
At the start: 11 parts, among them U60 ADC108S102, U61 ADC108S102

Commit message: pi connector and adc
Parts:
- removed FB1: Ferrite_Bead_Small, symbol Device:Ferrite_Bead_Small
Connections:
- net labels added: DIN_MOSI_PI, DOUT_MISO_PI, SCLK_CLK_PI, VD_3V3_PI
- net labels removed: DIN_PI, DOUT_PI, SCLK_PI, VD
- wire segments 39 -> 43
Other:
- note removed: "1- How to split AGND and DGND, should they be on the same net?\n2- Is a ferrite bead fine for splitting analog and digital supply, vs coil vs 51ohm resistor?\n\nhttps://resources.altium.com/p/how-use-ferrite-bead-your-design-reduce-emi"
- note removed: "Questions:"
- moved on the sheet: C100, C101, C102, C103, C104, C105, C106, C99

Commit message: minor fixes
Parts:
- added J?: Conn_02x20_Odd_Even, symbol Connector_Generic:Conn_02x20_Odd_Even
Connections:
- no-connect marks 0 -> 2
Other:
- note added: "TX\nRX"
- moved on the sheet: C100, C101, C102, C103, C104, C105, C106, C99

Commit message: fixed rect labels
Parts:
- gave numbers to parts that had none: 1
- renumbered C99 to C206, C100 to C207, C101 to C208, C102 to C209, C103 to C210, C104 to C211, C105 to C212, C106 to C213, U60 to U59, U61 to U60
Changed lines of the file:
@@
 $EndDescr
 $Comp
-L Device:C C103
+L Device:C C210
 U 1 1 61C4C270
 P 6100 3400
-F 0 "C103" H 6100 3500 50  0000 L CNN
+F 0 "C210" H 6100 3500 50  0000 L CNN
 F 1 "0.1uF" H 6100 3300 50  0000 L CNN
 F 2 "" H 6138 3250 50  0001 C CNN
@@
 DGND
 $Comp
-L Device:C C105
+L Device:C C212
 U 1 1 61C50D59
 P 6350 3400
-F 0 "C105" H 6465 3446 50  0000 L CNN
+F 0 "C212" H 6465 3446 50  0000 L CNN
 F 1 "1.0uF" H 6465 3355 50  0000 L CNN
 F 2 "" H 6388 3250 50  0001 C CNN
@@
 SCLK_CLK_PI
 $Comp
-L Device:C C104
+L Device:C C211
 U 1 1 61C90C65
 P 6100 4550
-F 0 "C104" H 6100 4650 50  0000 L CNN
+F 0 "C211" H 6100 4650 50  0000 L CNN
 F 1 "0.1uF" H 6100 4450 50  0000 L CNN
 F 2 "" H 6138 4400 50  0001 C CNN
@@
 DGND
 $Comp
-L Device:C C106
+L Device:C C213
 U 1 1 61C90C6D
 P 6350 4550
-F 0 "C106" H 6465 4596 50  0000 L CNN
+F 0 "C213" H 6465 4596 50  0000 L CNN
 F 1 "1.0uF" H 6465 4505 50  0000 L CNN
 F 2 "" H 6388 4400 50  0001 C CNN
@@
 $EndComp
 $Comp
-L Device:C C100
+L Device:C C207
 U 1 1 61C90C73
 P 3100 4350
-F 0 "C100" H 3215 4396 50  0000 L CNN
+F 0 "C207" H 3215 4396 50  0000 L CNN
 F 1 "0.1uF" H 3215 4305 50  0000 L CNN
 F 2 "" H 3138 4200 50  0001 C CNN
@@
 !CS_2_PI
 $Comp
-L emg-filter:ADC108S102 U60
+L emg-filter:ADC108S102 U59
 U 1 1 61C5454E
 P 4750 3250
-F 0 "U60" H 4750 3825 50  0000 C CNN
+F 0 "U59" H 4750 3825 50  0000 C CNN
 F 1 "ADC108S102" H 4750 3734 50  0000 C CNN
 F 2 "" H 4750 3775 50  0001 C CNN
@@
 $EndComp
 $Comp
-L emg-filter:ADC108S102 U61
+L emg-filter:ADC108S102 U60
 U 1 1 61C5515F
 P 4750 4400
-F 0 "U61" H 4750 4975 50  0000 C CNN
+F 0 "U60" H 4750 4975 50  0000 C CNN
 F 1 "ADC108S102" H 4750 4884 50  0000 C CNN
 F 2 "" H 4750 4925 50  0001 C CNN
@@
 $EndComp
 $Comp
-L Device:C C102
+L Device:C C209
 U 1 1 61CCDE4C
 P 3350 4350
-F 0 "C102" H 3400 4450 50  0000 L CNN
+F 0 "C209" H 3400 4450 50  0000 L CNN
 F 1 "1.0uF" H 3350 4250 50  0000 L CNN
 F 2 "" H 3388 4200 50  0001 C CNN
@@
 	3350 4150 3100 4150
 $Comp
-L Device:C C99
+L Device:C C206
 U 1 1 61CDD1F6
 P 3100 3200
-F 0 "C99" H 3215 3246 50  0000 L CNN
+F 0 "C206" H 3215 3246 50  0000 L CNN
 F 1 "0.1uF" H 3215 3155 50  0000 L CNN
 F 2 "" H 3138 3050 50  0001 C CNN
@@
 	3100 3000 3100 3050
 $Comp
-L Device:C C101
+L Device:C C208
 U 1 1 61CDD207
 P 3350 3200
-F 0 "C101" H 3400 3300 50  0000 L CNN
+F 0 "C208" H 3400 3300 50  0000 L CNN
 F 1 "1.0uF" H 3350 3100 50  0000 L CNN
 F 2 "" H 3388 3050 50  0001 C CNN
@@
 AGND
 $Comp
-L power:GND #PWR0205
+L power:GND #PWR0188
 U 1 1 61C5013A
 P 4750 5325
-F 0 "#PWR0205" H 4750 5075 50  0001 C CNN
+F 0 "#PWR0188" H 4750 5075 50  0001 C CNN
 F 1 "GND" H 4755 5152 50  0000 C CNN
 F 2 "" H 4750 5325 50  0001 C CNN
@@
 Connection ~ 4750 5275
 $Comp
-L power:+5V #PWR?
+L power:+5V #PWR0186
 U 1 1 62012A20
 P 2900 2950
-F 0 "#PWR?" H 2900 2800 50  0001 C CNN
+F 0 "#PWR0186" H 2900 2800 50  0001 C CNN
 F 1 "+5V" H 2915 3123 50  0000 C CNN
 F 2 "" H 2900 2950 50  0001 C CNN
@@
 $EndComp
 $Comp
-L power:+5V #PWR0204
+L power:+5V #PWR0187
 U 1 1 61C654D9
 P 2900 4100
-F 0 "#PWR0204" H 2900 3950 50  0001 C CNN
+F 0 "#PWR0187" H 2900 3950 50  0001 C CNN
 F 1 "+5V" H 2915 4273 50  0000 C CNN
 F 2 "" H 2900 4100 50  0001 C CNN
@@
 !CS_1_PI
 $Comp
-L Connector_Generic:Conn_02x20_Odd_Even J?
+L Connector_Generic:Conn_02x20_Odd_Even J3
 U 1 1 6207EE55
 P 8200 3775
-F 0 "J?" H 8250 4892 50  0000 C CNN
+F 0 "J3" H 8250 4892 50  0000 C CNN
 F 1 "Conn_02x20_Odd_Even" H 8250 4801 50  0000 C CNN
 F 2 "" H 8200 3775 50  0001 C CNN

Commit message: -5V caps and cap voltages
Connections:
- no-connect marks 2 -> 33
Changed lines of the file:
@@
 $Descr USLetter 11000 8500
 encoding utf-8
-Sheet 10 11
+Sheet 9 11
 Title "EMG Filter for Prosthetic Limb Control System"
 Date "2022-01-07"
@@
 	1    0    0    -1
 $EndComp
+NoConn ~ 8000 2875
+NoConn ~ 8000 2975
+NoConn ~ 8000 3075
+NoConn ~ 8000 3175
+NoConn ~ 8000 3275
+NoConn ~ 8000 3375
+NoConn ~ 8000 4175
+NoConn ~ 8000 4275
+NoConn ~ 8000 4375
+NoConn ~ 8000 4475
+NoConn ~ 8000 4575
+NoConn ~ 8000 4675
+NoConn ~ 8000 4775
+NoConn ~ 8500 2875
+NoConn ~ 8500 2975
+NoConn ~ 8500 3075
+NoConn ~ 8500 3375
+NoConn ~ 8500 3475
+NoConn ~ 8500 3575
+NoConn ~ 8500 3675
+NoConn ~ 8500 3775
+NoConn ~ 8500 3875
+NoConn ~ 8500 3975
+NoConn ~ 8500 4075
+NoConn ~ 8500 4175
+NoConn ~ 8500 4275
+NoConn ~ 8500 4375
+NoConn ~ 8500 4475
+NoConn ~ 8500 4575
+NoConn ~ 8500 4675
+NoConn ~ 8500 4775
 $EndSCHEMATC

Commit message: footprint association
Parts:
- C206, C207, C208, C209, C210, C211, C212, C213: footprint (none) -> Capacitor_SMD:C_0805_2012Metric
- J3: footprint (none) -> Connector_PinHeader_2.54mm:PinHeader_2x20_P2.54mm_Vertical
- U51: renamed from U59; footprint (none) -> Package_SO:TSSOP-16_4.4x5mm_P0.65mm
- U52: renamed from U60; footprint (none) -> Package_SO:TSSOP-16_4.4x5mm_P0.65mm
Changed lines of the file:
@@
 F 0 "C210" H 6100 3500 50  0000 L CNN
 F 1 "0.1uF" H 6100 3300 50  0000 L CNN
-F 2 "" H 6138 3250 50  0001 C CNN
+F 2 "Capacitor_SMD:C_0805_2012Metric" H 6138 3250 50  0001 C CNN
 F 3 "~" H 6100 3400 50  0001 C CNN
 	1    6100 3400
@@
 F 0 "C212" H 6465 3446 50  0000 L CNN
 F 1 "1.0uF" H 6465 3355 50  0000 L CNN
-F 2 "" H 6388 3250 50  0001 C CNN
+F 2 "Capacitor_SMD:C_0805_2012Metric" H 6388 3250 50  0001 C CNN
 F 3 "~" H 6350 3400 50  0001 C CNN
 	1    6350 3400
@@
 F 0 "C211" H 6100 4650 50  0000 L CNN
 F 1 "0.1uF" H 6100 4450 50  0000 L CNN
-F 2 "" H 6138 4400 50  0001 C CNN
+F 2 "Capacitor_SMD:C_0805_2012Metric" H 6138 4400 50  0001 C CNN
 F 3 "~" H 6100 4550 50  0001 C CNN
 	1    6100 4550
@@
 F 0 "C213" H 6465 4596 50  0000 L CNN
 F 1 "1.0uF" H 6465 4505 50  0000 L CNN
-F 2 "" H 6388 4400 50  0001 C CNN
+F 2 "Capacitor_SMD:C_0805_2012Metric" H 6388 4400 50  0001 C CNN
 F 3 "~" H 6350 4550 50  0001 C CNN
 	1    6350 4550
@@
 F 0 "C207" H 3215 4396 50  0000 L CNN
 F 1 "0.1uF" H 3215 4305 50  0000 L CNN
-F 2 "" H 3138 4200 50  0001 C CNN
+F 2 "Capacitor_SMD:C_0805_2012Metric" H 3138 4200 50  0001 C CNN
 F 3 "~" H 3100 4350 50  0001 C CNN
 	1    3100 4350
@@
 !CS_2_PI
 $Comp
-L emg-filter:ADC108S102 U59
+L emg-filter:ADC108S102 U51
 U 1 1 61C5454E
 P 4750 3250
-F 0 "U59" H 4750 3825 50  0000 C CNN
+F 0 "U51" H 4750 3825 50  0000 C CNN
 F 1 "ADC108S102" H 4750 3734 50  0000 C CNN
-F 2 "" H 4750 3775 50  0001 C CNN
+F 2 "Package_SO:TSSOP-16_4.4x5mm_P0.65mm" H 4750 3775 50  0001 C CNN
 F 3 "https://www.ti.com/lit/ds/symlink/adc108s102.pdf" H 4750 3775 50  0001 C CNN
 	1    4750 3250
@@
 $EndComp
 $Comp
-L emg-filter:ADC108S102 U60
+L emg-filter:ADC108S102 U52
 U 1 1 61C5515F
 P 4750 4400
-F 0 "U60" H 4750 4975 50  0000 C CNN
+F 0 "U52" H 4750 4975 50  0000 C CNN
 F 1 "ADC108S102" H 4750 4884 50  0000 C CNN
-F 2 "" H 4750 4925 50  0001 C CNN
+F 2 "Package_SO:TSSOP-16_4.4x5mm_P0.65mm" H 4750 4925 50  0001 C CNN
 F 3 "https://www.ti.com/lit/ds/symlink/adc108s102.pdf" H 4750 4925 50  0001 C CNN
 	1    4750 4400
@@
 F 0 "C209" H 3400 4450 50  0000 L CNN
 F 1 "1.0uF" H 3350 4250 50  0000 L CNN
-F 2 "" H 3388 4200 50  0001 C CNN
+F 2 "Capacitor_SMD:C_0805_2012Metric" H 3388 4200 50  0001 C CNN
 F 3 "~" H 3350 4350 50  0001 C CNN
 	1    3350 4350
@@
 F 0 "C206" H 3215 3246 50  0000 L CNN
 F 1 "0.1uF" H 3215 3155 50  0000 L CNN
-F 2 "" H 3138 3050 50  0001 C CNN
+F 2 "Capacitor_SMD:C_0805_2012Metric" H 3138 3050 50  0001 C CNN
 F 3 "~" H 3100 3200 50  0001 C CNN
 	1    3100 3200
@@
 F 0 "C208" H 3400 3300 50  0000 L CNN
 F 1 "1.0uF" H 3350 3100 50  0000 L CNN
-F 2 "" H 3388 3050 50  0001 C CNN
+F 2 "Capacitor_SMD:C_0805_2012Metric" H 3388 3050 50  0001 C CNN
 F 3 "~" H 3350 3200 50  0001 C CNN
 	1    3350 3200
@@
 AGND
 $Comp
-L power:GND #PWR0188
+L power:GND #PWR0172
 U 1 1 61C5013A
 P 4750 5325
-F 0 "#PWR0188" H 4750 5075 50  0001 C CNN
+F 0 "#PWR0172" H 4750 5075 50  0001 C CNN
 F 1 "GND" H 4755 5152 50  0000 C CNN
 F 2 "" H 4750 5325 50  0001 C CNN
@@
 Connection ~ 4750 5275
 $Comp
-L power:+5V #PWR0186
+L power:+5V #PWR0170
 U 1 1 62012A20
 P 2900 2950
-F 0 "#PWR0186" H 2900 2800 50  0001 C CNN
+F 0 "#PWR0170" H 2900 2800 50  0001 C CNN
 F 1 "+5V" H 2915 3123 50  0000 C CNN
 F 2 "" H 2900 2950 50  0001 C CNN
@@
 $EndComp
 $Comp
-L power:+5V #PWR0187
+L power:+5V #PWR0171
 U 1 1 61C654D9
 P 2900 4100
-F 0 "#PWR0187" H 2900 3950 50  0001 C CNN
+F 0 "#PWR0171" H 2900 3950 50  0001 C CNN
 F 1 "+5V" H 2915 4273 50  0000 C CNN
 F 2 "" H 2900 4100 50  0001 C CNN
@@
 F 0 "J3" H 8250 4892 50  0000 C CNN
 F 1 "Conn_02x20_Odd_Even" H 8250 4801 50  0000 C CNN
-F 2 "" H 8200 3775 50  0001 C CNN
+F 2 "Connector_PinHeader_2.54mm:PinHeader_2x20_P2.54mm_Vertical" H 8200 3775 50  0001 C CNN
 F 3 "~" H 8200 3775 50  0001 C CNN
 	1    8200 3775

Commit message: Solving Stuff for Free
Connections:
- net labels added: +3.3V
- net labels removed: VD_3V3_PI
- wire segments 43 -> 42
Changed lines of the file:
@@
 	6100 3550 6100 3600
 Connection ~ 6100 3200
-Text GLabel 6400 3200 2    50   Input ~ 0
-VD_3V3_PI
-Wire Wire Line
-	6350 3200 6400 3200
-Connection ~ 6350 3200
 Wire Wire Line
 	6100 3200 6350 3200
@@
 	6350 3600 6350 3650
 Connection ~ 6350 3600
-Text GLabel 5100 3000 2    50   Input ~ 0
-DOUT_MISO_PI
 Text GLabel 5100 3100 2    50   Input ~ 0
 DIN_MOSI_PI
@@
 Wire Wire Line
 	3100 4150 3100 4200
-Wire Wire Line
-	6350 4350 6400 4350
-Connection ~ 6350 4350
 Wire Wire Line
 	6100 4350 6350 4350
@@
 Text GLabel 4400 4450 0    50   Input ~ 0
 OUT_AMP_10
-Text GLabel 5100 4150 2    50   Input ~ 0
-DOUT_MISO_PI
 Text GLabel 5100 4250 2    50   Input ~ 0
 DIN_MOSI_PI
 Text GLabel 5100 4050 2    50   Input ~ 0
 SCLK_CLK_PI
-Text GLabel 6400 4350 2    50   Input ~ 0
-VD_3V3_PI
 Wire Wire Line
 	2900 3000 3100 3000
@@
 AGND
 $Comp
-L power:GND #PWR0172
+L power:GND #PWR0170
 U 1 1 61C5013A
 P 4750 5325
-F 0 "#PWR0172" H 4750 5075 50  0001 C CNN
+F 0 "#PWR0170" H 4750 5075 50  0001 C CNN
 F 1 "GND" H 4755 5152 50  0000 C CNN
 F 2 "" H 4750 5325 50  0001 C CNN
@@
 Connection ~ 4750 5275
 $Comp
-L power:+5V #PWR0170
+L power:+5V #PWR0168
 U 1 1 62012A20
 P 2900 2950
-F 0 "#PWR0170" H 2900 2800 50  0001 C CNN
+F 0 "#PWR0168" H 2900 2800 50  0001 C CNN
 F 1 "+5V" H 2915 3123 50  0000 C CNN
 F 2 "" H 2900 2950 50  0001 C CNN
@@
 $EndComp
 $Comp
-L power:+5V #PWR0171
+L power:+5V #PWR0169
 U 1 1 61C654D9
 P 2900 4100
-F 0 "#PWR0171" H 2900 3950 50  0001 C CNN
+F 0 "#PWR0169" H 2900 3950 50  0001 C CNN
 F 1 "+5V" H 2915 4273 50  0000 C CNN
 F 2 "" H 2900 4100 50  0001 C CNN
@@
 Text GLabel 8000 4075 0    50   Input ~ 0
 DGND
-Text GLabel 8000 3675 0    50   Input ~ 0
-VD_3V3_PI
 Text GLabel 8000 3975 0    50   Input ~ 0
 SCLK_CLK_PI
 Text GLabel 8000 3775 0    50   Input ~ 0
 DIN_MOSI_PI
-Text GLabel 8000 3875 0    50   Input ~ 0
-DOUT_MISO_PI
 Text GLabel 8000 3575 0    50   Input ~ 0
 !CS_2_PI
@@
 NoConn ~ 8500 4675
 NoConn ~ 8500 4775
+Text GLabel 5100 3000 2    50   Output ~ 0
+DOUT_MISO_PI
+Text GLabel 5100 4150 2    50   Output ~ 0
+DOUT_MISO_PI
+Text GLabel 8000 3875 0    50   Input ~ 0
+DOUT_MISO_PI
+$Comp
+L power:+3.3V #PWR0172
+U 1 1 62C64A47
+P 6100 3200
+F 0 "#PWR0172" H 6100 3050 50  0001 C CNN
+F 1 "+3.3V" H 6115 3373 50  0000 C CNN
+F 2 "" H 6100 3200 50  0001 C CNN
+F 3 "" H 6100 3200 50  0001 C CNN
+	1    6100 3200
+	1    0    0    -1
+$EndComp
+$Comp
+L power:+3.3V #PWR0173
+U 1 1 62C64E5F
+P 6100 4350
+F 0 "#PWR0173" H 6100 4200 50  0001 C CNN
+F 1 "+3.3V" H 6115 4523 50  0000 C CNN
+F 2 "" H 6100 4350 50  0001 C CNN
+F 3 "" H 6100 4350 50  0001 C CNN
+	1    6100 4350
+	1    0    0    -1
+$EndComp
+$Comp
+L power:+3.3V #PWR0171
+U 1 1 62C6644F
+P 850 850
+F 0 "#PWR0171" H 850 700 50  0001 C CNN
+F 1 "+3.3V" H 865 1023 50  0000 C CNN
+F 2 "" H 850 850 50  0001 C CNN
+F 3 "" H 850 850 50  0001 C CNN
+	1    850  850
+	1    0    0    -1
+$EndComp
+$Comp
+L power:PWR_FLAG #FLG04
+U 1 1 62C66FCF
+P 850 850
+F 0 "#FLG04" H 850 925 50  0001 C CNN
+F 1 "PWR_FLAG" H 850 1023 50  0000 C CNN
+F 2 "" H 850 850 50  0001 C CNN
+F 3 "~" H 850 850 50  0001 C CNN
+	1    850  850
+	-1   0    0    1
+$EndComp
+$Comp
+L power:+3.3V #PWR0174
+U 1 1 62C658F1
+P 7325 3675
+F 0 "#PWR0174" H 7325 3525 50  0001 C CNN
+F 1 "+3.3V" V 7340 3803 50  0000 L CNN
+F 2 "" H 7325 3675 50  0001 C CNN
+F 3 "" H 7325 3675 50  0001 C CNN
+	1    7325 3675
+	1    0    0    -1
+$EndComp
+Wire Wire Line
+	8000 3675 7325 3675
 $EndSCHEMATC
