File: hardware/kicad/emg-filter/adc.sch (KiCad schematic (older format))
At the start: 11 parts, among them J3 Conn_02x20_Odd_Even, U51 ADC108S102, U52 ADC108S102

Commit message: fixed remaining errors
Parts:
- U51, U52: footprint Package_SO:TSSOP-16_4.4x5mm_P0.65mm -> (none)
Changed lines of the file:
@@
 !CS_2_PI
-$Comp
-L emg-filter:ADC108S102 U51
-U 1 1 61C5454E
-P 4750 3250
-F 0 "U51" H 4750 3825 50  0000 C CNN
-F 1 "ADC108S102" H 4750 3734 50  0000 C CNN
-F 2 "Package_SO:TSSOP-16_4.4x5mm_P0.65mm" H 4750 3775 50  0001 C CNN
-F 3 "https://www.ti.com/lit/ds/symlink/adc108s102.pdf" H 4750 3775 50  0001 C CNN
-	1    4750 3250
-	1    0    0    -1
-$EndComp
-$Comp
-L emg-filter:ADC108S102 U52
-U 1 1 61C5515F
-P 4750 4400
-F 0 "U52" H 4750 4975 50  0000 C CNN
-F 1 "ADC108S102" H 4750 4884 50  0000 C CNN
-F 2 "Package_SO:TSSOP-16_4.4x5mm_P0.65mm" H 4750 4925 50  0001 C CNN
-F 3 "https://www.ti.com/lit/ds/symlink/adc108s102.pdf" H 4750 4925 50  0001 C CNN
-	1    4750 4400
-	1    0    0    -1
-$EndComp
 $Comp
 L Device:C C209
@@
 NoConn ~ 8500 4675
 NoConn ~ 8500 4775
-Text GLabel 5100 3000 2    50   Output ~ 0
+Text GLabel 5100 3000 2    50   BiDi ~ 0
 DOUT_MISO_PI
-Text GLabel 5100 4150 2    50   Output ~ 0
+Text GLabel 5100 4150 2    50   BiDi ~ 0
 DOUT_MISO_PI
 Text GLabel 8000 3875 0    50   Input ~ 0
@@
 $EndComp
 $Comp
-L power:PWR_FLAG #FLG04
+L power:PWR_FLAG #FLG06
 U 1 1 62C66FCF
 P 850 850
-F 0 "#FLG04" H 850 925 50  0001 C CNN
+F 0 "#FLG06" H 850 925 50  0001 C CNN
 F 1 "PWR_FLAG" H 850 1023 50  0000 C CNN
 F 2 "" H 850 850 50  0001 C CNN
@@
 Wire Wire Line
 	8000 3675 7325 3675
+$Comp
+L emg-filter:ADC108S102 U51
+U 1 1 61E647A5
+P 4750 3250
+F 0 "U51" H 4750 3825 50  0000 C CNN
+F 1 "ADC108S102" H 4750 3734 50  0000 C CNN
+F 2 "" H 4750 3775 50  0001 C CNN
+F 3 "https://www.ti.com/lit/ds/symlink/adc108s102.pdf" H 4750 3775 50  0001 C CNN
+	1    4750 3250
+	1    0    0    -1
+$EndComp
+$Comp
+L emg-filter:ADC108S102 U52
+U 1 1 61E652F3
+P 4750 4400
+F 0 "U52" H 4750 4975 50  0000 C CNN
+F 1 "ADC108S102" H 4750 4884 50  0000 C CNN
+F 2 "" H 4750 4925 50  0001 C CNN
+F 3 "https://www.ti.com/lit/ds/symlink/adc108s102.pdf" H 4750 4925 50  0001 C CNN
+	1    4750 4400
+	1    0    0    -1
+$EndComp
 $EndSCHEMATC

Commit message: pcb
Parts:
- U51, U52: footprint (none) -> Package_SO:TSSOP-16_4.4x5mm_P0.65mm
Changed lines of the file:
@@
 F 0 "U51" H 4750 3825 50  0000 C CNN
 F 1 "ADC108S102" H 4750 3734 50  0000 C CNN
-F 2 "" H 4750 3775 50  0001 C CNN
+F 2 "Package_SO:TSSOP-16_4.4x5mm_P0.65mm" H 4750 3775 50  0001 C CNN
 F 3 "https://www.ti.com/lit/ds/symlink/adc108s102.pdf" H 4750 3775 50  0001 C CNN
 	1    4750 3250
@@
 F 0 "U52" H 4750 4975 50  0000 C CNN
 F 1 "ADC108S102" H 4750 4884 50  0000 C CNN
-F 2 "" H 4750 4925 50  0001 C CNN
+F 2 "Package_SO:TSSOP-16_4.4x5mm_P0.65mm" H 4750 4925 50  0001 C CNN
 F 3 "https://www.ti.com/lit/ds/symlink/adc108s102.pdf" H 4750 4925 50  0001 C CNN
 	1    4750 4400

Commit message: Fix Rectifier
Parts:
- U51, U52: symbol emg-filter:ADC108S102 -> emg-filter-rescue:ADC108S102-emg-filter
Changed lines of the file:
@@
 	8000 3675 7325 3675
 $Comp
-L emg-filter:ADC108S102 U51
+L emg-filter-rescue:ADC108S102-emg-filter U51
 U 1 1 61E647A5
 P 4750 3250
@@
 $EndComp
 $Comp
-L emg-filter:ADC108S102 U52
+L emg-filter-rescue:ADC108S102-emg-filter U52
 U 1 1 61E652F3
 P 4750 4400

Commit message: Block implementation
Parts:
- renumbered C206 to C158, C207 to C159, C208 to C160, C209 to C161, C210 to C162, C211 to C163, C212 to C164, C213 to C165, U51 to U43, U52 to U44
Changed lines of the file:
@@
 $Descr USLetter 11000 8500
 encoding utf-8
-Sheet 9 11
+Sheet 27 43
 Title "EMG Filter for Prosthetic Limb Control System"
 Date "2022-01-07"
@@
 $EndDescr
 $Comp
-L Device:C C210
+L Device:C C162
 U 1 1 61C4C270
 P 6100 3400
-F 0 "C210" H 6100 3500 50  0000 L CNN
+F 0 "C162" H 6100 3500 50  0000 L CNN
 F 1 "0.1uF" H 6100 3300 50  0000 L CNN
 F 2 "Capacitor_SMD:C_0805_2012Metric" H 6138 3250 50  0001 C CNN
@@
 DGND
 $Comp
-L Device:C C212
+L Device:C C164
 U 1 1 61C50D59
 P 6350 3400
-F 0 "C212" H 6465 3446 50  0000 L CNN
+F 0 "C164" H 6465 3446 50  0000 L CNN
 F 1 "1.0uF" H 6465 3355 50  0000 L CNN
 F 2 "Capacitor_SMD:C_0805_2012Metric" H 6388 3250 50  0001 C CNN
@@
 SCLK_CLK_PI
 $Comp
-L Device:C C211
+L Device:C C163
 U 1 1 61C90C65
 P 6100 4550
-F 0 "C211" H 6100 4650 50  0000 L CNN
+F 0 "C163" H 6100 4650 50  0000 L CNN
 F 1 "0.1uF" H 6100 4450 50  0000 L CNN
 F 2 "Capacitor_SMD:C_0805_2012Metric" H 6138 4400 50  0001 C CNN
@@
 DGND
 $Comp
-L Device:C C213
+L Device:C C165
 U 1 1 61C90C6D
 P 6350 4550
-F 0 "C213" H 6465 4596 50  0000 L CNN
+F 0 "C165" H 6465 4596 50  0000 L CNN
 F 1 "1.0uF" H 6465 4505 50  0000 L CNN
 F 2 "Capacitor_SMD:C_0805_2012Metric" H 6388 4400 50  0001 C CNN
@@
 $EndComp
 $Comp
-L Device:C C207
+L Device:C C159
 U 1 1 61C90C73
 P 3100 4350
-F 0 "C207" H 3215 4396 50  0000 L CNN
+F 0 "C159" H 3215 4396 50  0000 L CNN
 F 1 "0.1uF" H 3215 4305 50  0000 L CNN
 F 2 "Capacitor_SMD:C_0805_2012Metric" H 3138 4200 50  0001 C CNN
@@
 !CS_2_PI
 $Comp
-L Device:C C209
+L Device:C C161
 U 1 1 61CCDE4C
 P 3350 4350
-F 0 "C209" H 3400 4450 50  0000 L CNN
+F 0 "C161" H 3400 4450 50  0000 L CNN
 F 1 "1.0uF" H 3350 4250 50  0000 L CNN
 F 2 "Capacitor_SMD:C_0805_2012Metric" H 3388 4200 50  0001 C CNN
@@
 	3350 4150 3100 4150
 $Comp
-L Device:C C206
+L Device:C C158
 U 1 1 61CDD1F6
 P 3100 3200
-F 0 "C206" H 3215 3246 50  0000 L CNN
+F 0 "C158" H 3215 3246 50  0000 L CNN
 F 1 "0.1uF" H 3215 3155 50  0000 L CNN
 F 2 "Capacitor_SMD:C_0805_2012Metric" H 3138 3050 50  0001 C CNN
@@
 	3100 3000 3100 3050
 $Comp
-L Device:C C208
+L Device:C C160
 U 1 1 61CDD207
 P 3350 3200
-F 0 "C208" H 3400 3300 50  0000 L CNN
+F 0 "C160" H 3400 3300 50  0000 L CNN
 F 1 "1.0uF" H 3350 3100 50  0000 L CNN
 F 2 "Capacitor_SMD:C_0805_2012Metric" H 3388 3050 50  0001 C CNN
@@
 Wire Wire Line
 	3350 3000 3100 3000
-Text GLabel 4400 3200 0    50   Input ~ 0
-OUT_AMP_1
-Text GLabel 4400 3300 0    50   Input ~ 0
-OUT_AMP_2
-Text GLabel 4400 3400 0    50   Input ~ 0
-OUT_AMP_3
-Text GLabel 4400 3500 0    50   Input ~ 0
-OUT_AMP_4
-Text GLabel 4400 3600 0    50   Input ~ 0
-OUT_AMP_5
-Text GLabel 4400 4650 0    50   Input ~ 0
-OUT_AMP_12
-Text GLabel 4400 4750 0    50   Input ~ 0
-OUT_AMP_13
-Text GLabel 5100 4750 2    50   Input ~ 0
-OUT_AMP_14
-Text GLabel 5100 4650 2    50   Input ~ 0
-OUT_AMP_15
-Text GLabel 5100 4550 2    50   Input ~ 0
-OUT_AMP_16
-Text GLabel 4400 4550 0    50   Input ~ 0
-OUT_AMP_11
-Text GLabel 5100 3600 2    50   Input ~ 0
-OUT_AMP_6
-Text GLabel 5100 3500 2    50   Input ~ 0
-OUT_AMP_7
-Text GLabel 5100 3400 2    50   Input ~ 0
-OUT_AMP_8
-Text GLabel 4400 4350 0    50   Input ~ 0
-OUT_AMP_9
-Text GLabel 4400 4450 0    50   Input ~ 0
-OUT_AMP_10
 Text GLabel 5100 4250 2    50   Input ~ 0
 DIN_MOSI_PI
@@
 AGND
 $Comp
-L power:GND #PWR0169
+L power:GND #PWR0145
 U 1 1 61C5013A
 P 4750 5325
-F 0 "#PWR0169" H 4750 5075 50  0001 C CNN
+F 0 "#PWR0145" H 4750 5075 50  0001 C CNN
 F 1 "GND" H 4755 5152 50  0000 C CNN
 F 2 "" H 4750 5325 50  0001 C CNN
@@
 Connection ~ 4750 5275
 $Comp
-L power:+5V #PWR0167
+L power:+5V #PWR0143
 U 1 1 62012A20
 P 2900 2950
-F 0 "#PWR0167" H 2900 2800 50  0001 C CNN
+F 0 "#PWR0143" H 2900 2800 50  0001 C CNN
 F 1 "+5V" H 2915 3123 50  0000 C CNN
 F 2 "" H 2900 2950 50  0001 C CNN
@@
 $EndComp
 $Comp
-L power:+5V #PWR0168
+L power:+5V #PWR0144
 U 1 1 61C654D9
 P 2900 4100
-F 0 "#PWR0168" H 2900 3950 50  0001 C CNN
+F 0 "#PWR0144" H 2900 3950 50  0001 C CNN
 F 1 "+5V" H 2915 4273 50  0000 C CNN
 F 2 "" H 2900 4100 50  0001 C CNN
@@
 DOUT_MISO_PI
 $Comp
-L power:+3.3V #PWR0170
+L power:+3.3V #PWR0146
 U 1 1 62C64A47
 P 6100 3200
-F 0 "#PWR0170" H 6100 3050 50  0001 C CNN
+F 0 "#PWR0146" H 6100 3050 50  0001 C CNN
 F 1 "+3.3V" H 6115 3373 50  0000 C CNN
 F 2 "" H 6100 3200 50  0001 C CNN
@@
 $EndComp
 $Comp
-L power:+3.3V #PWR0171
+L power:+3.3V #PWR0147
 U 1 1 62C64E5F
 P 6100 4350
-F 0 "#PWR0171" H 6100 4200 50  0001 C CNN
+F 0 "#PWR0147" H 6100 4200 50  0001 C CNN
 F 1 "+3.3V" H 6115 4523 50  0000 C CNN
 F 2 "" H 6100 4350 50  0001 C CNN
@@
 $EndComp
 $Comp
-L power:+3.3V #PWR0166
+L power:+3.3V #PWR0142
 U 1 1 62C6644F
 P 850 850
-F 0 "#PWR0166" H 850 700 50  0001 C CNN
+F 0 "#PWR0142" H 850 700 50  0001 C CNN
 F 1 "+3.3V" H 865 1023 50  0000 C CNN
 F 2 "" H 850 850 50  0001 C CNN
@@
 $EndComp
 $Comp
-L power:+3.3V #PWR0172
+L power:+3.3V #PWR0148
 U 1 1 62C658F1
 P 7325 3675
-F 0 "#PWR0172" H 7325 3525 50  0001 C CNN
+F 0 "#PWR0148" H 7325 3525 50  0001 C CNN
 F 1 "+3.3V" V 7340 3803 50  0000 L CNN
 F 2 "" H 7325 3675 50  0001 C CNN
@@
 	8000 3675 7325 3675
 $Comp
-L emg-filter-rescue:ADC108S102-emg-filter U51
+L emg-filter-rescue:ADC108S102-emg-filter U43
 U 1 1 61E647A5
 P 4750 3250
-F 0 "U51" H 4750 3825 50  0000 C CNN
+F 0 "U43" H 4750 3825 50  0000 C CNN
 F 1 "ADC108S102" H 4750 3734 50  0000 C CNN
 F 2 "Package_SO:TSSOP-16_4.4x5mm_P0.65mm" H 4750 3775 50  0001 C CNN
@@
 $EndComp
 $Comp
-L emg-filter-rescue:ADC108S102-emg-filter U52
+L emg-filter-rescue:ADC108S102-emg-filter U44
 U 1 1 61E652F3
 P 4750 4400
-F 0 "U52" H 4750 4975 50  0000 C CNN
+F 0 "U44" H 4750 4975 50  0000 C CNN
 F 1 "ADC108S102" H 4750 4884 50  0000 C CNN
 F 2 "Package_SO:TSSOP-16_4.4x5mm_P0.65mm" H 4750 4925 50  0001 C CNN
@@
 	1    0    0    -1
 $EndComp
+Text HLabel 4400 3200 0    50   Input ~ 0
+OUT_AMP_1
+Text HLabel 4400 3300 0    50   Input ~ 0
+OUT_AMP_2
+Text HLabel 4400 3400 0    50   Input ~ 0
+OUT_AMP_3
+Text HLabel 4400 3500 0    50   Input ~ 0
+OUT_AMP_4
+Text HLabel 4400 3600 0    50   Input ~ 0
+OUT_AMP_5
+Text HLabel 5100 3600 2    50   Input ~ 0
+OUT_AMP_6
+Text HLabel 5100 3500 2    50   Input ~ 0
+OUT_AMP_7
+Text HLabel 5100 3400 2    50   Input ~ 0
+OUT_AMP_8
+Text HLabel 4400 4350 0    50   Input ~ 0
+OUT_AMP_9
+Text HLabel 4400 4450 0    50   Input ~ 0
+OUT_AMP_10
+Text HLabel 4400 4550 0    50   Input ~ 0
+OUT_AMP_11
+Text HLabel 4400 4650 0    50   Input ~ 0
+OUT_AMP_12
+Text HLabel 4400 4750 0    50   Input ~ 0
+OUT_AMP_13
+Text HLabel 5100 4750 2    50   Input ~ 0
+OUT_AMP_14
+Text HLabel 5100 4650 2    50   Input ~ 0
+OUT_AMP_15
+Text HLabel 5100 4550 2    50   Input ~ 0
+OUT_AMP_16
 $EndSCHEMATC

Commit message: Fixed errors
Parts:
- removed U43, U44: ADC108S102, Package_SO:TSSOP-16_4.4x5mm_P0.65mm, symbol emg-filter-rescue:ADC108S102-emg-filter
- added U43, U44: ADC108S102, Package_SO:TSSOP-16_4.4x5mm_P0.65mm, symbol emg-filter:ADC108S102
Changed lines of the file:
@@
 $EndComp
 $Comp
-L power:PWR_FLAG #FLG06
+L power:PWR_FLAG #FLG05
 U 1 1 62C66FCF
 P 850 850
-F 0 "#FLG06" H 850 925 50  0001 C CNN
+F 0 "#FLG05" H 850 925 50  0001 C CNN
 F 1 "PWR_FLAG" H 850 1023 50  0000 C CNN
 F 2 "" H 850 850 50  0001 C CNN
@@
 Wire Wire Line
 	8000 3675 7325 3675
-$Comp
-L emg-filter-rescue:ADC108S102-emg-filter U43
-U 1 1 61E647A5
-P 4750 3250
-F 0 "U43" H 4750 3825 50  0000 C CNN
-F 1 "ADC108S102" H 4750 3734 50  0000 C CNN
-F 2 "Package_SO:TSSOP-16_4.4x5mm_P0.65mm" H 4750 3775 50  0001 C CNN
-F 3 "https://www.ti.com/lit/ds/symlink/adc108s102.pdf" H 4750 3775 50  0001 C CNN
-	1    4750 3250
-	1    0    0    -1
-$EndComp
-$Comp
-L emg-filter-rescue:ADC108S102-emg-filter U44
-U 1 1 61E652F3
-P 4750 4400
-F 0 "U44" H 4750 4975 50  0000 C CNN
-F 1 "ADC108S102" H 4750 4884 50  0000 C CNN
-F 2 "Package_SO:TSSOP-16_4.4x5mm_P0.65mm" H 4750 4925 50  0001 C CNN
-F 3 "https://www.ti.com/lit/ds/symlink/adc108s102.pdf" H 4750 4925 50  0001 C CNN
-	1    4750 4400
-	1    0    0    -1
-$EndComp
 Text HLabel 4400 3200 0    50   Input ~ 0
 OUT_AMP_1
@@
 Text HLabel 5100 4550 2    50   Input ~ 0
 OUT_AMP_16
+$Comp
+L emg-filter:ADC108S102 U43
+U 1 1 61EDDCFE
+P 4750 3250
+F 0 "U43" H 4750 3825 50  0000 C CNN
+F 1 "ADC108S102" H 4750 3734 50  0000 C CNN
+F 2 "Package_SO:TSSOP-16_4.4x5mm_P0.65mm" H 4750 3775 50  0001 C CNN
+F 3 "https://www.ti.com/lit/ds/symlink/adc108s102.pdf" H 4750 3775 50  0001 C CNN
+	1    4750 3250
+	1    0    0    -1
+$EndComp
+$Comp
+L emg-filter:ADC108S102 U44
+U 1 1 61EDF58B
+P 4750 4400
+F 0 "U44" H 4750 4975 50  0000 C CNN
+F 1 "ADC108S102" H 4750 4884 50  0000 C CNN
+F 2 "Package_SO:TSSOP-16_4.4x5mm_P0.65mm" H 4750 4925 50  0001 C CNN
+F 3 "https://www.ti.com/lit/ds/symlink/adc108s102.pdf" H 4750 4925 50  0001 C CNN
+	1    4750 4400
+	1    0    0    -1
+$EndComp
 $EndSCHEMATC

Commit message: compact design
Parts:
- renumbered C158 to C206, C159 to C207, C160 to C208, C161 to C209, C162 to C210, C163 to C211, C164 to C212, C165 to C213
Changed lines of the file:
@@
 $EndDescr
 $Comp
-L Device:C C162
+L Device:C C210
 U 1 1 61C4C270
 P 6100 3400
-F 0 "C162" H 6100 3500 50  0000 L CNN
+F 0 "C210" H 6100 3500 50  0000 L CNN
 F 1 "0.1uF" H 6100 3300 50  0000 L CNN
 F 2 "Capacitor_SMD:C_0805_2012Metric" H 6138 3250 50  0001 C CNN
@@
 DGND
 $Comp
-L Device:C C164
+L Device:C C212
 U 1 1 61C50D59
 P 6350 3400
-F 0 "C164" H 6465 3446 50  0000 L CNN
+F 0 "C212" H 6465 3446 50  0000 L CNN
 F 1 "1.0uF" H 6465 3355 50  0000 L CNN
 F 2 "Capacitor_SMD:C_0805_2012Metric" H 6388 3250 50  0001 C CNN
@@
 SCLK_CLK_PI
 $Comp
-L Device:C C163
+L Device:C C211
 U 1 1 61C90C65
 P 6100 4550
-F 0 "C163" H 6100 4650 50  0000 L CNN
+F 0 "C211" H 6100 4650 50  0000 L CNN
 F 1 "0.1uF" H 6100 4450 50  0000 L CNN
 F 2 "Capacitor_SMD:C_0805_2012Metric" H 6138 4400 50  0001 C CNN
@@
 DGND
 $Comp
-L Device:C C165
+L Device:C C213
 U 1 1 61C90C6D
 P 6350 4550
-F 0 "C165" H 6465 4596 50  0000 L CNN
+F 0 "C213" H 6465 4596 50  0000 L CNN
 F 1 "1.0uF" H 6465 4505 50  0000 L CNN
 F 2 "Capacitor_SMD:C_0805_2012Metric" H 6388 4400 50  0001 C CNN
@@
 $EndComp
 $Comp
-L Device:C C159
+L Device:C C207
 U 1 1 61C90C73
 P 3100 4350
-F 0 "C159" H 3215 4396 50  0000 L CNN
+F 0 "C207" H 3215 4396 50  0000 L CNN
 F 1 "0.1uF" H 3215 4305 50  0000 L CNN
 F 2 "Capacitor_SMD:C_0805_2012Metric" H 3138 4200 50  0001 C CNN
@@
 !CS_2_PI
 $Comp
-L Device:C C161
+L Device:C C209
 U 1 1 61CCDE4C
 P 3350 4350
-F 0 "C161" H 3400 4450 50  0000 L CNN
+F 0 "C209" H 3400 4450 50  0000 L CNN
 F 1 "1.0uF" H 3350 4250 50  0000 L CNN
 F 2 "Capacitor_SMD:C_0805_2012Metric" H 3388 4200 50  0001 C CNN
@@
 	3350 4150 3100 4150
 $Comp
-L Device:C C158
+L Device:C C206
 U 1 1 61CDD1F6
 P 3100 3200
-F 0 "C158" H 3215 3246 50  0000 L CNN
+F 0 "C206" H 3215 3246 50  0000 L CNN
 F 1 "0.1uF" H 3215 3155 50  0000 L CNN
 F 2 "Capacitor_SMD:C_0805_2012Metric" H 3138 3050 50  0001 C CNN
@@
 	3100 3000 3100 3050
 $Comp
-L Device:C C160
+L Device:C C208
 U 1 1 61CDD207
 P 3350 3200
-F 0 "C160" H 3400 3300 50  0000 L CNN
+F 0 "C208" H 3400 3300 50  0000 L CNN
 F 1 "1.0uF" H 3350 3100 50  0000 L CNN
 F 2 "Capacitor_SMD:C_0805_2012Metric" H 3388 3050 50  0001 C CNN

Commit message: modular design
Other:
- moved on the sheet: C206, C208, C210, C212
Changed lines of the file:
@@
 $Descr USLetter 11000 8500
 encoding utf-8
-Sheet 27 43
+Sheet 55 55
 Title "EMG Filter for Prosthetic Limb Control System"
 Date "2022-01-07"
@@
 L Device:C C210
 U 1 1 61C4C270
-P 6100 3400
-F 0 "C210" H 6100 3500 50  0000 L CNN
-F 1 "0.1uF" H 6100 3300 50  0000 L CNN
-F 2 "Capacitor_SMD:C_0805_2012Metric" H 6138 3250 50  0001 C CNN
-F 3 "~" H 6100 3400 50  0001 C CNN
-	1    6100 3400
-	1    0    0    -1
-$EndComp
-Text GLabel 4400 3100 0    50   Input ~ 0
+P 6075 2775
+F 0 "C210" H 6075 2875 50  0000 L CNN
+F 1 "0.1uF" H 6075 2675 50  0000 L CNN
+F 2 "Capacitor_SMD:C_0805_2012Metric" H 6113 2625 50  0001 C CNN
+F 3 "~" H 6075 2775 50  0001 C CNN
+	1    6075 2775
+	1    0    0    -1
+$EndComp
+Text GLabel 4375 2475 0    50   Input ~ 0
 AGND
-Text GLabel 5100 3300 2    50   Input ~ 0
+Text GLabel 5075 2675 2    50   Input ~ 0
 DGND
 $Comp
 L Device:C C212
 U 1 1 61C50D59
-P 6350 3400
-F 0 "C212" H 6465 3446 50  0000 L CNN
-F 1 "1.0uF" H 6465 3355 50  0000 L CNN
-F 2 "Capacitor_SMD:C_0805_2012Metric" H 6388 3250 50  0001 C CNN
-F 3 "~" H 6350 3400 50  0001 C CNN
-	1    6350 3400
-	1    0    0    -1
-$EndComp
-Wire Wire Line
-	6100 3250 6100 3200
-Wire Wire Line
-	6350 3200 6350 3250
-Text GLabel 6350 3650 3    50   Input ~ 0
-DGND
-Wire Wire Line
-	6100 3550 6100 3600
-Connection ~ 6100 3200
-Wire Wire Line
-	6100 3200 6350 3200
-Wire Wire Line
-	5100 3200 6100 3200
-Wire Wire Line
-	6100 3600 6350 3600
-Wire Wire Line
-	6350 3600 6350 3550
-Wire Wire Line
-	6350 3600 6350 3650
-Connection ~ 6350 3600
-Text GLabel 5100 3100 2    50   Input ~ 0
+P 6325 2775
+F 0 "C212" H 6440 2821 50  0000 L CNN
+F 1 "1.0uF" H 6440 2730 50  0000 L CNN
+F 2 "Capacitor_SMD:C_0805_2012Metric" H 6363 2625 50  0001 C CNN
+F 3 "~" H 6325 2775 50  0001 C CNN
+	1    6325 2775
+	1    0    0    -1
+$EndComp
+Wire Wire Line
+	6075 2625 6075 2575
+Wire Wire Line
+	6325 2575 6325 2625
+Text GLabel 6325 3025 3    50   Input ~ 0
+DGND
+Wire Wire Line
+	6075 2925 6075 2975
+Connection ~ 6075 2575
+Wire Wire Line
+	6075 2575 6325 2575
+Wire Wire Line
+	5075 2575 6075 2575
+Wire Wire Line
+	6075 2975 6325 2975
+Wire Wire Line
+	6325 2975 6325 2925
+Wire Wire Line
+	6325 2975 6325 3025
+Connection ~ 6325 2975
+Text GLabel 5075 2475 2    50   Input ~ 0
 DIN_MOSI_PI
-Text GLabel 4400 2900 0    50   Input ~ 0
+Text GLabel 4375 2275 0    50   Input ~ 0
 !CS_1_PI
-Text GLabel 5100 2900 2    50   Input ~ 0
+Text GLabel 5075 2275 2    50   Input ~ 0
 SCLK_CLK_PI
 $Comp
@@
 L Device:C C206
 U 1 1 61CDD1F6
-P 3100 3200
-F 0 "C206" H 3215 3246 50  0000 L CNN
-F 1 "0.1uF" H 3215 3155 50  0000 L CNN
-F 2 "Capacitor_SMD:C_0805_2012Metric" H 3138 3050 50  0001 C CNN
-F 3 "~" H 3100 3200 50  0001 C CNN
-	1    3100 3200
+P 3075 2575
+F 0 "C206" H 3190 2621 50  0000 L CNN
+F 1 "0.1uF" H 3190 2530 50  0000 L CNN
+F 2 "Capacitor_SMD:C_0805_2012Metric" H 3113 2425 50  0001 C CNN
+F 3 "~" H 3075 2575 50  0001 C CNN
+	1    3075 2575
 	-1   0    0    -1
 $EndComp
 Wire Wire Line
-	4400 3000 3350 3000
-Wire Wire Line
-	3100 3000 3100 3050
+	4375 2375 3325 2375
+Wire Wire Line
+	3075 2375 3075 2425
 $Comp
 L Device:C C208
 U 1 1 61CDD207
-P 3350 3200
-F 0 "C208" H 3400 3300 50  0000 L CNN
-F 1 "1.0uF" H 3350 3100 50  0000 L CNN
-F 2 "Capacitor_SMD:C_0805_2012Metric" H 3388 3050 50  0001 C CNN
-F 3 "~" H 3350 3200 50  0001 C CNN
-	1    3350 3200
+P 3325 2575
+F 0 "C208" H 3375 2675 50  0000 L CNN
+F 1 "1.0uF" H 3325 2475 50  0000 L CNN
+F 2 "Capacitor_SMD:C_0805_2012Metric" H 3363 2425 50  0001 C CNN
+F 3 "~" H 3325 2575 50  0001 C CNN
+	1    3325 2575
 	-1   0    0    -1
 $EndComp
 Wire Wire Line
-	3100 3350 3100 3400
-Wire Wire Line
-	3100 3400 3350 3400
-Wire Wire Line
-	3350 3400 3350 3350
-Connection ~ 3100 3400
-Wire Wire Line
-	3100 3400 3100 3450
-Wire Wire Line
-	3350 3050 3350 3000
-Connection ~ 3350 3000
-Wire Wire Line
-	3350 3000 3100 3000
+	3075 2725 3075 2775
+Wire Wire Line
+	3075 2775 3325 2775
+Wire Wire Line
+	3325 2775 3325 2725
+Connection ~ 3075 2775
+Wire Wire Line
+	3075 2775 3075 2825
+Wire Wire Line
+	3325 2425 3325 2375
+Connection ~ 3325 2375
+Wire Wire Line
+	3325 2375 3075 2375
 Text GLabel 5100 4250 2    50   Input ~ 0
 DIN_MOSI_PI
@@
 SCLK_CLK_PI
 Wire Wire Line
-	2900 3000 3100 3000
-Connection ~ 3100 3000
+	2875 2375 3075 2375
+Connection ~ 3075 2375
 Wire Wire Line
 	2900 4150 3100 4150
@@
 Text GLabel 3100 4600 3    50   Input ~ 0
 AGND
-Text GLabel 3100 3450 3    50   Input ~ 0
+Text GLabel 3075 2825 3    50   Input ~ 0
 AGND
 $Comp
@@
 L power:+5V #PWR0143
 U 1 1 62012A20
-P 2900 2950
-F 0 "#PWR0143" H 2900 2800 50  0001 C CNN
-F 1 "+5V" H 2915 3123 50  0000 C CNN
-F 2 "" H 2900 2950 50  0001 C CNN
-F 3 "" H 2900 2950 50  0001 C CNN
-	1    2900 2950
+P 2875 2325
+F 0 "#PWR0143" H 2875 2175 50  0001 C CNN
+F 1 "+5V" H 2890 2498 50  0000 C CNN
+F 2 "" H 2875 2325 50  0001 C CNN
+F 3 "" H 2875 2325 50  0001 C CNN
+	1    2875 2325
 	1    0    0    -1
 $EndComp
@@
 $EndComp
 Wire Wire Line
-	2900 2950 2900 3000
+	2875 2325 2875 2375
 Wire Wire Line
 	2900 4100 2900 4150
@@
 NoConn ~ 8500 4675
 NoConn ~ 8500 4775
-Text GLabel 5100 3000 2    50   BiDi ~ 0
+Text GLabel 5075 2375 2    50   BiDi ~ 0
 DOUT_MISO_PI
 Text GLabel 5100 4150 2    50   BiDi ~ 0
@@
 L power:+3.3V #PWR0146
 U 1 1 62C64A47
-P 6100 3200
-F 0 "#PWR0146" H 6100 3050 50  0001 C CNN
-F 1 "+3.3V" H 6115 3373 50  0000 C CNN
-F 2 "" H 6100 3200 50  0001 C CNN
-F 3 "" H 6100 3200 50  0001 C CNN
-	1    6100 3200
+P 6075 2575
+F 0 "#PWR0146" H 6075 2425 50  0001 C CNN
+F 1 "+3.3V" H 6090 2748 50  0000 C CNN
+F 2 "" H 6075 2575 50  0001 C CNN
+F 3 "" H 6075 2575 50  0001 C CNN
+	1    6075 2575
 	1    0    0    -1
 $EndComp
@@
 Wire Wire Line
 	8000 3675 7325 3675
-Text HLabel 4400 3200 0    50   Input ~ 0
+Text HLabel 4375 2575 0    50   Input ~ 0
 OUT_AMP_1
-Text HLabel 4400 3300 0    50   Input ~ 0
+Text HLabel 4375 2675 0    50   Input ~ 0
 OUT_AMP_2
-Text HLabel 4400 3400 0    50   Input ~ 0
+Text HLabel 4375 2775 0    50   Input ~ 0
 OUT_AMP_3
-Text HLabel 4400 3500 0    50   Input ~ 0
+Text HLabel 4375 2875 0    50   Input ~ 0
 OUT_AMP_4
-Text HLabel 4400 3600 0    50   Input ~ 0
+Text HLabel 4375 2975 0    50   Input ~ 0
 OUT_AMP_5
-Text HLabel 5100 3600 2    50   Input ~ 0
+Text HLabel 5075 2975 2    50   Input ~ 0
 OUT_AMP_6
-Text HLabel 5100 3500 2    50   Input ~ 0
+Text HLabel 5075 2875 2    50   Input ~ 0
 OUT_AMP_7
-Text HLabel 5100 3400 2    50   Input ~ 0
+Text HLabel 5075 2775 2    50   Input ~ 0
 OUT_AMP_8
 Text HLabel 4400 4350 0    50   Input ~ 0
@@
 L emg-filter:ADC108S102 U43
 U 1 1 61EDDCFE
-P 4750 3250
-F 0 "U43" H 4750 3825 50  0000 C CNN
-F 1 "ADC108S102" H 4750 3734 50  0000 C CNN
-F 2 "Package_SO:TSSOP-16_4.4x5mm_P0.65mm" H 4750 3775 50  0001 C CNN
-F 3 "https://www.ti.com/lit/ds/symlink/adc108s102.pdf" H 4750 3775 50  0001 C CNN
-	1    4750 3250
-	1    0    0    -1
-$EndComp
+P 4725 2625
+F 0 "U43" H 4725 3200 50  0000 C CNN
+F 1 "ADC108S102" H 4725 3109 50  0000 C CNN
+F 2 "Package_SO:TSSOP-16_4.4x5mm_P0.65mm" H 4725 3150 50  0001 C CNN
+F 3 "https://www.ti.com/lit/ds/symlink/adc108s102.pdf" H 4725 3150 50  0001 C CNN
+	1    4725 2625
+	1    0    0    -1
+$EndComp
