File: hardware/kicad/emg-filter/bandpass.sch (KiCad schematic (older format))
At the start: 72 parts, among them U1 LM4565, U2 LM4565, U3 LM4565, U4 LM4565, U5 LM4565, U6 LM4565, U7 LM4565, U8 LM4565

Commit message: annotation
Parts:
- renumbered C1 to C19, C2 to C20, C3 to C21, C4 to C22, C5 to C23, C6 to C24, C7 to C25, C8 to C26, C9 to C27, C10 to C28, C11 to C29, C12 to C30, C13 to C31, C14 to C32, C15 to C33, C16 to C34, C17 to C35, C18 to C36, C19 to C37, C20 to C38, C21 to C39, C22 to C40, C23 to C41, C24 to C42, C25 to C43, C26 to C44, C27 to C45, C28 to C46, C29 to C47, C30 to C48, C31 to C49, C32 to C50, R1 to R43, R2 to R44, R3 to R45, R4 to R46, R5 to R47, R6 to R48, R7 to R49, R8 to R50, R9 to R51, R10 to R52, R11 to R53, R12 to R54, R13 to R55, R14 to R56, R15 to R57, R16 to R58, R17 to R59, R18 to R60, R19 to R61, R20 to R62, R21 to R63, R22 to R64, R23 to R65, R24 to R66, R25 to R67, R26 to R68, R27 to R69, R28 to R70, R29 to R71, R30 to R72, R31 to R73, R32 to R74, U1 to U12, U2 to U13, U3 to U14, U4 to U15, U5 to U16, U6 to U17, U7 to U18, U8 to U19

Commit message: linked stages by renaming labels
Connections:
- net INPUT_10_BANDPASS renamed INA_BP_10
- net INPUT_11_BANDPASS renamed INA_BP_11
- net INPUT_12_BANDPASS renamed INA_BP_12
- net INPUT_13_BANDPASS renamed INA_BP_13
- net INPUT_14_BANDPASS renamed INA_BP_14
- net INPUT_15_BANDPASS renamed INA_BP_15
- net INPUT_16_BANDPASS renamed INA_BP_16
- net INPUT_1_BANDPASS renamed INA_BP_1
- net INPUT_2_BANDPASS renamed INA_BP_2
- net INPUT_3_BANDPASS renamed INA_BP_3
- net INPUT_4_BANDPASS renamed INA_BP_4
- net INPUT_5_BANDPASS renamed INA_BP_5
- net INPUT_6_BANDPASS renamed INA_BP_6
- net INPUT_7_BANDPASS renamed INA_BP_7
- net INPUT_8_BANDPASS renamed INA_BP_8
- net INPUT_9_BANDPASS renamed INA_BP_9
- net OUTPUT_10_BANDPASS renamed BP_NOTCH_10
- net OUTPUT_11_BANDPASS renamed BP_NOTCH_11
- net OUTPUT_12_BANDPASS renamed BP_NOTCH_12
- net OUTPUT_13_BANDPASS renamed BP_NOTCH_13
- net OUTPUT_14_BANDPASS renamed BP_NOTCH_14
- net OUTPUT_15_BANDPASS renamed BP_NOTCH_15
- net OUTPUT_16_BANDPASS renamed BP_NOTCH_16
- net OUTPUT_1_BANDPASS renamed BP_NOTCH_1
- net OUTPUT_2_BANDPASS renamed BP_NOTCH_2
- net OUTPUT_3_BANDPASS renamed BP_NOTCH_3
- net OUTPUT_4_BANDPASS renamed BP_NOTCH_4
- net OUTPUT_5_BANDPASS renamed BP_NOTCH_5
- net OUTPUT_6_BANDPASS renamed BP_NOTCH_6
- net OUTPUT_7_BANDPASS renamed BP_NOTCH_7
- net OUTPUT_8_BANDPASS renamed BP_NOTCH_8
- net OUTPUT_9_BANDPASS renamed BP_NOTCH_9
Changed lines of the file:
@@
 $Descr A4 11693 8268
 encoding utf-8
-Sheet 1 10
+Sheet 4 10
 Title ""
 Date ""
@@
 	3450 6550 3500 6550
 Connection ~ 3450 6550
-Text GLabel 1300 1700 0    50   Input ~ 0
-INPUT_1_BANDPASS
-Text GLabel 1300 1950 0    50   Input ~ 0
-INPUT_2_BANDPASS
-Text GLabel 1300 4000 0    50   Input ~ 0
-INPUT_3_BANDPASS
-Text GLabel 1300 4250 0    50   Input ~ 0
-INPUT_4_BANDPASS
-Text GLabel 1300 6300 0    50   Input ~ 0
-INPUT_5_BANDPASS
-Text GLabel 1300 6550 0    50   Input ~ 0
-INPUT_6_BANDPASS
-Text GLabel 7050 1550 2    50   Input ~ 0
-INPUT_7_BANDPASS
-Text GLabel 7050 1800 2    50   Input ~ 0
-INPUT_8_BANDPASS
-Text GLabel 7050 3850 2    50   Input ~ 0
-INPUT_9_BANDPASS
-Text GLabel 7050 4100 2    50   Input ~ 0
-INPUT_10_BANDPASS
-Text GLabel 7050 6150 2    50   Input ~ 0
-INPUT_11_BANDPASS
-Text GLabel 7850 2650 0    50   Input ~ 0
-INPUT_13_BANDPASS
-Text GLabel 7850 2900 0    50   Input ~ 0
-INPUT_14_BANDPASS
-Text GLabel 7850 4950 0    50   Input ~ 0
-INPUT_15_BANDPASS
 $Comp
 L power:+5V #PWR042
@@
 	10000 5200 10050 5200
 Connection ~ 10000 5200
+Text GLabel 1300 1700 0    50   Input ~ 0
+INA_BP_1
+Text GLabel 1300 1950 0    50   Input ~ 0
+INA_BP_2
+Text GLabel 1300 4000 0    50   Input ~ 0
+INA_BP_3
+Text GLabel 1300 4250 0    50   Input ~ 0
+INA_BP_4
+Text GLabel 1300 6300 0    50   Input ~ 0
+INA_BP_5
+Text GLabel 1300 6550 0    50   Input ~ 0
+INA_BP_6
+Text GLabel 7050 1550 2    50   Input ~ 0
+INA_BP_7
+Text GLabel 7050 1800 2    50   Input ~ 0
+INA_BP_8
+Text GLabel 7050 3850 2    50   Input ~ 0
+INA_BP_9
+Text GLabel 7050 4100 2    50   Input ~ 0
+INA_BP_10
+Text GLabel 7050 6150 2    50   Input ~ 0
+INA_BP_11
+Text GLabel 7050 6400 2    50   Input ~ 0
+INA_BP_12
+Text GLabel 7850 2650 0    50   Input ~ 0
+INA_BP_13
+Text GLabel 7850 2900 0    50   Input ~ 0
+INA_BP_14
+Text GLabel 7850 4950 0    50   Input ~ 0
+INA_BP_15
 Text GLabel 7850 5200 0    50   Input ~ 0
-INPUT_16_BANDPASS
-Text GLabel 7050 6400 2    50   Input ~ 0
-INPUT_12_BANDPASS
+INA_BP_16
 Text GLabel 3500 1600 2    50   Input ~ 0
-OUTPUT_1_BANDPASS
+BP_NOTCH_1
 Text GLabel 3500 1950 2    50   Input ~ 0
-OUTPUT_2_BANDPASS
+BP_NOTCH_2
 Text GLabel 3500 3900 2    50   Input ~ 0
-OUTPUT_3_BANDPASS
+BP_NOTCH_3
 Text GLabel 3500 4250 2    50   Input ~ 0
-OUTPUT_4_BANDPASS
+BP_NOTCH_4
 Text GLabel 3500 6200 2    50   Input ~ 0
-OUTPUT_5_BANDPASS
+BP_NOTCH_5
 Text GLabel 3500 6550 2    50   Input ~ 0
-OUTPUT_6_BANDPASS
+BP_NOTCH_6
 Text GLabel 4850 1450 0    50   Input ~ 0
-OUTPUT_7_BANDPASS
+BP_NOTCH_7
 Text GLabel 4850 1800 0    50   Input ~ 0
-OUTPUT_8_BANDPASS
+BP_NOTCH_8
 Text GLabel 4850 3750 0    50   Input ~ 0
-OUTPUT_9_BANDPASS
+BP_NOTCH_9
 Text GLabel 4850 4100 0    50   Input ~ 0
-OUTPUT_10_BANDPASS
+BP_NOTCH_10
 Text GLabel 4850 6050 0    50   Input ~ 0
-OUTPUT_11_BANDPASS
+BP_NOTCH_11
 Text GLabel 4850 6400 0    50   Input ~ 0
-OUTPUT_12_BANDPASS
+BP_NOTCH_12
 Text GLabel 10050 2550 2    50   Input ~ 0
-OUTPUT_13_BANDPASS
+BP_NOTCH_13
 Text GLabel 10050 2900 2    50   Input ~ 0
-OUTPUT_14_BANDPASS
+BP_NOTCH_14
 Text GLabel 10050 4850 2    50   Input ~ 0
-OUTPUT_15_BANDPASS
+BP_NOTCH_15
 Text GLabel 10050 5200 2    50   Input ~ 0
-OUTPUT_16_BANDPASS
+BP_NOTCH_16
 $EndSCHEMATC

Commit message: notes from review with Dmitry, 01-06-22
Changed lines of the file:
@@
 Sheet 4 10
 Title ""
-Date ""
+Date "2022-01-06"
 Rev ""
 Comp ""
@@
 U 1 1 61CA77C9
 P 2850 750
-F 0 "C28" V 2900 600 50  0000 L CNN
+F 0 "C28" V 2900 550 50  0000 L CNN
 F 1 "2n" V 2800 600 50  0000 L CNN
 F 2 "" H 2888 600 50  0001 C CNN
@@
 U 1 1 62452189
 P 5500 2900
-F 0 "C32" V 5550 2750 50  0000 L CNN
+F 0 "C32" V 5550 2700 50  0000 L CNN
 F 1 "2n" V 5450 2750 50  0000 L CNN
 F 2 "" H 5538 2750 50  0001 C CNN
@@
 U 1 1 6245227F
 P 5500 600
-F 0 "C31" V 5550 450 50  0000 L CNN
+F 0 "C31" V 5550 350 50  0000 L CNN
 F 1 "2n" V 5450 450 50  0000 L CNN
 F 2 "" H 5538 450 50  0001 C CNN
@@
 U 1 1 62452295
 P 5550 2650
-F 0 "C34" V 5600 2500 50  0000 L CNN
+F 0 "C34" V 5600 2450 50  0000 L CNN
 F 1 "2n" V 5500 2500 50  0000 L CNN
 F 2 "" H 5588 2500 50  0001 C CNN
