File: hardware/kicad/emg-filter/bandpass.sch (KiCad schematic (older format))
At the start: 88 parts, among them U10 LM4565, U3 LM4565, U4 LM4565, U5 LM4565, U6 LM4565, U7 LM4565, U8 LM4565, U9 LM4565

Commit message: pcb
Parts:
- U10, U3, U4, U5, U6, U7, U8, U9: footprint (none) -> emg-filter:LM4565
Changed lines of the file:
@@
 F 0 "U3" H 2500 2800 50  0000 C CNN
 F 1 "LM4565" H 2850 2800 50  0000 C CNN
-F 2 "" H 3700 2500 50  0001 C CNN
+F 2 "emg-filter:LM4565" H 3700 2500 50  0001 C CNN
 F 3 "" H 3700 2500 50  0001 C CNN
 	1    2700 2500
@@
 F 0 "U4" H 2500 4450 50  0000 C CNN
 F 1 "LM4565" H 2850 4450 50  0000 C CNN
-F 2 "" H 3700 4150 50  0001 C CNN
+F 2 "emg-filter:LM4565" H 3700 4150 50  0001 C CNN
 F 3 "" H 3700 4150 50  0001 C CNN
 	1    2700 4150
@@
 F 0 "U5" H 2500 6100 50  0000 C CNN
 F 1 "LM4565" H 2850 6100 50  0000 C CNN
-F 2 "" H 3700 5800 50  0001 C CNN
+F 2 "emg-filter:LM4565" H 3700 5800 50  0001 C CNN
 F 3 "" H 3700 5800 50  0001 C CNN
 	1    2700 5800
@@
 F 0 "U6" H 5800 2800 50  0000 C CNN
 F 1 "LM4565" H 6150 2800 50  0000 C CNN
-F 2 "" H 7000 2500 50  0001 C CNN
+F 2 "emg-filter:LM4565" H 7000 2500 50  0001 C CNN
 F 3 "" H 7000 2500 50  0001 C CNN
 	1    6000 2500
@@
 F 0 "U7" H 5800 4450 50  0000 C CNN
 F 1 "LM4565" H 6150 4450 50  0000 C CNN
-F 2 "" H 7000 4150 50  0001 C CNN
+F 2 "emg-filter:LM4565" H 7000 4150 50  0001 C CNN
 F 3 "" H 7000 4150 50  0001 C CNN
 	1    6000 4150
@@
 F 0 "U8" H 5800 6100 50  0000 C CNN
 F 1 "LM4565" H 6150 6100 50  0000 C CNN
-F 2 "" H 7000 5800 50  0001 C CNN
+F 2 "emg-filter:LM4565" H 7000 5800 50  0001 C CNN
 F 3 "" H 7000 5800 50  0001 C CNN
 	1    6000 5800
@@
 F 0 "U9" H 9050 2800 50  0000 C CNN
 F 1 "LM4565" H 9400 2800 50  0000 C CNN
-F 2 "" H 10250 2500 50  0001 C CNN
+F 2 "emg-filter:LM4565" H 10250 2500 50  0001 C CNN
 F 3 "" H 10250 2500 50  0001 C CNN
 	1    9250 2500
@@
 F 0 "U10" H 9050 4450 50  0000 C CNN
 F 1 "LM4565" H 9400 4450 50  0000 C CNN
-F 2 "" H 10250 4150 50  0001 C CNN
+F 2 "emg-filter:LM4565" H 10250 4150 50  0001 C CNN
 F 3 "" H 10250 4150 50  0001 C CNN
 	1    9250 4150
