File: hardware/kicad/emg-filter/power.sch (KiCad schematic (older format))
At the start: 38 parts, among them U1 LM7805_TO220, U2 LM7905_TO220, U3 LM7805_TO220

Commit message: annotation
Parts:
- gave numbers to parts that had none: 33
- renumbered C1 to C3, U3 to U1, U1 to U2, U2 to U3

Commit message: diode and led values
Parts:
- D1, D2, D3: value D -> 1N4007
- D4, D5, D6: value LED -> LTST-C170TBKT
Other:
- note added: "Resistor direction?"
Changed lines of the file:
@@
-$EndComp
-$Comp
-L Device:D D1
-U 1 1 61C6D969
-P 4250 850
-F 0 "D1" H 4250 1067 50  0000 C CNN
-F 1 "D" H 4250 976 50  0000 C CNN
-F 2 "" H 4250 850 50  0001 C CNN
-F 3 "~" H 4250 850 50  0001 C CNN
-	1    4250 850
-	1    0    0    -1
 $EndComp
 $Comp
@@
 P 4250 4550
 F 0 "D3" H 4250 4650 50  0000 C CNN
-F 1 "D" H 4250 4750 50  0000 C CNN
+F 1 "1N4007" H 4250 4750 50  0000 C CNN
 F 2 "" H 4250 4550 50  0001 C CNN
 F 3 "~" H 4250 4550 50  0001 C CNN
@@
 P 6800 3100
 F 0 "D5" V 6839 2982 50  0000 R CNN
-F 1 "LED" V 6748 2982 50  0000 R CNN
+F 1 "LTST-C170TBKT" V 6748 2982 50  0000 R CNN
 F 2 "" H 6800 3100 50  0001 C CNN
 F 3 "~" H 6800 3100 50  0001 C CNN
@@
 P 6800 3700
 F 0 "D6" V 6839 3582 50  0000 R CNN
-F 1 "LED" V 6748 3582 50  0000 R CNN
+F 1 "LTST-C170TBKT" V 6748 3582 50  0000 R CNN
 F 2 "" H 6800 3700 50  0001 C CNN
 F 3 "~" H 6800 3700 50  0001 C CNN
@@
 	6300 4150 6300 3850
 Connection ~ 6300 3850
-Connection ~ 6800 2950
-Connection ~ 6800 4150
 $Comp
 L Device:C C6
@@
 P 6800 1400
 F 0 "D4" V 6839 1282 50  0000 R CNN
-F 1 "LED" V 6748 1282 50  0000 R CNN
+F 1 "LTST-C170TBKT" V 6748 1282 50  0000 R CNN
 F 2 "" H 6800 1400 50  0001 C CNN
 F 3 "~" H 6800 1400 50  0001 C CNN
@@
 	1    0    0    -1
 $EndComp
-Connection ~ 6800 1850
 Wire Wire Line
 	6300 1250 6300 1550
 Connection ~ 6300 1550
 Wire Wire Line
-	6800 1250 7300 1250
-Connection ~ 6800 1250
+	6800 1250 7700 1250
 Wire Wire Line
 	4650 1250 4900 1250
@@
 P 4250 2350
 F 0 "D2" H 4250 2567 50  0000 C CNN
-F 1 "D" H 4250 2476 50  0000 C CNN
+F 1 "1N4007" H 4250 2476 50  0000 C CNN
 F 2 "" H 4250 2350 50  0001 C CNN
 F 3 "~" H 4250 2350 50  0001 C CNN
@@
 Wire Wire Line
 	2800 3250 3200 3250
-Text GLabel 7300 1250 2    50   Input ~ 0
+Text GLabel 7700 1250 2    50   Input ~ 0
 +5V_PI
 Wire Wire Line
-	6800 3550 7300 3550
+	6800 3550 7700 3550
 $Comp
 L power:-5V #PWR011
 U 1 1 61D9BE69
-P 7300 4200
-F 0 "#PWR011" H 7300 4300 50  0001 C CNN
-F 1 "-5V" H 7315 4373 50  0000 C CNN
-F 2 "" H 7300 4200 50  0001 C CNN
-F 3 "" H 7300 4200 50  0001 C CNN
-	1    7300 4200
+P 7700 4200
+F 0 "#PWR011" H 7700 4300 50  0001 C CNN
+F 1 "-5V" H 7715 4373 50  0000 C CNN
+F 2 "" H 7700 4200 50  0001 C CNN
+F 3 "" H 7700 4200 50  0001 C CNN
+	1    7700 4200
 	-1   0    0    1
 $EndComp
@@
 L power:+5V #PWR09
 U 1 1 61DA16DE
-P 7300 2900
-F 0 "#PWR09" H 7300 2750 50  0001 C CNN
-F 1 "+5V" H 7315 3073 50  0000 C CNN
-F 2 "" H 7300 2900 50  0001 C CNN
-F 3 "" H 7300 2900 50  0001 C CNN
-	1    7300 2900
-	1    0    0    -1
-$EndComp
-Wire Wire Line
-	6800 2950 7300 2950
-Wire Wire Line
-	6800 4150 7300 4150
+P 7700 2900
+F 0 "#PWR09" H 7700 2750 50  0001 C CNN
+F 1 "+5V" H 7715 3073 50  0000 C CNN
+F 2 "" H 7700 2900 50  0001 C CNN
+F 3 "" H 7700 2900 50  0001 C CNN
+	1    7700 2900
+	1    0    0    -1
+$EndComp
+Wire Wire Line
+	6800 2950 7700 2950
+Wire Wire Line
+	6800 4150 7700 4150
 $Comp
 L power:GND #PWR010
 U 1 1 61D1A2AE
-P 7300 3600
-F 0 "#PWR010" H 7300 3350 50  0001 C CNN
-F 1 "GND" H 7305 3427 50  0000 C CNN
-F 2 "" H 7300 3600 50  0001 C CNN
-F 3 "" H 7300 3600 50  0001 C CNN
-	1    7300 3600
-	1    0    0    -1
-$EndComp
-Wire Wire Line
-	7300 3550 7300 3600
-Wire Wire Line
-	7300 4150 7300 4200
-Wire Wire Line
-	7300 2900 7300 2950
+P 7700 3600
+F 0 "#PWR010" H 7700 3350 50  0001 C CNN
+F 1 "GND" H 7705 3427 50  0000 C CNN
+F 2 "" H 7700 3600 50  0001 C CNN
+F 3 "" H 7700 3600 50  0001 C CNN
+	1    7700 3600
+	1    0    0    -1
+$EndComp
+Wire Wire Line
+	7700 3550 7700 3600
+Wire Wire Line
+	7700 4150 7700 4200
+Wire Wire Line
+	7700 2900 7700 2950
 $Comp
 L power:GND #PWR08
 U 1 1 61D34546
-P 7300 1900
-F 0 "#PWR08" H 7300 1650 50  0001 C CNN
-F 1 "GND" H 7305 1727 50  0000 C CNN
-F 2 "" H 7300 1900 50  0001 C CNN
-F 3 "" H 7300 1900 50  0001 C CNN
-	1    7300 1900
-	1    0    0    -1
-$EndComp
-Wire Wire Line
-	7300 1850 7300 1900
-Wire Wire Line
-	6800 1850 7300 1850
+P 7700 1900
+F 0 "#PWR08" H 7700 1650 50  0001 C CNN
+F 1 "GND" H 7705 1727 50  0000 C CNN
+F 2 "" H 7700 1900 50  0001 C CNN
+F 3 "" H 7700 1900 50  0001 C CNN
+	1    7700 1900
+	1    0    0    -1
+$EndComp
+Wire Wire Line
+	7700 1850 7700 1900
+Wire Wire Line
+	6800 1850 7700 1850
 Connection ~ 4250 1850
 Connection ~ 4550 1250
@@
 	1    0    0    -1
 $EndComp
+$Comp
+L Device:D D1
+U 1 1 61C6D969
+P 4250 850
+F 0 "D1" H 4250 1067 50  0000 C CNN
+F 1 "1N4007" H 4250 976 50  0000 C CNN
+F 2 "" H 4250 850 50  0001 C CNN
+F 3 "~" H 4250 850 50  0001 C CNN
+	1    4250 850
+	1    0    0    -1
+$EndComp
+Connection ~ 6800 1250
+Connection ~ 6800 1850
+Connection ~ 6800 2950
+Connection ~ 6800 4150
+Text Notes 4950 4050 0    50   ~ 0
+Resistor direction?
 $EndSCHEMATC

Commit message: notes from review with Dmitry, 01-06-22
Other:
- note added: "Checkout isolated Vreg isolate 24V from 5V (usually for low A) switching near bat with decoup caps\n"
- note added: "Use 2 batteries?\n"
Changed lines of the file:
@@
 Text Notes 4950 4050 0    50   ~ 0
 Resistor direction?
+Text Notes 4850 800  0    50   ~ 0
+Checkout isolated Vreg isolate 24V from 5V (usually for low A) switching near bat with decoup caps\n
+Text Notes 1550 2250 0    50   ~ 0
+Use 2 batteries?\n
 $EndSCHEMATC
