File: hardware/kicad/emg-filter/power.sch (KiCad schematic (older format))
At the start: 38 parts, among them U1 LM7805_TO220, U2 LM7805_TO220, U3 LM7905_TO220

Commit message: added cap bank for op-amp supply rails, removed pi power supply
Parts:
- removed C10: 0.1uF, symbol Device:C
- removed C13: 1uF, symbol Device:C
- removed C16: 0.01uF, symbol Device:C
- removed C6: 2200uF, symbol Device:C
- removed C7: 470uF, symbol Device:C
- removed D1: 1N4007, symbol Device:D
- removed D4: LTST-C170TBKT, symbol Device:LED
- removed R3: 10, symbol Device:R
- removed R5: 1k, symbol Device:R
- removed R8: 470, symbol Device:R
- removed U1: LM7805_TO220, Package_TO_SOT_THT:TO-220-3_Vertical, symbol Regulator_Linear:LM7805_TO220
- added C? (x96): 0.1uF, symbol Device:C
Connections:
- net labels removed: +5V_PI
- wire segments 95 -> 455
Other:
- note added: "Caps for op-amp supply rails, they need to be positioned as close as possible to the supply terminals on the PCB."
- note removed: "Diode direction?"
- note removed: "Resistor direction?"
- moved on the sheet: C1, C11, C12, C14, C15, C17, C18, C2, C3, C4, C5, C8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

Commit message: added pi gnd flag
Connections:
- net labels added: GND_PI
- wire segments 455 -> 456
Changed lines of the file:
@@
 Text Notes 1100 3725 0    50   ~ 0
 Caps for op-amp supply rails, they need to be positioned as close as possible to the supply terminals on the PCB.
+Text GLabel 7675 2000 2    50   Output ~ 0
+GND_PI
+Wire Wire Line
+	7600 2000 7675 2000
+Connection ~ 7600 2000
 $EndSCHEMATC

Commit message: Rectifier Fit on US letter format
Parts:
- gave numbers to parts that had none: 96
- renumbered C14 to C106, C15 to C107, C17 to C108, C18 to C109, C2 to C14, C3 to C27, C4 to C52, C5 to C53, C1 to C7, C8 to C84, C9 to C85, C11 to C92, C12 to C93, D2 to D1, D3 to D2, D5 to D3, D6 to D4, R4 to R3, R6 to R4, R7 to R5, R9 to R6, R10 to R7, U2 to U1, U3 to U2
