File: hardware/kicad/emg-filter/rectifier2.sch (KiCad schematic (older format))
At the start: 80 parts, among them U43 LM4565, U44 LM4565, U45 LM4565, U46 LM4565, U47 LM4565, U48 LM4565, U49 LM4565, U50 LM4565

Commit message: footprint association
Parts:
- C190, C191, C192, C193, C194, C195, C196, C197, C198, C199, C200, C201, C202, C203, C204, C205: footprint (none) -> Capacitor_SMD:C_0805_2012Metric
- D21, D22, D23, D24, D25, D26, D27, D28, D29, D30, D31, D32, D33, D34, D35, D36: footprint (none) -> Diode_SMD:D_SOD-323
- R160: renamed from R192; footprint (none) -> Resistor_SMD:R_0805_2012Metric
- R161: renamed from R193; footprint (none) -> Resistor_SMD:R_0805_2012Metric
- R162: renamed from R194; footprint (none) -> Resistor_SMD:R_0805_2012Metric
- R163: renamed from R195; footprint (none) -> Resistor_SMD:R_0805_2012Metric
- R164: renamed from R196; footprint (none) -> Resistor_SMD:R_0805_2012Metric
- R165: renamed from R197; footprint (none) -> Resistor_SMD:R_0805_2012Metric
- R166: renamed from R198; footprint (none) -> Resistor_SMD:R_0805_2012Metric
- R167: renamed from R199; footprint (none) -> Resistor_SMD:R_0805_2012Metric
- R168: renamed from R200; footprint (none) -> Resistor_SMD:R_0805_2012Metric
- R169: renamed from R201; footprint (none) -> Resistor_SMD:R_0805_2012Metric
- R170: renamed from R202; footprint (none) -> Resistor_SMD:R_0805_2012Metric
- R171: renamed from R203; footprint (none) -> Resistor_SMD:R_0805_2012Metric
- R172: renamed from R204; footprint (none) -> Resistor_SMD:R_0805_2012Metric
- R173: renamed from R205; footprint (none) -> Resistor_SMD:R_0805_2012Metric
- R174: renamed from R206; footprint (none) -> Resistor_SMD:R_0805_2012Metric
- R175: renamed from R207; footprint (none) -> Resistor_SMD:R_0805_2012Metric
- R176: renamed from R208; footprint (none) -> Resistor_SMD:R_0805_2012Metric
- R177: renamed from R209; footprint (none) -> Resistor_SMD:R_0805_2012Metric
- R178: renamed from R210; footprint (none) -> Resistor_SMD:R_0805_2012Metric
- R179: renamed from R211; footprint (none) -> Resistor_SMD:R_0805_2012Metric
- R180: renamed from R212; footprint (none) -> Resistor_SMD:R_0805_2012Metric
- R181: renamed from R213; footprint (none) -> Resistor_SMD:R_0805_2012Metric
- R182: renamed from R214; footprint (none) -> Resistor_SMD:R_0805_2012Metric
- R183: renamed from R215; footprint (none) -> Resistor_SMD:R_0805_2012Metric
- R184: renamed from R216; footprint (none) -> Resistor_SMD:R_0805_2012Metric
- R185: renamed from R217; footprint (none) -> Resistor_SMD:R_0805_2012Metric
- R186: renamed from R218; footprint (none) -> Resistor_SMD:R_0805_2012Metric
- R187: renamed from R219; footprint (none) -> Resistor_SMD:R_0805_2012Metric
- R188: renamed from R220; footprint (none) -> Resistor_SMD:R_0805_2012Metric
- R189: renamed from R221; footprint (none) -> Resistor_SMD:R_0805_2012Metric
- R190: renamed from R222; footprint (none) -> Resistor_SMD:R_0805_2012Metric
- R191: renamed from R223; footprint (none) -> Resistor_SMD:R_0805_2012Metric
- R192: renamed from R224; footprint (none) -> Resistor_SMD:R_0805_2012Metric
- R193: renamed from R225; footprint (none) -> Resistor_SMD:R_0805_2012Metric
- R194: renamed from R226; footprint (none) -> Resistor_SMD:R_0805_2012Metric
- R195: renamed from R227; footprint (none) -> Resistor_SMD:R_0805_2012Metric
- R196: renamed from R228; footprint (none) -> Resistor_SMD:R_0805_2012Metric
- R197: renamed from R229; footprint (none) -> Resistor_SMD:R_0805_2012Metric
- R198: renamed from R230; footprint (none) -> Resistor_SMD:R_0805_2012Metric
- R199: renamed from R231; footprint (none) -> Resistor_SMD:R_0805_2012Metric
- renumbered U43 to U35, U44 to U36, U45 to U37, U46 to U38, U47 to U39, U48 to U40, U49 to U41, U50 to U42
