File: hardware/kicad/emg-filter/rectifier2.sch (KiCad schematic (older format))
At the start: 80 parts, among them U35 LM4565, U36 LM4565, U37 LM4565, U38 LM4565, U39 LM4565, U40 LM4565, U41 LM4565, U42 LM4565

Commit message: Solving Stuff for Free
Parts:
- renumbered R160 to R192, R161 to R193, R162 to R194, R163 to R195, R164 to R196, R165 to R197, R166 to R198, R167 to R199, R168 to R200, R169 to R201, R170 to R202, R171 to R203, R172 to R204, R173 to R205, R174 to R206, R175 to R207, R176 to R208, R177 to R209, R178 to R210, R179 to R211, R180 to R212, R181 to R213, R182 to R214, R183 to R215, R184 to R216, R185 to R217, R186 to R218, R187 to R219, R188 to R220, R189 to R221, R190 to R222, R191 to R223, R192 to R224, R193 to R225, R194 to R226, R195 to R227, R196 to R228, R197 to R229, R198 to R230, R199 to R231

Commit message: pcb
Parts:
- U35, U36, U37, U38, U39, U40, U41, U42: footprint (none) -> emg-filter:LM4565
Changed lines of the file:
@@
 F 0 "U42" H 5350 6475 50  0000 C CNN
 F 1 "LM4565" H 5300 7125 50  0000 C CNN
-F 2 "" H 6150 6825 50  0001 C CNN
+F 2 "emg-filter:LM4565" H 6150 6825 50  0001 C CNN
 F 3 "" H 6150 6825 50  0001 C CNN
 	1    5150 6825
@@
 F 0 "U41" H 5350 4650 50  0000 C CNN
 F 1 "LM4565" H 5300 5300 50  0000 C CNN
-F 2 "" H 6150 5000 50  0001 C CNN
+F 2 "emg-filter:LM4565" H 6150 5000 50  0001 C CNN
 F 3 "" H 6150 5000 50  0001 C CNN
 	1    5150 5000
@@
 F 0 "U40" H 5350 2850 50  0000 C CNN
 F 1 "LM4565" H 5300 3500 50  0000 C CNN
-F 2 "" H 6150 3200 50  0001 C CNN
+F 2 "emg-filter:LM4565" H 6150 3200 50  0001 C CNN
 F 3 "" H 6150 3200 50  0001 C CNN
 	1    5150 3200
@@
 F 0 "U39" H 5350 1000 50  0000 C CNN
 F 1 "LM4565" H 5300 1650 50  0000 C CNN
-F 2 "" H 6150 1350 50  0001 C CNN
+F 2 "emg-filter:LM4565" H 6150 1350 50  0001 C CNN
 F 3 "" H 6150 1350 50  0001 C CNN
 	1    5150 1350
@@
 F 0 "U38" H 2450 6475 50  0000 C CNN
 F 1 "LM4565" H 2400 7125 50  0000 C CNN
-F 2 "" H 3250 6825 50  0001 C CNN
+F 2 "emg-filter:LM4565" H 3250 6825 50  0001 C CNN
 F 3 "" H 3250 6825 50  0001 C CNN
 	1    2250 6825
@@
 F 0 "U37" H 2450 4650 50  0000 C CNN
 F 1 "LM4565" H 2400 5300 50  0000 C CNN
-F 2 "" H 3250 5000 50  0001 C CNN
+F 2 "emg-filter:LM4565" H 3250 5000 50  0001 C CNN
 F 3 "" H 3250 5000 50  0001 C CNN
 	1    2250 5000
@@
 F 0 "U36" H 2450 2850 50  0000 C CNN
 F 1 "LM4565" H 2400 3500 50  0000 C CNN
-F 2 "" H 3250 3200 50  0001 C CNN
+F 2 "emg-filter:LM4565" H 3250 3200 50  0001 C CNN
 F 3 "" H 3250 3200 50  0001 C CNN
 	1    2250 3200
@@
 F 0 "U35" H 2450 1000 50  0000 C CNN
 F 1 "LM4565" H 2400 1650 50  0000 C CNN
-F 2 "" H 3250 1350 50  0001 C CNN
+F 2 "emg-filter:LM4565" H 3250 1350 50  0001 C CNN
 F 3 "" H 3250 1350 50  0001 C CNN
 	1    2250 1350

Commit message: Fix Rectifier
Connections:
- wire segments 324 -> 320
Changed lines of the file:
@@
 Comment4 ""
 $EndDescr
-Wire Wire Line
-	1750 3150 1750 3300
-Wire Wire Line
-	1750 3150 1850 3150
-Connection ~ 1750 3150
-Wire Wire Line
-	1750 1300 1750 1450
-Wire Wire Line
-	1750 1300 1850 1300
-Connection ~ 1750 1300
 Connection ~ 5600 7025
 Wire Wire Line
@@
 AR Path="/61C38746/6BB1123B/61E2804F" Ref="C?"  Part="1"
 AR Path="/61C38746/61DCD9A2/61E2804F" Ref="C201"  Part="1"
-F 0 "C201" V 4850 6325 50  0000 C CNN
+F 0 "C201" V 4825 6275 50  0000 C CNN
 F 1 "0.1u" V 4750 6425 50  0000 C CNN
 F 2 "Capacitor_SMD:C_0805_2012Metric" H 4938 6275 50  0001 C CNN
@@
 AR Path="/61C38746/6BB1123B/61E2805D" Ref="C?"  Part="1"
 AR Path="/61C38746/61DCD9A2/61E2805D" Ref="C205"  Part="1"
-F 0 "C205" V 4900 7175 50  0000 C CNN
+F 0 "C205" V 4875 7125 50  0000 C CNN
 F 1 "0.1u" V 4800 7275 50  0000 C CNN
 F 2 "Capacitor_SMD:C_0805_2012Metric" H 4988 7125 50  0001 C CNN
@@
 AR Path="/61C38746/6BB1123B/61E280D4" Ref="C?"  Part="1"
 AR Path="/61C38746/61DCD9A2/61E280D4" Ref="C200"  Part="1"
-F 0 "C200" V 4850 4500 50  0000 C CNN
+F 0 "C200" V 4850 4450 50  0000 C CNN
 F 1 "0.1u" V 4750 4600 50  0000 C CNN
 F 2 "Capacitor_SMD:C_0805_2012Metric" H 4938 4450 50  0001 C CNN
@@
 AR Path="/61C38746/6BB1123B/61E280E2" Ref="C?"  Part="1"
 AR Path="/61C38746/61DCD9A2/61E280E2" Ref="C204"  Part="1"
-F 0 "C204" V 4900 5350 50  0000 C CNN
+F 0 "C204" V 4900 5300 50  0000 C CNN
 F 1 "0.1u" V 4800 5450 50  0000 C CNN
 F 2 "Capacitor_SMD:C_0805_2012Metric" H 4988 5300 50  0001 C CNN
@@
 AR Path="/61C38746/6BB1123B/61E28159" Ref="C?"  Part="1"
 AR Path="/61C38746/61DCD9A2/61E28159" Ref="C199"  Part="1"
-F 0 "C199" V 4850 2700 50  0000 C CNN
+F 0 "C199" V 4850 2650 50  0000 C CNN
 F 1 "0.1u" V 4750 2800 50  0000 C CNN
 F 2 "Capacitor_SMD:C_0805_2012Metric" H 4938 2650 50  0001 C CNN
@@
 AR Path="/61C38746/6BB1123B/61E28167" Ref="C?"  Part="1"
 AR Path="/61C38746/61DCD9A2/61E28167" Ref="C203"  Part="1"
-F 0 "C203" V 4900 3550 50  0000 C CNN
+F 0 "C203" V 4900 3500 50  0000 C CNN
 F 1 "0.1u" V 4800 3650 50  0000 C CNN
 F 2 "Capacitor_SMD:C_0805_2012Metric" H 4988 3500 50  0001 C CNN
@@
 AR Path="/61C38746/6BB1123B/61E281DE" Ref="C?"  Part="1"
 AR Path="/61C38746/61DCD9A2/61E281DE" Ref="C198"  Part="1"
-F 0 "C198" V 4850 850 50  0000 C CNN
+F 0 "C198" V 4850 800 50  0000 C CNN
 F 1 "0.1u" V 4750 950 50  0000 C CNN
 F 2 "Capacitor_SMD:C_0805_2012Metric" H 4938 800 50  0001 C CNN
@@
 AR Path="/61C38746/6BB1123B/61E281EC" Ref="C?"  Part="1"
 AR Path="/61C38746/61DCD9A2/61E281EC" Ref="C202"  Part="1"
-F 0 "C202" V 4900 1700 50  0000 C CNN
+F 0 "C202" V 4900 1650 50  0000 C CNN
 F 1 "0.1u" V 4800 1800 50  0000 C CNN
 F 2 "Capacitor_SMD:C_0805_2012Metric" H 4988 1650 50  0001 C CNN
@@
 AR Path="/61C38746/6BB1123B/61E28263" Ref="C?"  Part="1"
 AR Path="/61C38746/61DCD9A2/61E28263" Ref="C193"  Part="1"
-F 0 "C193" V 1950 6325 50  0000 C CNN
+F 0 "C193" V 1925 6275 50  0000 C CNN
 F 1 "0.1u" V 1850 6425 50  0000 C CNN
 F 2 "Capacitor_SMD:C_0805_2012Metric" H 2038 6275 50  0001 C CNN
@@
 AR Path="/61C38746/6BB1123B/61E28271" Ref="C?"  Part="1"
 AR Path="/61C38746/61DCD9A2/61E28271" Ref="C197"  Part="1"
-F 0 "C197" V 2000 7175 50  0000 C CNN
+F 0 "C197" V 1975 7125 50  0000 C CNN
 F 1 "0.1u" V 1900 7275 50  0000 C CNN
 F 2 "Capacitor_SMD:C_0805_2012Metric" H 2088 7125 50  0001 C CNN
@@
 AR Path="/61C38746/6BB1123B/61E282E8" Ref="C?"  Part="1"
 AR Path="/61C38746/61DCD9A2/61E282E8" Ref="C192"  Part="1"
-F 0 "C192" V 1950 4500 50  0000 C CNN
+F 0 "C192" V 1950 4450 50  0000 C CNN
 F 1 "0.1u" V 1850 4600 50  0000 C CNN
 F 2 "Capacitor_SMD:C_0805_2012Metric" H 2038 4450 50  0001 C CNN
@@
 AR Path="/61C38746/6BB1123B/61E282F6" Ref="C?"  Part="1"
 AR Path="/61C38746/61DCD9A2/61E282F6" Ref="C196"  Part="1"
-F 0 "C196" V 2000 5350 50  0000 C CNN
+F 0 "C196" V 2000 5300 50  0000 C CNN
 F 1 "0.1u" V 1900 5450 50  0000 C CNN
 F 2 "Capacitor_SMD:C_0805_2012Metric" H 2088 5300 50  0001 C CNN
@@
 AR Path="/61C38746/6BB1123B/61E2836D" Ref="C?"  Part="1"
 AR Path="/61C38746/61DCD9A2/61E2836D" Ref="C191"  Part="1"
-F 0 "C191" V 1950 2700 50  0000 C CNN
+F 0 "C191" V 1950 2650 50  0000 C CNN
 F 1 "0.1u" V 1850 2800 50  0000 C CNN
 F 2 "Capacitor_SMD:C_0805_2012Metric" H 2038 2650 50  0001 C CNN
@@
 AR Path="/61C38746/6BB1123B/61E2837B" Ref="C?"  Part="1"
 AR Path="/61C38746/61DCD9A2/61E2837B" Ref="C195"  Part="1"
-F 0 "C195" V 2000 3550 50  0000 C CNN
+F 0 "C195" V 2000 3500 50  0000 C CNN
 F 1 "0.1u" V 1900 3650 50  0000 C CNN
 F 2 "Capacitor_SMD:C_0805_2012Metric" H 2088 3500 50  0001 C CNN
@@
 	1750 3300 1850 3300
 Wire Wire Line
-	1750 3050 1750 3150
-Wire Wire Line
 	1850 3050 1750 3050
 Wire Wire Line
@@
 Wire Wire Line
 	1600 3550 1600 3400
-Wire Wire Line
-	1600 3150 1750 3150
 Wire Wire Line
 	1600 2950 1600 3150
@@
 AR Path="/61C38746/6BB1123B/61E283F2" Ref="C?"  Part="1"
 AR Path="/61C38746/61DCD9A2/61E283F2" Ref="C190"  Part="1"
-F 0 "C190" V 1950 850 50  0000 C CNN
+F 0 "C190" V 1950 800 50  0000 C CNN
 F 1 "0.1u" V 1850 950 50  0000 C CNN
 F 2 "Capacitor_SMD:C_0805_2012Metric" H 2038 800 50  0001 C CNN
@@
 AR Path="/61C38746/6BB1123B/61E28400" Ref="C?"  Part="1"
 AR Path="/61C38746/61DCD9A2/61E28400" Ref="C194"  Part="1"
-F 0 "C194" V 2000 1700 50  0000 C CNN
+F 0 "C194" V 2000 1650 50  0000 C CNN
 F 1 "0.1u" V 1900 1800 50  0000 C CNN
 F 2 "Capacitor_SMD:C_0805_2012Metric" H 2088 1650 50  0001 C CNN
@@
 	1750 1450 1850 1450
 Wire Wire Line
-	1750 1200 1750 1300
-Wire Wire Line
 	1850 1200 1750 1200
 Wire Wire Line
@@
 Wire Wire Line
 	1600 1700 1600 1550
-Wire Wire Line
-	1600 1300 1750 1300
 Wire Wire Line
 	1600 1100 1600 1300
@@
 Text GLabel 5700 7025 2    50   Input ~ 0
 RECT_AMP_16
+Wire Wire Line
+	1750 1200 1750 1450
+Wire Wire Line
+	1600 1300 1850 1300
+Wire Wire Line
+	1750 3050 1750 3300
+Wire Wire Line
+	1600 3150 1850 3150
 $EndSCHEMATC
