File: hardware/kicad/emg-filter/emg-connectors.sch (KiCad schematic (older format))
At the start: 78 parts, among them J10 Conn_01x02, J11 Conn_01x02, J12 Conn_01x02, J13 Conn_01x02, J14 Conn_01x02, J15 Conn_01x02, J16 Conn_01x02, J17 Conn_01x02, J18 Conn_01x02, J19 Conn_01x02, J20 Conn_01x02, J21 Conn_01x02, J22 Conn_01x02, J23 Conn_01x02, J24 Conn_01x02, J25 Conn_01x02, J26 Conn_01x02, J27 Conn_01x02, J28 Conn_01x02, J29 Conn_01x02, J30 Conn_01x02, J31 Conn_01x02, J32 Conn_01x02, J33 Conn_01x02, J34 Conn_01x02, J35 Conn_01x02, J36 Conn_01x02, J37 Conn_01x02, J38 Conn_01x02, J39 Conn_01x02, J4 Conn_01x02, J40 Conn_01x02, J41 Conn_01x02, J42 Conn_01x02, J43 Conn_01x02, J44 Conn_01x02, J45 Conn_01x02, J46 Conn_01x02, J47 Conn_01x02, J48 Conn_01x02, J49 Conn_01x02, J5 Conn_01x02, J50 Conn_01x02, J51 Conn_01x02, J6 Conn_01x02, J7 Conn_01x02, J8 Conn_01x02, J9 Conn_01x02

Commit message: Connectors done, but annotation bad
work will be transfer to another project
Parts:
- removed J10, J11, J12, J13, J14, J15, J17, J19, J21, J23, J25, J27, J28, J29, J30, J31, J32, J33, J34, J35, J36, J37, J38, J39, J4, J40, J41, J42, J43, J44, J45, J46, J47, J48, J49, J5, J50, J51, J6, J7, J8, J9: Conn_01x02, emg-filter:EMG_CONN_01x02, symbol Connector_Generic:Conn_01x02
- removed R10, R11, R12, R13, R14, R15, R16, R17, R18, R19, R20, R21, R22, R23, R24, R25, R26, R27, R28, R29, R30, R31, R32, R33, R34, R35, R36, R37, R8, R9: 0, Resistor_SMD:R_0805_2012Metric, symbol Device:R
- added J? (x2): Conn_01x02, symbol Connector_Generic:Conn_01x02
Connections:
- net labels added: REFA, REFB, VINA, VINB
- net labels removed: +VINA_1, +VINA_11, +VINA_13, +VINA_15, +VINA_5, +VINA_7, +VINA_9, +VINB_10, +VINB_12, +VINB_14, +VINB_16, +VINB_2, +VINB_6, +VINB_8, -VINA_1, -VINA_11, -VINA_13, -VINA_15, -VINA_5, -VINA_7, -VINA_9, -VINB_10, -VINB_12, -VINB_14, -VINB_16, -VINB_2, -VINB_6, -VINB_8, REFA_1, REFA_11, REFA_13, REFA_15, REFA_5, REFA_7, REFA_9, REFB_10, REFB_12, REFB_14, REFB_16, REFB_2, REFB_6, REFB_8
- wire segments 252 -> 33
Other:
- note added: "motherboard jumper connectors\n"

Commit message: saved files
Parts:
- gave numbers to parts that had none: 2
Connections:
- net labels added: +VINA, +VINB, -VINA, -VINB, REFA_JUMPER, REFB_JUMPER, VINA_JUMPER, VINB_JUMPER
- net labels removed: +VINA_3, +VINB_4, -VINA_3, -VINB_4, REFA_3, REFB_4, VINA, VINB
Other:
- note added: "jumper header\n"
- note added: "motherboard jumper headers"
- note added: "motherboard jumper headers\n"
- note removed: "motherboard jumper connectors\n"
Changed lines of the file:
@@
 $Descr USLetter 11000 8500
 encoding utf-8
-Sheet 2 3
+Sheet 3 3
 Title "EMG Filter for Prosthetic Limb Control System"
 Date "2022-01-07"
@@
 Wire Wire Line
 	4850 3475 4850 3625
-Text GLabel 4050 2675 1    50   Input ~ 0
--VINA_3
-Text GLabel 3250 2675 1    50   Input ~ 0
-+VINA_3
-Text GLabel 3650 2025 1    50   Input ~ 0
-REFA_3
-Text GLabel 4850 2025 1    50   Input ~ 0
-REFB_4
 $Comp
 L Connector_Generic:Conn_01x02 J?
@@
 	-1   0    0    1
 $EndComp
-Text GLabel 5250 2675 1    50   Input ~ 0
--VINB_4
-Text GLabel 4450 2675 1    50   Input ~ 0
-+VINB_4
 Wire Wire Line
 	4450 3475 4450 3625
@@
 	4225 3625 4450 3625
 Text Notes 1475 2425 0    50   ~ 0
-motherboard jumper connectors\n
+motherboard jumper headers
 Connection ~ 4225 3625
 $Comp
-L Connector_Generic:Conn_01x02 J?
+L Connector_Generic:Conn_01x02 J4
 U 1 1 620731DE
 P 4200 2525
-F 0 "J?" V 4350 2500 50  0000 R CNN
+F 0 "J4" V 4350 2500 50  0000 R CNN
 F 1 "Conn_01x02" V 4450 2700 50  0000 R CNN
 F 2 "" H 4200 2525 50  0001 C CNN
@@
 	4050 2725 4200 2725
 $Comp
-L Connector_Generic:Conn_01x02 J?
+L Connector_Generic:Conn_01x02 J3
 U 1 1 62075FD9
 P 4200 1875
-F 0 "J?" V 4350 1850 50  0000 R CNN
+F 0 "J3" V 4350 1850 50  0000 R CNN
 F 1 "Conn_01x02" V 4450 2050 50  0000 R CNN
 F 2 "" H 4200 1875 50  0001 C CNN
@@
 Wire Wire Line
 	2775 2725 3250 2725
-Wire Wire Line
-	5250 2775 5750 2775
-Wire Wire Line
-	5250 2775 5250 3375
-Connection ~ 5250 2775
-Wire Wire Line
-	5250 2675 5250 2775
 Text HLabel 5750 2075 2    50   Input ~ 0
+REFB_JUMPER
+Text HLabel 2775 2725 0    50   Input ~ 0
+VINA_JUMPER
+Text HLabel 2775 2075 0    50   Input ~ 0
+REFA_JUMPER
+Text Notes 5775 2400 0    50   ~ 0
+motherboard jumper headers\n
+Text Notes 4000 1375 0    50   ~ 0
+jumper header\n
+Text HLabel 4050 2675 1    50   Input ~ 0
+-VINA
+Text HLabel 4450 2675 1    50   Input ~ 0
++VINB
+Text HLabel 3650 2025 1    50   Input ~ 0
+REFA
+Text HLabel 4850 2025 1    50   Input ~ 0
 REFB
-Text HLabel 5750 2775 2    50   Input ~ 0
-VINB
-Text HLabel 2775 2725 0    50   Input ~ 0
-VINA
-Text HLabel 2775 2075 0    50   Input ~ 0
-REFA
-Text Notes 5775 2400 0    50   ~ 0
-motherboard jumper connectors\n
+Text HLabel 5250 2675 1    50   Input ~ 0
+-VINB
+Wire Wire Line
+	5250 2725 5250 3375
+Connection ~ 5250 2725
+Wire Wire Line
+	5250 2675 5250 2725
+Text HLabel 5750 2725 2    50   Input ~ 0
+VINB_JUMPER
+Wire Wire Line
+	5250 2725 5750 2725
+Text HLabel 3250 2675 1    50   Input ~ 0
++VINA
 $EndSCHEMATC
