File: hardware/kicad/emg-filter/emg-connectors.sch (KiCad schematic (older format))
At the start: 78 parts

Commit message: fixed rect labels
Parts:
- gave numbers to parts that had none: 78

Commit message: footprint association
Parts:
- R232: renamed from R264; footprint (none) -> Resistor_SMD:R_0805_2012Metric
- R233: renamed from R265; footprint (none) -> Resistor_SMD:R_0805_2012Metric
- R234: renamed from R266; footprint (none) -> Resistor_SMD:R_0805_2012Metric
- R235: renamed from R267; footprint (none) -> Resistor_SMD:R_0805_2012Metric
- R236: renamed from R268; footprint (none) -> Resistor_SMD:R_0805_2012Metric
- R237: renamed from R269; footprint (none) -> Resistor_SMD:R_0805_2012Metric
- R238: renamed from R270; footprint (none) -> Resistor_SMD:R_0805_2012Metric
- R239: renamed from R271; footprint (none) -> Resistor_SMD:R_0805_2012Metric
- R240: renamed from R272; footprint (none) -> Resistor_SMD:R_0805_2012Metric
- R241: renamed from R273; footprint (none) -> Resistor_SMD:R_0805_2012Metric
- R242: renamed from R274; footprint (none) -> Resistor_SMD:R_0805_2012Metric
- R243: renamed from R275; footprint (none) -> Resistor_SMD:R_0805_2012Metric
- R244: renamed from R276; footprint (none) -> Resistor_SMD:R_0805_2012Metric
- R245: renamed from R277; footprint (none) -> Resistor_SMD:R_0805_2012Metric
- R246: renamed from R278; footprint (none) -> Resistor_SMD:R_0805_2012Metric
- R247: renamed from R279; footprint (none) -> Resistor_SMD:R_0805_2012Metric
- R248: renamed from R280; footprint (none) -> Resistor_SMD:R_0805_2012Metric
- R249: renamed from R281; footprint (none) -> Resistor_SMD:R_0805_2012Metric
- R250: renamed from R282; footprint (none) -> Resistor_SMD:R_0805_2012Metric
- R251: renamed from R283; footprint (none) -> Resistor_SMD:R_0805_2012Metric
- R252: renamed from R284; footprint (none) -> Resistor_SMD:R_0805_2012Metric
- R253: renamed from R285; footprint (none) -> Resistor_SMD:R_0805_2012Metric
- R254: renamed from R286; footprint (none) -> Resistor_SMD:R_0805_2012Metric
- R255: renamed from R287; footprint (none) -> Resistor_SMD:R_0805_2012Metric
- R256: renamed from R288; footprint (none) -> Resistor_SMD:R_0805_2012Metric
- R257: renamed from R289; footprint (none) -> Resistor_SMD:R_0805_2012Metric
- R258: renamed from R290; footprint (none) -> Resistor_SMD:R_0805_2012Metric
- R259: renamed from R291; footprint (none) -> Resistor_SMD:R_0805_2012Metric
- R260: renamed from R292; footprint (none) -> Resistor_SMD:R_0805_2012Metric
- R261: renamed from R293; footprint (none) -> Resistor_SMD:R_0805_2012Metric

Commit message: Solving Stuff for Free
Parts:
- renumbered R232 to R264, R233 to R265, R234 to R266, R235 to R267, R236 to R268, R237 to R269, R238 to R270, R239 to R271, R240 to R272, R241 to R273, R242 to R274, R243 to R275, R244 to R276, R245 to R277, R246 to R278, R247 to R279, R248 to R280, R249 to R281, R250 to R282, R251 to R283, R252 to R284, R253 to R285, R254 to R286, R255 to R287, R256 to R288, R257 to R289, R258 to R290, R259 to R291, R260 to R292, R261 to R293

Commit message: Renaming Labels
Connections:
- net labels added: +VINA_11_INA, +VINA_13_INA, +VINA_15_INA, +VINA_9_INA, +VINB_10_INA, +VINB_12_INA, +VINB_14_INA, +VINB_16_INA, -VINA_11_INA, -VINA_13_INA, -VINA_15_INA, -VINA_9_INA, -VINB_10_INA, -VINB_12_INA, -VINB_14_INA, -VINB_16_INA, REFA_11_INA, REFA_13_INA, REFA_15_INA, REFA_9_INA, REFB_10_INA, REFB_12_INA, REFB_14_INA, REFB_16_INA
- net labels removed: +VINA_10_INA, +VINA_12_INA, +VINA_14_INA, +VINA_16_INA, +VINB_11_INA, +VINB_13_INA, +VINB_15_INA, +VINB_9_INA, -VINA_10_INA, -VINA_12_INA, -VINA_14_INA, -VINA_16_INA, -VINB_11_INA, -VINB_13_INA, -VINB_15_INA, -VINB_9_INA, REFA_10_INA, REFA_12_INA, REFA_14_INA, REFA_16_INA, REFB_11_INA, REFB_13_INA, REFB_15_INA, REFB_9_INA
Changed lines of the file:
@@
 $EndComp
 Text GLabel 1650 4975 3    50   Input ~ 0
--VINA_16_INA
+-VINB_16_INA
 Text GLabel 1250 5625 3    50   Input ~ 0
-REFA_16_INA
+REFB_16_INA
 Text GLabel 2450 5625 3    50   Input ~ 0
-REFB_15_INA
+REFA_15_INA
 $Comp
 L Connector_Generic:Conn_01x02 J?
@@
 	0    -1   1    0
 $EndComp
-Text GLabel 2850 4975 3    50   Input ~ 0
--VINB_15_INA
 Wire Wire Line
 	1700 4925 1650 4925
 Text GLabel 2050 4975 3    50   Input ~ 0
-+VINB_15_INA
++VINA_15_INA
 Wire Wire Line
 	2050 4175 2050 4025
@@
 $EndComp
 Text GLabel 4050 4975 3    50   Input ~ 0
--VINA_14_INA
+-VINB_14_INA
 Text GLabel 3250 4975 3    50   Input ~ 0
-+VINA_14_INA
++VINB_14_INA
 Text GLabel 3650 5625 3    50   Input ~ 0
-REFA_14_INA
+REFB_14_INA
 Text GLabel 4850 5625 3    50   Input ~ 0
-REFB_13_INA
+REFA_13_INA
 $Comp
 L Connector_Generic:Conn_01x02 J?
@@
 	0    -1   1    0
 $EndComp
-Text GLabel 5250 4975 3    50   Input ~ 0
--VINB_13_INA
 Wire Wire Line
 	4100 4925 4050 4925
 Text GLabel 4450 4975 3    50   Input ~ 0
-+VINB_13_INA
++VINA_13_INA
 Wire Wire Line
 	4450 4175 4450 4025
@@
 $EndComp
 Text GLabel 6450 4975 3    50   Input ~ 0
--VINA_12_INA
+-VINB_12_INA
 Text GLabel 5650 4975 3    50   Input ~ 0
-+VINA_12_INA
++VINB_12_INA
 Text GLabel 6050 5625 3    50   Input ~ 0
-REFA_12_INA
+REFB_12_INA
 Text GLabel 7250 5625 3    50   Input ~ 0
-REFB_11_INA
+REFA_11_INA
 $Comp
 L Connector_Generic:Conn_01x02 J?
@@
 	-1   0    0    -1
 $EndComp
-Text GLabel 7650 4975 3    50   Input ~ 0
--VINB_11_INA
 Wire Wire Line
 	6500 4925 6450 4925
 Text GLabel 6850 4975 3    50   Input ~ 0
-+VINB_11_INA
++VINA_11_INA
 Wire Wire Line
 	6850 4175 6850 4025
@@
 $EndComp
 Text GLabel 8850 4975 3    50   Input ~ 0
--VINA_10_INA
-Text GLabel 8050 4975 3    50   Input ~ 0
-+VINA_10_INA
+-VINB_10_INA
 Text GLabel 8450 5625 3    50   Input ~ 0
-REFA_10_INA
-Text GLabel 9650 5625 3    50   Input ~ 0
-REFB_9_INA
+REFB_10_INA
 $Comp
 L Connector_Generic:Conn_01x02 J?
@@
 	-1   0    0    -1
 $EndComp
-Text GLabel 10050 4975 3    50   Input ~ 0
--VINB_9_INA
 Wire Wire Line
 	8900 4925 8850 4925
 Text GLabel 9250 4975 3    50   Input ~ 0
-+VINB_9_INA
++VINA_9_INA
 Wire Wire Line
 	9250 4175 9250 4025
@@
 $EndComp
 Text GLabel 850  4975 3    50   Input ~ 0
-+VINA_16_INA
++VINB_16_INA
 $Comp
 L power:GND #PWR?
@@
 P 850 3700
 AR Path="/61C386B1/62801FCD" Ref="#PWR?"  Part="1"
-AR Path="/61C389A8/62801FCD" Ref="#PWR0175"  Part="1"
-F 0 "#PWR0175" H 850 3450 50  0001 C CNN
+AR Path="/61C389A8/62801FCD" Ref="#PWR0173"  Part="1"
+F 0 "#PWR0173" H 850 3450 50  0001 C CNN
 F 1 "GND" H 855 3527 50  0000 C CNN
 F 2 "" H 850 3700 50  0001 C CNN
@@
 Wire Wire Line
 	10375 5575 9650 5575
+Text GLabel 7650 4975 3    50   Input ~ 0
+-VINA_11_INA
+Text GLabel 8050 4975 3    50   Input ~ 0
++VINB_10_INA
+Text GLabel 9650 5625 3    50   Input ~ 0
+REFA_9_INA
+Text GLabel 10050 4975 3    50   Input ~ 0
+-VINA_9_INA
+Text GLabel 5250 4975 3    50   Input ~ 0
+-VINA_13_INA
+Text GLabel 2850 4975 3    50   Input ~ 0
+-VINA_15_INA
 $EndSCHEMATC

Commit message: pcb
Parts:
- J10, J11, J12, J13, J14, J15, J16, J17, J18, J19, J20, J21, J22, J23, J24, J25, J26, J27, J28, J29, J30, J31, J32, J33, J34, J35, J36, J37, J38, J39, J4, J40, J41, J42, J43, J44, J45, J46, J47, J48, J49, J5, J50, J51, J6, J7, J8, J9: footprint (none) -> emg-filter:EMG_CONN_01x02

Commit message: rearranged layout
Parts:
- renumbered R266 to R10, R267 to R11, R268 to R12, R269 to R13, R270 to R14, R271 to R15, R272 to R16, R273 to R17, R274 to R18, R275 to R19, R276 to R20, R277 to R21, R278 to R22, R279 to R23, R280 to R24, R281 to R25, R282 to R26, R283 to R27, R284 to R28, R285 to R29, R286 to R30, R287 to R31, R288 to R32, R289 to R33, R290 to R34, R291 to R35, R292 to R36, R293 to R37, R264 to R8, R265 to R9

Commit message: restructured entire schematic to use hierarchichal labels
Connections:
- net labels added: +VINA_1, +VINA_11, +VINA_13, +VINA_15, +VINA_3, +VINA_5, +VINA_7, +VINA_9, +VINB_10, +VINB_12, +VINB_14, +VINB_16, +VINB_2, +VINB_4, +VINB_6, +VINB_8, -VINA_1, -VINA_11, -VINA_13, -VINA_15, -VINA_3, -VINA_5, -VINA_7, -VINA_9, -VINB_10, -VINB_12, -VINB_14, -VINB_16, -VINB_2, -VINB_4, -VINB_6, -VINB_8, REFA_1, REFA_11, REFA_13, REFA_15, REFA_3, REFA_5, REFA_7, REFA_9, REFB_10, REFB_12, REFB_14, REFB_16, REFB_2, REFB_4, REFB_6, REFB_8
- net labels removed: +VINA_11_INA, +VINA_13_INA, +VINA_15_INA, +VINA_1_INA, +VINA_3_INA, +VINA_5_INA, +VINA_7_INA, +VINA_9_INA, +VINB_10_INA, +VINB_12_INA, +VINB_14_INA, +VINB_16_INA, +VINB_2_INA, +VINB_4_INA, +VINB_6_INA, +VINB_8_INA, -VINA_11_INA, -VINA_13_INA, -VINA_15_INA, -VINA_1_INA, -VINA_3_INA, -VINA_5_INA, -VINA_7_INA, -VINA_9_INA, -VINB_10_INA, -VINB_12_INA, -VINB_14_INA, -VINB_16_INA, -VINB_2_INA, -VINB_4_INA, -VINB_6_INA, -VINB_8_INA, REFA_11_INA, REFA_13_INA, REFA_15_INA, REFA_1_INA, REFA_3_INA, REFA_5_INA, REFA_7_INA, REFA_9_INA, REFB_10_INA, REFB_12_INA, REFB_14_INA, REFB_16_INA, REFB_2_INA, REFB_4_INA, REFB_6_INA, REFB_8_INA
Changed lines of the file:
@@
 $EndComp
 Text GLabel 1650 4975 3    50   Input ~ 0
--VINB_16_INA
+-VINB_16
 Text GLabel 1250 5625 3    50   Input ~ 0
-REFB_16_INA
+REFB_16
 Text GLabel 2450 5625 3    50   Input ~ 0
-REFA_15_INA
+REFA_15
 $Comp
 L Connector_Generic:Conn_01x02 J?
@@
 	1700 4925 1650 4925
 Text GLabel 2050 4975 3    50   Input ~ 0
-+VINA_15_INA
++VINA_15
 Wire Wire Line
 	2050 4175 2050 4025
@@
 $EndComp
 Text GLabel 4050 4975 3    50   Input ~ 0
--VINB_14_INA
+-VINB_14
 Text GLabel 3250 4975 3    50   Input ~ 0
-+VINB_14_INA
++VINB_14
 Text GLabel 3650 5625 3    50   Input ~ 0
-REFB_14_INA
+REFB_14
 Text GLabel 4850 5625 3    50   Input ~ 0
-REFA_13_INA
+REFA_13
 $Comp
 L Connector_Generic:Conn_01x02 J?
@@
 	4100 4925 4050 4925
 Text GLabel 4450 4975 3    50   Input ~ 0
-+VINA_13_INA
++VINA_13
 Wire Wire Line
 	4450 4175 4450 4025
@@
 $EndComp
 Text GLabel 6450 4975 3    50   Input ~ 0
--VINB_12_INA
+-VINB_12
 Text GLabel 5650 4975 3    50   Input ~ 0
-+VINB_12_INA
++VINB_12
 Text GLabel 6050 5625 3    50   Input ~ 0
-REFB_12_INA
+REFB_12
 Text GLabel 7250 5625 3    50   Input ~ 0
-REFA_11_INA
+REFA_11
 $Comp
 L Connector_Generic:Conn_01x02 J?
@@
 	6500 4925 6450 4925
 Text GLabel 6850 4975 3    50   Input ~ 0
-+VINA_11_INA
++VINA_11
 Wire Wire Line
 	6850 4175 6850 4025
@@
 $EndComp
 Text GLabel 8850 4975 3    50   Input ~ 0
--VINB_10_INA
+-VINB_10
 Text GLabel 8450 5625 3    50   Input ~ 0
-REFB_10_INA
+REFB_10
 $Comp
 L Connector_Generic:Conn_01x02 J?
@@
 	8900 4925 8850 4925
 Text GLabel 9250 4975 3    50   Input ~ 0
-+VINA_9_INA
++VINA_9
 Wire Wire Line
 	9250 4175 9250 4025
@@
 $EndComp
 Text GLabel 1650 2675 1    50   Input ~ 0
--VINA_1_INA
+-VINA_1
 Text GLabel 850  2675 1    50   Input ~ 0
-+VINA_1_INA
++VINA_1
 Text GLabel 1250 2025 1    50   Input ~ 0
-REFA_1_INA
+REFA_1
 Text GLabel 2450 2025 1    50   Input ~ 0
-REFB_2_INA
+REFB_2
 $Comp
 L Connector_Generic:Conn_01x02 J?
@@
 $EndComp
 Text GLabel 2850 2675 1    50   Input ~ 0
--VINB_2_INA
+-VINB_2
 Wire Wire Line
 	1700 2725 1650 2725
 Text GLabel 2050 2675 1    50   Input ~ 0
-+VINB_2_INA
++VINB_2
 Wire Wire Line
 	2050 3475 2050 3625
@@
 $EndComp
 Text GLabel 4050 2675 1    50   Input ~ 0
--VINA_3_INA
+-VINA_3
 Text GLabel 3250 2675 1    50   Input ~ 0
-+VINA_3_INA
++VINA_3
 Text GLabel 3650 2025 1    50   Input ~ 0
-REFA_3_INA
+REFA_3
 Text GLabel 4850 2025 1    50   Input ~ 0
-REFB_4_INA
+REFB_4
 $Comp
 L Connector_Generic:Conn_01x02 J?
@@
 $EndComp
 Text GLabel 5250 2675 1    50   Input ~ 0
--VINB_4_INA
+-VINB_4
 Wire Wire Line
 	4100 2725 4050 2725
 Text GLabel 4450 2675 1    50   Input ~ 0
-+VINB_4_INA
++VINB_4
 Wire Wire Line
 	4450 3475 4450 3625
@@
 $EndComp
 Text GLabel 6450 2675 1    50   Input ~ 0
--VINA_5_INA
+-VINA_5
 Text GLabel 5650 2675 1    50   Input ~ 0
-+VINA_5_INA
++VINA_5
 Text GLabel 6050 2025 1    50   Input ~ 0
-REFA_5_INA
+REFA_5
 Text GLabel 7250 2025 1    50   Input ~ 0
-REFB_6_INA
+REFB_6
 $Comp
 L Connector_Generic:Conn_01x02 J?
@@
 $EndComp
 Text GLabel 7650 2675 1    50   Input ~ 0
--VINB_6_INA
+-VINB_6
 Wire Wire Line
 	6500 2725 6450 2725
 Text GLabel 6850 2675 1    50   Input ~ 0
-+VINB_6_INA
++VINB_6
 Wire Wire Line
 	6850 3475 6850 3625
@@
 $EndComp
 Text GLabel 8850 2675 1    50   Input ~ 0
--VINA_7_INA
+-VINA_7
 Text GLabel 8050 2675 1    50   Input ~ 0
-+VINA_7_INA
++VINA_7
 Text GLabel 8450 2025 1    50   Input ~ 0
-REFA_7_INA
+REFA_7
 Text GLabel 9650 2025 1    50   Input ~ 0
-REFB_8_INA
+REFB_8
 $Comp
 L Connector_Generic:Conn_01x02 J?
@@
 $EndComp
 Text GLabel 10050 2675 1    50   Input ~ 0
--VINB_8_INA
+-VINB_8
 Wire Wire Line
 	8900 2725 8850 2725
 Text GLabel 9250 2675 1    50   Input ~ 0
-+VINB_8_INA
++VINB_8
 Wire Wire Line
 	9250 3475 9250 3625
@@
 $EndComp
 Text GLabel 850  4975 3    50   Input ~ 0
-+VINB_16_INA
++VINB_16
 $Comp
 L power:GND #PWR?
@@
 	10375 5575 9650 5575
 Text GLabel 7650 4975 3    50   Input ~ 0
--VINA_11_INA
+-VINA_11
+Text GLabel 9650 5625 3    50   Input ~ 0
+REFA_9
+Text GLabel 10050 4975 3    50   Input ~ 0
+-VINA_9
+Text GLabel 5250 4975 3    50   Input ~ 0
+-VINA_13
+Text GLabel 2850 4975 3    50   Input ~ 0
+-VINA_15
 Text GLabel 8050 4975 3    50   Input ~ 0
-+VINB_10_INA
-Text GLabel 9650 5625 3    50   Input ~ 0
-REFA_9_INA
-Text GLabel 10050 4975 3    50   Input ~ 0
--VINA_9_INA
-Text GLabel 5250 4975 3    50   Input ~ 0
--VINA_13_INA
-Text GLabel 2850 4975 3    50   Input ~ 0
--VINA_15_INA
++VINB_10
 $EndSCHEMATC

Commit message: added 5 pin conn, got rid of filters
Parts:
- added J? (x16): Conn_01x02, symbol Connector_Generic:Conn_01x02
Changed lines of the file:
@@
 Text GLabel 8050 4975 3    50   Input ~ 0
 +VINB_10
+$Comp
+L Connector_Generic:Conn_01x02 J?
+U 1 1 62075168
+P -4850 1200
+F 0 "J?" H -4770 1192 50  0000 L CNN
+F 1 "Conn_01x02" H -4770 1101 50  0000 L CNN
+F 2 "" H -4850 1200 50  0001 C CNN
+F 3 "~" H -4850 1200 50  0001 C CNN
+	1    -4850 1200
+	1    0    0    -1
+$EndComp
+$Comp
+L Connector_Generic:Conn_01x02 J?
+U 1 1 6207750E
+P -4850 1675
+F 0 "J?" H -4770 1667 50  0000 L CNN
+F 1 "Conn_01x02" H -4770 1576 50  0000 L CNN
+F 2 "" H -4850 1675 50  0001 C CNN
+F 3 "~" H -4850 1675 50  0001 C CNN
+	1    -4850 1675
+	1    0    0    -1
+$EndComp
+$Comp
+L Connector_Generic:Conn_01x02 J?
+U 1 1 6210D646
+P -3850 1250
+F 0 "J?" H -3770 1242 50  0000 L CNN
+F 1 "Conn_01x02" H -3770 1151 50  0000 L CNN
+F 2 "" H -3850 1250 50  0001 C CNN
+F 3 "~" H -3850 1250 50  0001 C CNN
+	1    -3850 1250
+	1    0    0    -1
+$EndComp
+$Comp
+L Connector_Generic:Conn_01x02 J?
+U 1 1 6210D64C
+P -3850 1725
+F 0 "J?" H -3770 1717 50  0000 L CNN
+F 1 "Conn_01x02" H -3770 1626 50  0000 L CNN
+F 2 "" H -3850 1725 50  0001 C CNN
+F 3 "~" H -3850 1725 50  0001 C CNN
+	1    -3850 1725
+	1    0    0    -1
+$EndComp
+$Comp
+L Connector_Generic:Conn_01x02 J?
+U 1 1 6211DCBE
+P -2775 1250
+F 0 "J?" H -2695 1242 50  0000 L CNN
+F 1 "Conn_01x02" H -2695 1151 50  0000 L CNN
+F 2 "" H -2775 1250 50  0001 C CNN
+F 3 "~" H -2775 1250 50  0001 C CNN
+	1    -2775 1250
+	1    0    0    -1
+$EndComp
+$Comp
+L Connector_Generic:Conn_01x02 J?
+U 1 1 6211DCC4
+P -2775 1725
+F 0 "J?" H -2695 1717 50  0000 L CNN
+F 1 "Conn_01x02" H -2695 1626 50  0000 L CNN
+F 2 "" H -2775 1725 50  0001 C CNN
+F 3 "~" H -2775 1725 50  0001 C CNN
+	1    -2775 1725
+	1    0    0    -1
+$EndComp
+$Comp
+L Connector_Generic:Conn_01x02 J?
+U 1 1 6212E57C
+P -1625 1250
+F 0 "J?" H -1545 1242 50  0000 L CNN
+F 1 "Conn_01x02" H -1545 1151 50  0000 L CNN
+F 2 "" H -1625 1250 50  0001 C CNN
+F 3 "~" H -1625 1250 50  0001 C CNN
+	1    -1625 1250
+	1    0    0    -1
+$EndComp
+$Comp
+L Connector_Generic:Conn_01x02 J?
+U 1 1 6212E582
+P -1625 1725
+F 0 "J?" H -1545 1717 50  0000 L CNN
+F 1 "Conn_01x02" H -1545 1626 50  0000 L CNN
+F 2 "" H -1625 1725 50  0001 C CNN
+F 3 "~" H -1625 1725 50  0001 C CNN
+	1    -1625 1725
+	1    0    0    -1
+$EndComp
+$Comp
+L Connector_Generic:Conn_01x02 J?
+U 1 1 6214D5BE
+P -4850 175
+F 0 "J?" H -4770 167 50  0000 L CNN
+F 1 "Conn_01x02" H -4770 76  50  0000 L CNN
+F 2 "" H -4850 175 50  0001 C CNN
+F 3 "~" H -4850 175 50  0001 C CNN
+	1    -4850 175
+	1    0    0    -1
+$EndComp
+$Comp
+L Connector_Generic:Conn_01x02 J?
+U 1 1 6214D5C4
+P -4850 650
+F 0 "J?" H -4770 642 50  0000 L CNN
+F 1 "Conn_01x02" H -4770 551 50  0000 L CNN
+F 2 "" H -4850 650 50  0001 C CNN
+F 3 "~" H -4850 650 50  0001 C CNN
+	1    -4850 650
+	1    0    0    -1
+$EndComp
+$Comp
+L Connector_Generic:Conn_01x02 J?
+U 1 1 6214D5CA
+P -3850 225
+F 0 "J?" H -3770 217 50  0000 L CNN
+F 1 "Conn_01x02" H -3770 126 50  0000 L CNN
+F 2 "" H -3850 225 50  0001 C CNN
+F 3 "~" H -3850 225 50  0001 C CNN
+	1    -3850 225
+	1    0    0    -1
+$EndComp
+$Comp
+L Connector_Generic:Conn_01x02 J?
+U 1 1 6214D5D0
+P -3850 700
+F 0 "J?" H -3770 692 50  0000 L CNN
+F 1 "Conn_01x02" H -3770 601 50  0000 L CNN
+F 2 "" H -3850 700 50  0001 C CNN
+F 3 "~" H -3850 700 50  0001 C CNN
+	1    -3850 700
+	1    0    0    -1
+$EndComp
+$Comp
+L Connector_Generic:Conn_01x02 J?
+U 1 1 6214D5D6
+P -2775 225
+F 0 "J?" H -2695 217 50  0000 L CNN
+F 1 "Conn_01x02" H -2695 126 50  0000 L CNN
+F 2 "" H -2775 225 50  0001 C CNN
+F 3 "~" H -2775 225 50  0001 C CNN
+	1    -2775 225
+	1    0    0    -1
+$EndComp
+$Comp
+L Connector_Generic:Conn_01x02 J?
+U 1 1 6214D5DC
+P -2775 700
+F 0 "J?" H -2695 692 50  0000 L CNN
+F 1 "Conn_01x02" H -2695 601 50  0000 L CNN
+F 2 "" H -2775 700 50  0001 C CNN
+F 3 "~" H -2775 700 50  0001 C CNN
+	1    -2775 700
+	1    0    0    -1
+$EndComp
+$Comp
+L Connector_Generic:Conn_01x02 J?
+U 1 1 6214D5E2
+P -1625 225
+F 0 "J?" H -1545 217 50  0000 L CNN
+F 1 "Conn_01x02" H -1545 126 50  0000 L CNN
+F 2 "" H -1625 225 50  0001 C CNN
+F 3 "~" H -1625 225 50  0001 C CNN
+	1    -1625 225
+	1    0    0    -1
+$EndComp
+$Comp
+L Connector_Generic:Conn_01x02 J?
+U 1 1 6214D5E8
+P -1625 700
+F 0 "J?" H -1545 692 50  0000 L CNN
+F 1 "Conn_01x02" H -1545 601 50  0000 L CNN
+F 2 "" H -1625 700 50  0001 C CNN
+F 3 "~" H -1625 700 50  0001 C CNN
+	1    -1625 700
+	1    0    0    -1
+$EndComp
 $EndSCHEMATC
