File: hardware/kicad/emg-filter/filter.sch (KiCad schematic (older format))
At the start: 63 parts, among them U10 LM4565, U11 LM4565, U5 INA2332, U6 LM4565, U7 LM4565, U8 LM4565, U9 LM4565

Commit message: restructured entire schematic to use hierarchichal labels
Parts:
- removed C88, C96: 10n, Capacitor_SMD:C_0805_2012Metric, symbol Device:C
- removed C92: 20n, Capacitor_SMD:C_0805_2012Metric, symbol Device:C
- removed R40, R44: 132k, Resistor_SMD:R_0805_2012Metric, symbol Device:R
- removed R45, R48: 133k, Resistor_SMD:R_0805_2012Metric, symbol Device:R
- removed R56: 2k, Resistor_SMD:R_0805_2012Metric, symbol Device:R
- removed R57: 266k, Resistor_SMD:R_0805_2012Metric, symbol Device:R
- removed U7: LM4565, emg-filter:LM4565, symbol emg-filter:LM4565
- added C93, C97: 10n, Capacitor_SMD:C_0805_2012Metric, symbol Device:C
- added C95: 20n, Capacitor_SMD:C_0805_2012Metric, symbol Device:C
- added R47: 132k, Resistor_SMD:R_0805_2012Metric, symbol Device:R
- added R51, R53, R55: 133k, Resistor_SMD:R_0805_2012Metric, symbol Device:R
- added R58: 2k, Resistor_SMD:R_0805_2012Metric, symbol Device:R
- added R59: 266k, Resistor_SMD:R_0805_2012Metric, symbol Device:R
- added U8: LM4565, emg-filter:LM4565, symbol emg-filter:LM4565
- R50: value 133k -> 132k
- renumbered C90 to C88, C91 to C89, C94 to C90, C95 to C91, C89 to C92, C93 to C94, C97 to C96, R42 to R40, R43 to R41, R52 to R42, R53 to R43, R54 to R44, R55 to R45, R41 to R46, R46 to R48, R47 to R49, R49 to R52, R51 to R54, R58 to R56, R59 to R57, U8 to U7
Connections:
- net labels added: +VIN_A, +VIN_B, -VIN_A, -VIN_B, OUT_A, OUT_B, REF_A, REF_B
- net labels removed: +IN2_1_NOTCH, +IN2_2_NOTCH, +VINA_1_INA, +VINB_2_INA, -VINA_1_INA, -VINB_2_INA, BP_NOTCH_1, BP_NOTCH_2, INA_BP_1, INA_BP_2, NOTCH_RECT_1, NOTCH_RECT_2, OUT_AMP_1, OUT_AMP_2, RECT_AMP_1, RECT_AMP_2, REFA_1_INA, REFB_2_INA, SHTDWN_INA
- wire segments 243 -> 261
Other:
- moved on the sheet: C102, C103, C104, C105, C106, C107, C108, C110, C112, C114, C115, C116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
