File: hardware/kicad/emg-filter/input_ina.sch (KiCad schematic (older format))
At the start: 8 parts, among them J4 Conn_01x02, J5 Conn_01x02, J6 Conn_01x02, J7 Conn_01x02, J8 Conn_01x02, J9 Conn_01x02

Commit message: compact design
Parts:
- renumbered R246 to R326, R247 to R327
Changed lines of the file:
@@
 $Descr A4 11693 8268
 encoding utf-8
-Sheet 36 43
+Sheet 28 43
 Title ""
 Date ""
@@
 AR Path="/61C386B1/623023B9" Ref="R?"  Part="1"
 AR Path="/61C389A8/623023B9" Ref="R?"  Part="1"
-AR Path="/622FC90E/623023B9" Ref="R247"  Part="1"
+AR Path="/622FC90E/623023B9" Ref="R327"  Part="1"
 AR Path="/623EBE47/623023B9" Ref="R?"  Part="1"
-AR Path="/624814DA/623023B9" Ref="R257"  Part="1"
-AR Path="/6248A382/623023B9" Ref="R267"  Part="1"
-AR Path="/6248A3A0/623023B9" Ref="R277"  Part="1"
-AR Path="/624986BC/623023B9" Ref="R287"  Part="1"
-AR Path="/624986DA/623023B9" Ref="R297"  Part="1"
-AR Path="/624986F8/623023B9" Ref="R307"  Part="1"
-AR Path="/62498716/623023B9" Ref="R317"  Part="1"
-F 0 "R317" H 5420 3521 50  0000 L CNN
+AR Path="/624814DA/623023B9" Ref="R337"  Part="1"
+AR Path="/6248A382/623023B9" Ref="R347"  Part="1"
+AR Path="/6248A3A0/623023B9" Ref="R357"  Part="1"
+AR Path="/624986BC/623023B9" Ref="R367"  Part="1"
+AR Path="/624986DA/623023B9" Ref="R377"  Part="1"
+AR Path="/624986F8/623023B9" Ref="R387"  Part="1"
+AR Path="/62498716/623023B9" Ref="R397"  Part="1"
+F 0 "R397" H 5420 3521 50  0000 L CNN
 F 1 "0" H 5420 3430 50  0000 L CNN
 F 2 "Resistor_SMD:R_0805_2012Metric" V 5280 3475 50  0001 C CNN
@@
 AR Path="/61C386B1/623023BF" Ref="R?"  Part="1"
 AR Path="/61C389A8/623023BF" Ref="R?"  Part="1"
-AR Path="/622FC90E/623023BF" Ref="R246"  Part="1"
+AR Path="/622FC90E/623023BF" Ref="R326"  Part="1"
 AR Path="/623EBE47/623023BF" Ref="R?"  Part="1"
-AR Path="/624814DA/623023BF" Ref="R256"  Part="1"
-AR Path="/6248A382/623023BF" Ref="R266"  Part="1"
-AR Path="/6248A3A0/623023BF" Ref="R276"  Part="1"
-AR Path="/624986BC/623023BF" Ref="R286"  Part="1"
-AR Path="/624986DA/623023BF" Ref="R296"  Part="1"
-AR Path="/624986F8/623023BF" Ref="R306"  Part="1"
-AR Path="/62498716/623023BF" Ref="R316"  Part="1"
-F 0 "R316" H 5145 3521 50  0000 L CNN
+AR Path="/624814DA/623023BF" Ref="R336"  Part="1"
+AR Path="/6248A382/623023BF" Ref="R346"  Part="1"
+AR Path="/6248A3A0/623023BF" Ref="R356"  Part="1"
+AR Path="/624986BC/623023BF" Ref="R366"  Part="1"
+AR Path="/624986DA/623023BF" Ref="R376"  Part="1"
+AR Path="/624986F8/623023BF" Ref="R386"  Part="1"
+AR Path="/62498716/623023BF" Ref="R396"  Part="1"
+F 0 "R396" H 5145 3521 50  0000 L CNN
 F 1 "0" H 5145 3430 50  0000 L CNN
 F 2 "Resistor_SMD:R_0805_2012Metric" V 5005 3475 50  0001 C CNN
@@
 AR Path="/622FC90E/623023FB" Ref="#PWR0149"  Part="1"
 AR Path="/623EBE47/623023FB" Ref="#PWR?"  Part="1"
-AR Path="/624814DA/623023FB" Ref="#PWR0155"  Part="1"
-AR Path="/6248A382/623023FB" Ref="#PWR0161"  Part="1"
-AR Path="/6248A3A0/623023FB" Ref="#PWR0167"  Part="1"
-AR Path="/624986BC/623023FB" Ref="#PWR0173"  Part="1"
-AR Path="/624986DA/623023FB" Ref="#PWR0179"  Part="1"
-AR Path="/624986F8/623023FB" Ref="#PWR0185"  Part="1"
-AR Path="/62498716/623023FB" Ref="#PWR0191"  Part="1"
-F 0 "#PWR0191" H 4175 4275 50  0001 C CNN
+AR Path="/624814DA/623023FB" Ref="#PWR0157"  Part="1"
+AR Path="/6248A382/623023FB" Ref="#PWR0165"  Part="1"
+AR Path="/6248A3A0/623023FB" Ref="#PWR0173"  Part="1"
+AR Path="/624986BC/623023FB" Ref="#PWR0181"  Part="1"
+AR Path="/624986DA/623023FB" Ref="#PWR0189"  Part="1"
+AR Path="/624986F8/623023FB" Ref="#PWR0197"  Part="1"
+AR Path="/62498716/623023FB" Ref="#PWR0205"  Part="1"
+F 0 "#PWR0205" H 4175 4275 50  0001 C CNN
 F 1 "GND" H 4180 4352 50  0000 C CNN
 F 2 "" H 4175 4525 50  0001 C CNN

Commit message: update
Changed lines of the file:
@@
 $Descr A4 11693 8268
 encoding utf-8
-Sheet 28 43
+Sheet 28 7
 Title ""
 Date ""
@@
 AR Path="/624986F8/6230239E" Ref="J44"  Part="1"
 AR Path="/62498716/6230239E" Ref="J50"  Part="1"
-F 0 "J50" V 4289 3687 50  0000 R CNN
+F 0 "J8" V 4289 3687 50  0000 R CNN
 F 1 "Conn_01x02" V 4198 3687 50  0000 R CNN
 F 2 "emg-filter:EMG_CONN_01x02" H 4325 3875 50  0001 C CNN
@@
 AR Path="/624986F8/623023A4" Ref="J42"  Part="1"
 AR Path="/62498716/623023A4" Ref="J48"  Part="1"
-F 0 "J48" V 4289 2887 50  0000 R CNN
+F 0 "J6" V 4289 2887 50  0000 R CNN
 F 1 "Conn_01x02" V 4198 2887 50  0000 R CNN
 F 2 "emg-filter:EMG_CONN_01x02" H 4325 3075 50  0001 C CNN
@@
 AR Path="/624986F8/623023AA" Ref="J40"  Part="1"
 AR Path="/62498716/623023AA" Ref="J46"  Part="1"
-F 0 "J46" V 4289 2087 50  0000 R CNN
+F 0 "J4" V 4289 2087 50  0000 R CNN
 F 1 "Conn_01x02" V 4198 2087 50  0000 R CNN
 F 2 "emg-filter:EMG_CONN_01x02" H 4325 2275 50  0001 C CNN
@@
 AR Path="/624986F8/623023B0" Ref="J41"  Part="1"
 AR Path="/62498716/623023B0" Ref="J47"  Part="1"
-F 0 "J47" V 4289 2487 50  0000 R CNN
+F 0 "J5" V 4289 2487 50  0000 R CNN
 F 1 "Conn_01x02" V 4198 2487 50  0000 R CNN
 F 2 "emg-filter:EMG_CONN_01x02" H 4325 2675 50  0001 C CNN
@@
 AR Path="/624986F8/623023B9" Ref="R387"  Part="1"
 AR Path="/62498716/623023B9" Ref="R397"  Part="1"
-F 0 "R397" H 5420 3521 50  0000 L CNN
+F 0 "R327" H 5420 3521 50  0000 L CNN
 F 1 "0" H 5420 3430 50  0000 L CNN
 F 2 "Resistor_SMD:R_0805_2012Metric" V 5280 3475 50  0001 C CNN
@@
 AR Path="/624986F8/623023BF" Ref="R386"  Part="1"
 AR Path="/62498716/623023BF" Ref="R396"  Part="1"
-F 0 "R396" H 5145 3521 50  0000 L CNN
+F 0 "R326" H 5145 3521 50  0000 L CNN
 F 1 "0" H 5145 3430 50  0000 L CNN
 F 2 "Resistor_SMD:R_0805_2012Metric" V 5005 3475 50  0001 C CNN
@@
 AR Path="/624986F8/623023C9" Ref="J45"  Part="1"
 AR Path="/62498716/623023C9" Ref="J51"  Part="1"
-F 0 "J51" V 4289 4087 50  0000 R CNN
+F 0 "J9" V 4289 4087 50  0000 R CNN
 F 1 "Conn_01x02" V 4198 4087 50  0000 R CNN
 F 2 "emg-filter:EMG_CONN_01x02" H 4325 4275 50  0001 C CNN
@@
 AR Path="/624986F8/623023D3" Ref="J43"  Part="1"
 AR Path="/62498716/623023D3" Ref="J49"  Part="1"
-F 0 "J49" V 4289 3287 50  0000 R CNN
+F 0 "J7" V 4289 3287 50  0000 R CNN
 F 1 "Conn_01x02" V 4198 3287 50  0000 R CNN
 F 2 "emg-filter:EMG_CONN_01x02" H 4325 3475 50  0001 C CNN
@@
 AR Path="/624986F8/623023FB" Ref="#PWR0197"  Part="1"
 AR Path="/62498716/623023FB" Ref="#PWR0205"  Part="1"
-F 0 "#PWR0205" H 4175 4275 50  0001 C CNN
+F 0 "#PWR0149" H 4175 4275 50  0001 C CNN
 F 1 "GND" H 4180 4352 50  0000 C CNN
 F 2 "" H 4175 4525 50  0001 C CNN

Commit message: update
Parts:
- removed R326, R327: 0, Resistor_SMD:R_0805_2012Metric, symbol Device:R
- added J? (x2): Conn_01x02, emg-filter:EMG_CONN_01x02, symbol Connector_Generic:Conn_01x02
