File: hardware/kicad/emg-filter/input_ina.sch (KiCad schematic (older format))
At the start: 8 parts, among them J4 Conn_01x02, J5 Conn_01x02, J6 Conn_01x02, J66 Conn_01x02, J67 Conn_01x02, J7 Conn_01x02, J8 Conn_01x02, J9 Conn_01x02

Commit message: Isolating module
Parts:
- renumbered J8 to J10, J9 to J11, J66 to J4, J67 to J5, J4 to J6, J5 to J7, J6 to J8, J7 to J9

Commit message: Update pcb module
Parts:
- J7: renamed from J5; footprint (none) -> Connector_PinHeader_2.54mm:PinHeader_1x02_P2.54mm_Vertical
- J8: renamed from J4; footprint (none) -> Connector_PinHeader_2.54mm:PinHeader_1x02_P2.54mm_Vertical
- renumbered J6 to J4, J7 to J5, J8 to J6

Commit message: fixed shematic
Changed lines of the file:
@@
 $Descr A4 11693 8268
 encoding utf-8
-Sheet 4 7
+Sheet 7 7
 Title ""
 Date ""
@@
 Wire Wire Line
 	3475 4725 3325 4725
-Wire Wire Line
-	4150 4075 4150 3925
 Wire Wire Line
 	3475 4325 3325 4325
@@
 AR Path="/62498716/623023FB" Ref="#PWR?"  Part="1"
 AR Path="/622DADD3/622DC40E/623023FB" Ref="#PWR?"  Part="1"
-AR Path="/622DADD3/62542119/623023FB" Ref="#PWR011"  Part="1"
+AR Path="/622DADD3/62542119/623023FB" Ref="#PWR034"  Part="1"
 AR Path="/62646A72/62542119/623023FB" Ref="#PWR?"  Part="1"
 AR Path="/62807237/62542119/623023FB" Ref="#PWR?"  Part="1"
@@
 AR Path="/6284E31C/62542119/623023FB" Ref="#PWR?"  Part="1"
 AR Path="/6284E336/62542119/623023FB" Ref="#PWR?"  Part="1"
-F 0 "#PWR011" H 3325 3875 50  0001 C CNN
+F 0 "#PWR034" H 3325 3875 50  0001 C CNN
 F 1 "GND" H 3330 3952 50  0000 C CNN
 F 2 "" H 3325 4125 50  0001 C CNN
@@
 Wire Wire Line
 	5200 4175 5200 4725
-$Comp
-L Connector_Generic:Conn_01x02 J?
-U 1 1 622E4DD4
-P 4350 4075
-AR Path="/622FC90E/622E4DD4" Ref="J?"  Part="1"
-AR Path="/624814DA/622E4DD4" Ref="J?"  Part="1"
-AR Path="/6248A382/622E4DD4" Ref="J?"  Part="1"
-AR Path="/6248A3A0/622E4DD4" Ref="J?"  Part="1"
-AR Path="/624986BC/622E4DD4" Ref="J?"  Part="1"
-AR Path="/624986DA/622E4DD4" Ref="J?"  Part="1"
-AR Path="/624986F8/622E4DD4" Ref="J?"  Part="1"
-AR Path="/62498716/622E4DD4" Ref="J?"  Part="1"
-AR Path="/622DADD3/62542119/622E4DD4" Ref="J7"  Part="1"
-AR Path="/62646A72/62542119/622E4DD4" Ref="J?"  Part="1"
-AR Path="/62807237/62542119/622E4DD4" Ref="J?"  Part="1"
-AR Path="/62807263/62542119/622E4DD4" Ref="J?"  Part="1"
-AR Path="/6284E2B1/62542119/622E4DD4" Ref="J?"  Part="1"
-AR Path="/6284E2DD/62542119/622E4DD4" Ref="J?"  Part="1"
-AR Path="/6284E31C/62542119/622E4DD4" Ref="J?"  Part="1"
-AR Path="/6284E336/62542119/622E4DD4" Ref="J?"  Part="1"
-F 0 "J7" H 4525 3975 50  0000 R CNN
-F 1 "Conn_01x02" H 4900 4075 50  0000 R CNN
-F 2 "Connector_PinHeader_2.54mm:PinHeader_1x02_P2.54mm_Vertical" H 4350 4075 50  0001 C CNN
-F 3 "~" H 4350 4075 50  0001 C CNN
-	1    4350 4075
-	1    0    0    -1
-$EndComp
 Wire Wire Line
 	5200 3525 3575 3525
@@
 	0    -1   -1   0
 $EndComp
+Wire Wire Line
+	4150 4075 4150 3925
+$Comp
+L Connector_Generic:Conn_01x02 J?
+U 1 1 622E4DD4
+P 4350 4175
+AR Path="/622FC90E/622E4DD4" Ref="J?"  Part="1"
+AR Path="/624814DA/622E4DD4" Ref="J?"  Part="1"
+AR Path="/6248A382/622E4DD4" Ref="J?"  Part="1"
+AR Path="/6248A3A0/622E4DD4" Ref="J?"  Part="1"
+AR Path="/624986BC/622E4DD4" Ref="J?"  Part="1"
+AR Path="/624986DA/622E4DD4" Ref="J?"  Part="1"
+AR Path="/624986F8/622E4DD4" Ref="J?"  Part="1"
+AR Path="/62498716/622E4DD4" Ref="J?"  Part="1"
+AR Path="/622DADD3/62542119/622E4DD4" Ref="J7"  Part="1"
+AR Path="/62646A72/62542119/622E4DD4" Ref="J?"  Part="1"
+AR Path="/62807237/62542119/622E4DD4" Ref="J?"  Part="1"
+AR Path="/62807263/62542119/622E4DD4" Ref="J?"  Part="1"
+AR Path="/6284E2B1/62542119/622E4DD4" Ref="J?"  Part="1"
+AR Path="/6284E2DD/62542119/622E4DD4" Ref="J?"  Part="1"
+AR Path="/6284E31C/62542119/622E4DD4" Ref="J?"  Part="1"
+AR Path="/6284E336/62542119/622E4DD4" Ref="J?"  Part="1"
+F 0 "J7" H 4525 4075 50  0000 R CNN
+F 1 "Conn_01x02" H 4900 4175 50  0000 R CNN
+F 2 "Connector_PinHeader_2.54mm:PinHeader_1x02_P2.54mm_Vertical" H 4350 4175 50  0001 C CNN
+F 3 "~" H 4350 4175 50  0001 C CNN
+	1    4350 4175
+	1    0    0    1
+$EndComp
 $EndSCHEMATC
