File: hardware/kicad/emg-filter/input_ina.sch (KiCad schematic (older format))
At the start: 8 parts, among them J4 Conn_01x02, J5 Conn_01x02, J6 Conn_01x02, J7 Conn_01x02, J8 Conn_01x02, J9 Conn_01x02

Commit message: modular design
Parts:
- removed R326, R327: 0, Resistor_SMD:R_0805_2012Metric, symbol Device:R
- added J? (x2): Conn_01x02, symbol Connector_Generic:Conn_01x02

Commit message: Annotation
Parts:
- gave numbers to parts that had none: 2
