File: hardware/kicad/emg-filter/amplifier.sch (KiCad schematic (older format))
At the start: 7 parts, among them U42 LM4565

Commit message: Isolating module
Parts:
- renumbered C17 to C16, R324 to R25, R322 to R26, R323 to R27, R325 to R28, U42 to U5

Commit message: Update pcb module
Parts:
- C15, C16: value 0.1uF -> 0.1u
- renumbered R25 to R27, R26 to R28, R27 to R29, R28 to R30
Changed lines of the file:
@@
 $Descr USLetter 11000 8500
 encoding utf-8
-Sheet 22 7
+Sheet 5 7
 Title "EMG Filter for Prosthetic Limb Control System"
 Date "2022-01-07"
@@
 AR Path="/6224B28B/61C410A1" Ref="R?"  Part="1"
 AR Path="/622DADD3/622DC406/61C410A1" Ref="R?"  Part="1"
-AR Path="/622DADD3/62542111/61C410A1" Ref="R25"  Part="1"
+AR Path="/622DADD3/62542111/61C410A1" Ref="R27"  Part="1"
 AR Path="/62646A72/62542111/61C410A1" Ref="R?"  Part="1"
 AR Path="/62807237/62542111/61C410A1" Ref="R?"  Part="1"
@@
 AR Path="/6284E31C/62542111/61C410A1" Ref="R?"  Part="1"
 AR Path="/6284E336/62542111/61C410A1" Ref="R?"  Part="1"
-F 0 "R25" V 2693 1450 50  0000 C CNN
+F 0 "R27" V 2693 1450 50  0000 C CNN
 F 1 "10k" V 2784 1450 50  0000 C CNN
 F 2 "Resistor_SMD:R_0805_2012Metric" V 2830 1450 50  0001 C CNN
@@
 AR Path="/6224B28B/61C42A00" Ref="R?"  Part="1"
 AR Path="/622DADD3/622DC406/61C42A00" Ref="R?"  Part="1"
-AR Path="/622DADD3/62542111/61C42A00" Ref="R27"  Part="1"
+AR Path="/622DADD3/62542111/61C42A00" Ref="R29"  Part="1"
 AR Path="/62646A72/62542111/61C42A00" Ref="R?"  Part="1"
 AR Path="/62807237/62542111/61C42A00" Ref="R?"  Part="1"
@@
 AR Path="/6284E31C/62542111/61C42A00" Ref="R?"  Part="1"
 AR Path="/6284E336/62542111/61C42A00" Ref="R?"  Part="1"
-F 0 "R27" H 2320 2696 50  0000 L CNN
+F 0 "R29" H 2320 2696 50  0000 L CNN
 F 1 "2k" H 2320 2605 50  0000 L CNN
 F 2 "Resistor_SMD:R_0805_2012Metric" V 2180 2650 50  0001 C CNN
@@
 AR Path="/6224B28B/61C41765" Ref="R?"  Part="1"
 AR Path="/622DADD3/622DC406/61C41765" Ref="R?"  Part="1"
-AR Path="/622DADD3/62542111/61C41765" Ref="R28"  Part="1"
+AR Path="/622DADD3/62542111/61C41765" Ref="R30"  Part="1"
 AR Path="/62646A72/62542111/61C41765" Ref="R?"  Part="1"
 AR Path="/62807237/62542111/61C41765" Ref="R?"  Part="1"
@@
 AR Path="/6284E31C/62542111/61C41765" Ref="R?"  Part="1"
 AR Path="/6284E336/62542111/61C41765" Ref="R?"  Part="1"
-F 0 "R28" V 3000 3200 50  0000 C CNN
+F 0 "R30" V 3000 3200 50  0000 C CNN
 F 1 "10k" V 3100 3200 50  0000 C CNN
 F 2 "Resistor_SMD:R_0805_2012Metric" V 2830 3200 50  0001 C CNN
@@
 AR Path="/6224B28B/61C431CE" Ref="R?"  Part="1"
 AR Path="/622DADD3/622DC406/61C431CE" Ref="R?"  Part="1"
-AR Path="/622DADD3/62542111/61C431CE" Ref="R26"  Part="1"
+AR Path="/622DADD3/62542111/61C431CE" Ref="R28"  Part="1"
 AR Path="/62646A72/62542111/61C431CE" Ref="R?"  Part="1"
 AR Path="/62807237/62542111/61C431CE" Ref="R?"  Part="1"
@@
 AR Path="/6284E31C/62542111/61C431CE" Ref="R?"  Part="1"
 AR Path="/6284E336/62542111/61C431CE" Ref="R?"  Part="1"
-F 0 "R26" H 2320 1696 50  0000 L CNN
+F 0 "R28" H 2320 1696 50  0000 L CNN
 F 1 "2k" H 2320 1605 50  0000 L CNN
 F 2 "Resistor_SMD:R_0805_2012Metric" V 2180 1650 50  0001 C CNN
@@
 AR Path="/6284E336/62542111/62E5DD2B" Ref="C?"  Part="1"
 F 0 "C16" H 2650 2950 50  0000 L CNN
-F 1 "0.1uF" H 2650 2750 50  0000 L CNN
+F 1 "0.1u" H 2650 2750 50  0000 L CNN
 F 2 "Capacitor_SMD:C_0805_2012Metric" H 2638 2700 50  0001 C CNN
 F 3 "~" H 2600 2850 50  0001 C CNN
@@
 AR Path="/6284E336/62542111/62E6D056" Ref="C?"  Part="1"
 F 0 "C15" H 2650 1925 50  0000 L CNN
-F 1 "0.1uF" H 2650 1725 50  0000 L CNN
+F 1 "0.1u" H 2650 1725 50  0000 L CNN
 F 2 "Capacitor_SMD:C_0805_2012Metric" H 2638 1675 50  0001 C CNN
 F 3 "~" H 2600 1825 50  0001 C CNN
