File: hardware/kicad/emg-filter/ina_bandpass.sch (KiCad schematic (older format))
At the start: 16 parts, among them U45 INA2332, U46 LM4565

Commit message: Fixed errors
Changed lines of the file:
@@
 AR Path="/62498702/61EB8E9E" Ref="#PWR0187"  Part="1"
 AR Path="/62498720/61EB8E9E" Ref="#PWR0193"  Part="1"
-F 0 "#PWR0193" H 3350 4500 50  0001 C CNN
+F 0 "#PWR0151" H 3350 4500 50  0001 C CNN
 F 1 "-5V" H 3365 4573 50  0000 C CNN
 F 2 "" H 3350 4400 50  0001 C CNN
@@
 AR Path="/62498702/61EB8EB2" Ref="R309"  Part="1"
 AR Path="/62498720/61EB8EB2" Ref="R319"  Part="1"
-F 0 "R319" V 4050 3950 50  0000 L CNN
+F 0 "R249" V 4050 3950 50  0000 L CNN
 F 1 "191k" V 4150 3900 50  0000 L CNN
 F 2 "Resistor_SMD:R_0805_2012Metric" V 4180 4000 50  0001 C CNN
@@
 AR Path="/62498702/61EB8EBE" Ref="R311"  Part="1"
 AR Path="/62498720/61EB8EBE" Ref="R321"  Part="1"
-F 0 "R321" V 4450 3950 50  0000 L CNN
+F 0 "R251" V 4450 3950 50  0000 L CNN
 F 1 "10k" V 4550 3900 50  0000 L CNN
 F 2 "Resistor_SMD:R_0805_2012Metric" V 4580 4000 50  0001 C CNN
@@
 AR Path="/62498702/61EB8EC4" Ref="U57"  Part="1"
 AR Path="/62498720/61EB8EC4" Ref="U59"  Part="1"
-F 0 "U59" H 3100 4250 50  0000 C CNN
+F 0 "U45" H 3100 4250 50  0000 C CNN
 F 1 "INA2332" H 3550 4250 50  0000 C CNN
 F 2 "Package_SO:TSSOP-14_4.4x5mm_P0.65mm" H 3300 3800 50  0001 C CNN
@@
 AR Path="/62498702/61EB8ED8" Ref="R308"  Part="1"
 AR Path="/62498720/61EB8ED8" Ref="R318"  Part="1"
-F 0 "R318" V 4050 3550 50  0000 L CNN
+F 0 "R248" V 4050 3550 50  0000 L CNN
 F 1 "191k" V 4150 3500 50  0000 L CNN
 F 2 "Resistor_SMD:R_0805_2012Metric" V 4180 3600 50  0001 C CNN
@@
 AR Path="/62498702/61EB8EE5" Ref="#PWR0186"  Part="1"
 AR Path="/62498720/61EB8EE5" Ref="#PWR0192"  Part="1"
-F 0 "#PWR0192" H 3350 3050 50  0001 C CNN
+F 0 "#PWR0150" H 3350 3050 50  0001 C CNN
 F 1 "+5V" H 3365 3373 50  0000 C CNN
 F 2 "" H 3350 3200 50  0001 C CNN
@@
 AR Path="/62498702/61EB8EEF" Ref="R310"  Part="1"
 AR Path="/62498720/61EB8EEF" Ref="R320"  Part="1"
-F 0 "R320" V 4450 3550 50  0000 L CNN
+F 0 "R250" V 4450 3550 50  0000 L CNN
 F 1 "10k" V 4550 3500 50  0000 L CNN
 F 2 "Resistor_SMD:R_0805_2012Metric" V 4580 3600 50  0001 C CNN
@@
 AR Path="/62498702/620706D7" Ref="R315"  Part="1"
 AR Path="/62498720/620706D7" Ref="R325"  Part="1"
-F 0 "R325" V 6900 4400 50  0000 C CNN
+F 0 "R255" V 6900 4400 50  0000 C CNN
 F 1 "261k" V 7000 4400 50  0000 C CNN
 F 2 "Resistor_SMD:R_0805_2012Metric" V 6880 4200 50  0001 C CNN
@@
 AR Path="/62498702/620706D1" Ref="C205"  Part="1"
 AR Path="/62498720/620706D1" Ref="C211"  Part="1"
-F 0 "C211" V 6750 4250 50  0000 L CNN
+F 0 "C169" V 6750 4250 50  0000 L CNN
 F 1 "2n" V 6650 4250 50  0000 L CNN
 F 2 "Capacitor_SMD:C_0805_2012Metric" H 6738 4050 50  0001 C CNN
@@
 AR Path="/62498702/620706BF" Ref="U58"  Part="1"
 AR Path="/62498720/620706BF" Ref="U60"  Part="1"
-F 0 "U60" H 7400 4000 50  0000 C CNN
+F 0 "U46" H 7400 4000 50  0000 C CNN
 F 1 "LM4565" H 7750 4000 50  0000 C CNN
 F 2 "emg-filter:LM4565" H 8600 3700 50  0001 C CNN
@@
 AR Path="/62498702/620706B9" Ref="C207"  Part="1"
 AR Path="/62498720/620706B9" Ref="C213"  Part="1"
-F 0 "C213" V 7450 4250 50  0000 C CNN
+F 0 "C171" V 7450 4250 50  0000 C CNN
 F 1 "0.1u" V 7350 4300 50  0000 C CNN
 F 2 "Capacitor_SMD:C_0805_2012Metric" H 7438 4000 50  0001 C CNN
@@
 AR Path="/62498702/620706AF" Ref="#PWR0188"  Part="1"
 AR Path="/62498720/620706AF" Ref="#PWR0194"  Part="1"
-F 0 "#PWR0194" H 7150 4000 50  0001 C CNN
+F 0 "#PWR0152" H 7150 4000 50  0001 C CNN
 F 1 "GND" H 7250 4150 50  0000 C CNN
 F 2 "" H 7150 4250 50  0001 C CNN
@@
 AR Path="/62498702/620706A8" Ref="C206"  Part="1"
 AR Path="/62498720/620706A8" Ref="C212"  Part="1"
-F 0 "C212" V 7350 3150 50  0000 C CNN
+F 0 "C170" V 7350 3150 50  0000 C CNN
 F 1 "0.1u" V 7450 3100 50  0000 C CNN
 F 2 "Capacitor_SMD:C_0805_2012Metric" H 7438 3100 50  0001 C CNN
@@
 AR Path="/62498702/62070697" Ref="R314"  Part="1"
 AR Path="/62498720/62070697" Ref="R324"  Part="1"
-F 0 "R324" V 6900 3100 50  0000 C CNN
+F 0 "R254" V 6900 3100 50  0000 C CNN
 F 1 "261k" V 7000 3100 50  0000 C CNN
 F 2 "Resistor_SMD:R_0805_2012Metric" V 6880 3300 50  0001 C CNN
@@
 AR Path="/62498702/62070691" Ref="C204"  Part="1"
 AR Path="/62498720/62070691" Ref="C210"  Part="1"
-F 0 "C210" V 6750 3350 50  0000 L CNN
+F 0 "C168" V 6750 3350 50  0000 L CNN
 F 1 "2n" V 6650 3350 50  0000 L CNN
 F 2 "Capacitor_SMD:C_0805_2012Metric" H 6738 3150 50  0001 C CNN
@@
 AR Path="/62498702/6207068B" Ref="R313"  Part="1"
 AR Path="/62498720/6207068B" Ref="R323"  Part="1"
-F 0 "R323" V 6550 3900 50  0000 C CNN
+F 0 "R253" V 6550 3900 50  0000 C CNN
 F 1 "261k" V 6650 3900 50  0000 C CNN
 F 2 "Resistor_SMD:R_0805_2012Metric" V 6380 3900 50  0001 C CNN
@@
 AR Path="/62498702/62070685" Ref="C203"  Part="1"
 AR Path="/62498720/62070685" Ref="C209"  Part="1"
-F 0 "C209" V 6250 3900 50  0000 C CNN
+F 0 "C167" V 6250 3900 50  0000 C CNN
 F 1 "20n" V 6350 3900 50  0000 C CNN
 F 2 "Capacitor_SMD:C_0805_2012Metric" H 6138 3750 50  0001 C CNN
@@
 AR Path="/62498702/6207067F" Ref="R312"  Part="1"
 AR Path="/62498720/6207067F" Ref="R322"  Part="1"
-F 0 "R322" V 6250 3650 50  0000 C CNN
+F 0 "R252" V 6250 3650 50  0000 C CNN
 F 1 "261k" V 6350 3650 50  0000 C CNN
 F 2 "Resistor_SMD:R_0805_2012Metric" V 6380 3650 50  0001 C CNN
@@
 AR Path="/62498702/62070679" Ref="C202"  Part="1"
 AR Path="/62498720/62070679" Ref="C208"  Part="1"
-F 0 "C208" V 5850 3650 50  0000 C CNN
+F 0 "C166" V 5850 3650 50  0000 C CNN
 F 1 "20n" V 5950 3650 50  0000 C CNN
 F 2 "Capacitor_SMD:C_0805_2012Metric" H 6138 3500 50  0001 C CNN
@@
 AR Path="/62498702/62070673" Ref="#PWR0190"  Part="1"
 AR Path="/62498720/62070673" Ref="#PWR0196"  Part="1"
-F 0 "#PWR0196" H 7600 4300 50  0001 C CNN
+F 0 "#PWR0154" H 7600 4300 50  0001 C CNN
 F 1 "-5V" H 7500 4200 50  0000 C CNN
 F 2 "" H 7600 4200 50  0001 C CNN
@@
 AR Path="/62498702/6207066D" Ref="#PWR0189"  Part="1"
 AR Path="/62498720/6207066D" Ref="#PWR0195"  Part="1"
-F 0 "#PWR0195" H 7600 3050 50  0001 C CNN
+F 0 "#PWR0153" H 7600 3050 50  0001 C CNN
 F 1 "+5V" H 7700 3200 50  0000 C CNN
 F 2 "" H 7600 3200 50  0001 C CNN

Commit message: compact design
Parts:
- removed R248, R249: 191k, Resistor_SMD:R_0805_2012Metric, symbol Device:R
- removed R250, R251: 10k, Resistor_SMD:R_0805_2012Metric, symbol Device:R
- added C214, C215: 0.1u, Capacitor_SMD:C_0805_2012Metric, symbol Device:C
- added R328, R331: 191k, Resistor_SMD:R_0805_2012Metric, symbol Device:R
- added R329, R330: 10k, Resistor_SMD:R_0805_2012Metric, symbol Device:R
- renumbered C166 to C216, C167 to C217, C168 to C218, C169 to C219, C170 to C220, C171 to C221, R252 to R332, R253 to R333, R254 to R334, R255 to R335
Connections:
- wire segments 80 -> 87
Other:
- moved on the sheet: C272, C273

Commit message: Isolating module
Parts:
- renumbered C214 to C17, C220 to C18, C218 to C19, C216 to C20, C217 to C21, C221 to C22, C219 to C23, C215 to C24, R334 to R29, R328 to R30, R329 to R31, R332 to R32, R333 to R33, R330 to R34, R331 to R35, R335 to R36, U46 to U6, U45 to U7

Commit message: Update pcb module
Parts:
- renumbered C23 to C22, C22 to C23, R29 to R31, R30 to R32, R31 to R33, R32 to R34, R33 to R35, R34 to R36, R35 to R37, R36 to R38
Other:
- moved on the sheet: C23

Commit message: fixed length
Other:
- moved on the sheet: C17, C18, C19, C20, C21, C22, C23, C24, R31, R32, R33, R34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

Commit message: Amplifier done
Other:
- moved on the sheet: C17, C18, C19, C20, C21, C22, C23, C24, R31, R32, R33, R34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
