File: hardware/kicad/emg-filter/ina_bandpass.sch (KiCad schematic (older format))
At the start: 18 parts, among them U6 LM4565, U7 INA2332

Commit message: Done - Ready for manufacturing
Parts:
- renumbered C24 to C10, C17 to C3, C18 to C4, C19 to C5, C20 to C6, C21 to C7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
