File: hardware/kicad/emg-filter/ina_bandpass.sch (KiCad schematic (older format))
At the start: 18 parts, among them U45 INA2332, U46 LM4565

Commit message: update
Parts:
- renumbered C214 to C30, C220 to C31, C218 to C32, C216 to C33, C217 to C34, C221 to C35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
