File: hardware/kicad/emg-filter/notch_rect.sch (KiCad schematic (older format))
At the start: 24 parts, among them U1 LM4565, U2 LM4565

Commit message: update
Other:
- moved on the sheet: C1, C2, C3, C4, C5, C6, C7, D1, D2, R1, R10, R11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

Commit message: update
Other:
- moved on the sheet: C1, C2, C3, C4, C5, C6, C7, D1, D2, R1, R10, R11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

Commit message: Done - Ready for manufacturing
Parts:
- renumbered C1 to C11, C2 to C12, C3 to C13, C4 to C14, C5 to C15, C6 to C16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
