File: hardware/kicad/emg-filter/notch_rect.sch (KiCad schematic (older format))
At the start: 24 parts, among them U4 LM4565, U5 LM4565

Commit message: Updated diode footprint
and changed 5k to 4.99k resistor
reason: 4.99k resistor are less expensive and won't affect the output of the design
Parts:
- R25: value 5k -> 4.99k
