File: hardware/kicad/emg-filter/notch_rect.sch (KiCad schematic (older format))
At the start: 21 parts, among them U40 LM4565, U41 LM4565

Commit message: Fixed errors
Changed lines of the file:
@@
 $Descr A4 11693 8268
 encoding utf-8
-Sheet 14 43
+Sheet 3 43
 Title ""
 Date ""
@@
 AR Path="/6224B28F/621836B0" Ref="R44"  Part="1"
 AR Path="/6224B2A9/621836B0" Ref="R32"  Part="1"
-F 0 "R240" V 7557 2250 50  0000 C CNN
+F 0 "R32" V 7557 2250 50  0000 C CNN
 F 1 "10k" V 7466 2250 50  0000 C CNN
 F 2 "Resistor_SMD:R_0805_2012Metric" V 7280 2250 50  0001 C CNN
@@
 AR Path="/6224B28F/621836B6" Ref="R45"  Part="1"
 AR Path="/6224B2A9/621836B6" Ref="R33"  Part="1"
-F 0 "R241" V 7143 3150 50  0000 C CNN
+F 0 "R33" V 7143 3150 50  0000 C CNN
 F 1 "5k" V 7234 3150 50  0000 C CNN
 F 2 "Resistor_SMD:R_0805_2012Metric" V 7280 3150 50  0001 C CNN
@@
 AR Path="/6224B28F/621836BC" Ref="R42"  Part="1"
 AR Path="/6224B2A9/621836BC" Ref="R30"  Part="1"
-F 0 "R238" V 5657 2850 50  0000 C CNN
+F 0 "R30" V 5657 2850 50  0000 C CNN
 F 1 "10k" V 5566 2850 50  0000 C CNN
 F 2 "Resistor_SMD:R_0805_2012Metric" V 5380 2850 50  0001 C CNN
@@
 AR Path="/6224B28F/621836C2" Ref="D8"  Part="1"
 AR Path="/6224B2A9/621836C2" Ref="D6"  Part="1"
-F 0 "D36" H 6850 2400 50  0000 C CNN
+F 0 "D6" H 6850 2400 50  0000 C CNN
 F 1 "1N4148" H 6950 2300 50  0000 C CNN
 F 2 "Diode_SMD:D_SOD-323" H 6900 2500 50  0001 C CNN
@@
 AR Path="/6224B28F/621836C8" Ref="D7"  Part="1"
 AR Path="/6224B2A9/621836C8" Ref="D5"  Part="1"
-F 0 "D35" V 6604 2330 50  0000 L CNN
+F 0 "D5" V 6604 2330 50  0000 L CNN
 F 1 "1N4148" V 6695 2330 50  0000 L CNN
 F 2 "Diode_SMD:D_SOD-323" H 6650 2250 50  0001 C CNN
@@
 AR Path="/6224B28F/621836CE" Ref="R43"  Part="1"
 AR Path="/6224B2A9/621836CE" Ref="R31"  Part="1"
-F 0 "R239" V 6857 3150 50  0000 C CNN
+F 0 "R31" V 6857 3150 50  0000 C CNN
 F 1 "10k" V 6766 3150 50  0000 C CNN
 F 2 "Resistor_SMD:R_0805_2012Metric" V 6580 3150 50  0001 C CNN
@@
 AR Path="/6224B28F/621836D5" Ref="R41"  Part="1"
 AR Path="/6224B2A9/621836D5" Ref="R29"  Part="1"
-F 0 "R237" V 5657 2550 50  0000 C CNN
+F 0 "R29" V 5657 2550 50  0000 C CNN
 F 1 "10k" V 5566 2550 50  0000 C CNN
 F 2 "Resistor_SMD:R_0805_2012Metric" V 5380 2550 50  0001 C CNN
@@
 AR Path="/6224B28F/621836E0" Ref="U6"  Part="1"
 AR Path="/6224B2A9/621836E0" Ref="U4"  Part="1"
-F 0 "U41" H 6400 2300 50  0000 C CNN
+F 0 "U4" H 6400 2300 50  0000 C CNN
 F 1 "LM4565" H 6350 2950 50  0000 C CNN
 F 2 "emg-filter:LM4565" H 7200 2650 50  0001 C CNN
@@
 AR Path="/6224B28F/621836EC" Ref="#PWR023"  Part="1"
 AR Path="/6224B2A9/621836EC" Ref="#PWR017"  Part="1"
-F 0 "#PWR0135" H 5700 2950 50  0001 C CNN
+F 0 "#PWR017" H 5700 2950 50  0001 C CNN
 F 1 "GND" H 5600 3200 50  0000 C CNN
 F 2 "" H 5700 3200 50  0001 C CNN
@@
 AR Path="/6224B28F/621836F2" Ref="#PWR025"  Part="1"
 AR Path="/6224B2A9/621836F2" Ref="#PWR019"  Part="1"
-F 0 "#PWR0137" H 6200 3300 50  0001 C CNN
+F 0 "#PWR019" H 6200 3300 50  0001 C CNN
 F 1 "-5V" H 6215 3373 50  0000 C CNN
 F 2 "" H 6200 3200 50  0001 C CNN
@@
 AR Path="/6224B28F/621836F8" Ref="#PWR024"  Part="1"
 AR Path="/6224B2A9/621836F8" Ref="#PWR018"  Part="1"
-F 0 "#PWR0136" H 6200 2050 50  0001 C CNN
+F 0 "#PWR018" H 6200 2050 50  0001 C CNN
 F 1 "+5V" H 6215 2373 50  0000 C CNN
 F 2 "" H 6200 2200 50  0001 C CNN
@@
 AR Path="/6224B28F/621836FE" Ref="C87"  Part="1"
 AR Path="/6224B2A9/621836FE" Ref="C82"  Part="1"
-F 0 "C157" V 5950 2950 50  0000 C CNN
+F 0 "C82" V 5950 2950 50  0000 C CNN
 F 1 "0.1u" V 5850 3100 50  0000 C CNN
 F 2 "Capacitor_SMD:C_0805_2012Metric" H 6038 2950 50  0001 C CNN
@@
 AR Path="/6224B28F/6218370C" Ref="C86"  Part="1"
 AR Path="/6224B2A9/6218370C" Ref="C81"  Part="1"
-F 0 "C156" V 5900 2100 50  0000 C CNN
+F 0 "C81" V 5900 2100 50  0000 C CNN
 F 1 "0.1u" V 5800 2250 50  0000 C CNN
 F 2 "Capacitor_SMD:C_0805_2012Metric" H 5988 2100 50  0001 C CNN
@@
 AR Path="/6224B28F/62183732" Ref="R38"  Part="1"
 AR Path="/6224B2A9/62183732" Ref="R26"  Part="1"
-F 0 "R234" V 3675 2700 50  0000 C CNN
+F 0 "R26" V 3675 2700 50  0000 C CNN
 F 1 "133k" V 3575 2700 50  0000 C CNN
 F 2 "Resistor_SMD:R_0805_2012Metric" V 3405 2700 50  0001 C CNN
@@
 AR Path="/6224B28F/62183739" Ref="R37"  Part="1"
 AR Path="/6224B2A9/62183739" Ref="R25"  Part="1"
-F 0 "R233" V 3350 2700 50  0000 C CNN
+F 0 "R25" V 3350 2700 50  0000 C CNN
 F 1 "133k" V 3250 2700 50  0000 C CNN
 F 2 "Resistor_SMD:R_0805_2012Metric" V 3080 2700 50  0001 C CNN
@@
 AR Path="/6224B28F/62183744" Ref="R35"  Part="1"
 AR Path="/6224B2A9/62183744" Ref="R23"  Part="1"
-F 0 "R231" V 2950 2650 50  0000 L CNN
+F 0 "R23" V 2950 2650 50  0000 L CNN
 F 1 "132k" V 2850 2600 50  0000 L CNN
 F 2 "Resistor_SMD:R_0805_2012Metric" V 2680 2700 50  0001 C CNN
@@
 AR Path="/6224B28F/6218374D" Ref="R34"  Part="1"
 AR Path="/6224B2A9/6218374D" Ref="R22"  Part="1"
-F 0 "R230" V 2625 2650 50  0000 L CNN
+F 0 "R22" V 2625 2650 50  0000 L CNN
 F 1 "132k" V 2525 2600 50  0000 L CNN
 F 2 "Resistor_SMD:R_0805_2012Metric" V 2355 2700 50  0001 C CNN
@@
 AR Path="/6224B28F/62183756" Ref="#PWR021"  Part="1"
 AR Path="/6224B2A9/62183756" Ref="#PWR015"  Part="1"
-F 0 "#PWR0133" H 4275 3450 50  0001 C CNN
+F 0 "#PWR015" H 4275 3450 50  0001 C CNN
 F 1 "-5V" H 4290 3523 50  0000 C CNN
 F 2 "" H 4275 3350 50  0001 C CNN
@@
 AR Path="/6224B28F/6218375C" Ref="#PWR020"  Part="1"
 AR Path="/6224B2A9/6218375C" Ref="#PWR014"  Part="1"
-F 0 "#PWR0132" H 4275 2225 50  0001 C CNN
+F 0 "#PWR014" H 4275 2225 50  0001 C CNN
 F 1 "+5V" H 4290 2548 50  0000 C CNN
 F 2 "" H 4275 2375 50  0001 C CNN
@@
 AR Path="/6224B28F/62183763" Ref="R40"  Part="1"
 AR Path="/6224B2A9/62183763" Ref="R28"  Part="1"
-F 0 "R236" H 4995 3346 50  0000 L CNN
+F 0 "R28" H 4995 3346 50  0000 L CNN
 F 1 "266k" H 4995 3255 50  0000 L CNN
 F 2 "Resistor_SMD:R_0805_2012Metric" V 4855 3300 50  0001 C CNN
@@
 AR Path="/6224B28F/62183769" Ref="R39"  Part="1"
 AR Path="/6224B2A9/62183769" Ref="R27"  Part="1"
-F 0 "R235" H 4995 2946 50  0000 L CNN
+F 0 "R27" H 4995 2946 50  0000 L CNN
 F 1 "2k" H 4995 2855 50  0000 L CNN
 F 2 "Resistor_SMD:R_0805_2012Metric" V 4855 2900 50  0001 C CNN
@@
 AR Path="/6224B28F/62183771" Ref="#PWR022"  Part="1"
 AR Path="/6224B2A9/62183771" Ref="#PWR016"  Part="1"
-F 0 "#PWR0134" H 4925 3250 50  0001 C CNN
+F 0 "#PWR016" H 4925 3250 50  0001 C CNN
 F 1 "GND" H 4930 3327 50  0000 C CNN
 F 2 "" H 4925 3500 50  0001 C CNN
@@
 AR Path="/6224B28F/62183787" Ref="C85"  Part="1"
 AR Path="/6224B2A9/62183787" Ref="C80"  Part="1"
-F 0 "C155" V 3223 3100 50  0000 C CNN
+F 0 "C80" V 3223 3100 50  0000 C CNN
 F 1 "10n" V 3314 3100 50  0000 C CNN
 F 2 "Capacitor_SMD:C_0805_2012Metric" H 3513 2950 50  0001 C CNN
@@
 AR Path="/6224B28F/6218378D" Ref="C83"  Part="1"
 AR Path="/6224B2A9/6218378D" Ref="C78"  Part="1"
-F 0 "C153" V 2173 3100 50  0000 C CNN
+F 0 "C78" V 2173 3100 50  0000 C CNN
 F 1 "10n" V 2264 3100 50  0000 C CNN
 F 2 "Capacitor_SMD:C_0805_2012Metric" H 2463 2950 50  0001 C CNN
@@
 AR Path="/6224B28F/62183793" Ref="C84"  Part="1"
 AR Path="/6224B2A9/62183793" Ref="C79"  Part="1"
-F 0 "C154" H 2835 3304 50  0000 R CNN
+F 0 "C79" H 2835 3304 50  0000 R CNN
 F 1 "20n" H 2835 3395 50  0000 R CNN
 F 2 "Capacitor_SMD:C_0805_2012Metric" H 2988 3200 50  0001 C CNN
@@
 AR Path="/6224B28F/62183799" Ref="R36"  Part="1"
 AR Path="/6224B2A9/62183799" Ref="R24"  Part="1"
-F 0 "R232" H 2681 3304 50  0000 R CNN
+F 0 "R24" H 2681 3304 50  0000 R CNN
 F 1 "133k" H 2681 3395 50  0000 R CNN
 F 2 "Resistor_SMD:R_0805_2012Metric" V 2680 3350 50  0001 C CNN
@@
 AR Path="/6224B28F/6218379F" Ref="U5"  Part="1"
 AR Path="/6224B2A9/6218379F" Ref="U3"  Part="1"
-F 0 "U40" H 4075 3150 50  0000 C CNN
+F 0 "U3" H 4075 3150 50  0000 C CNN
 F 1 "LM4565" H 4425 3150 50  0000 C CNN
 F 2 "emg-filter:LM4565" H 5275 2850 50  0001 C CNN

Commit message: compact design
Parts:
- removed C153, C155: 10n, Capacitor_SMD:C_0805_2012Metric, symbol Device:C
- removed C154: 20n, Capacitor_SMD:C_0805_2012Metric, symbol Device:C
- removed R230, R231: 132k, Resistor_SMD:R_0805_2012Metric, symbol Device:R
- removed R232, R233, R234: 133k, Resistor_SMD:R_0805_2012Metric, symbol Device:R
- added C202, C203: 0.1u, Capacitor_SMD:C_0805_2012Metric, symbol Device:C
- added C? (x2): 10n, Capacitor_SMD:C_0805_2012Metric, symbol Device:C
- added C?: 20n, Capacitor_SMD:C_0805_2012Metric, symbol Device:C
- added R? (x3): 133k, Resistor_SMD:R_0805_2012Metric, symbol Device:R
- added R? (x2): 132k, Resistor_SMD:R_0805_2012Metric, symbol Device:R
- renumbered C156 to C204, C157 to C205, R235 to R315, R236 to R316, R237 to R317, R238 to R318, R239 to R319, R240 to R320, R241 to R321
Connections:
- wire segments 82 -> 85
Other:
- moved on the sheet: C96, C97, D11, D12, R87, R88, R89, R90, R91, R92, R93, U10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

Commit message: Annotation
Parts:
- gave numbers to parts that had none: 8
