File: hardware/kicad/emg-filter/emg-filter.sch (KiCad schematic (older format))
At the start: 62 parts, among them J10 Conn_01x02, J11 Conn_01x02, J12 Conn_01x02, J13 Conn_01x02, J14 Conn_01x05, J15 Conn_01x05, J16 Conn_01x02, J17 Conn_01x02, J18 Conn_01x02, J19 Conn_01x02, J20 Conn_01x02, J21 Conn_01x02, J22 Conn_01x05, J23 Conn_01x05, J24 Conn_01x02, J25 Conn_01x02, J26 Conn_01x02, J27 Conn_01x02, J28 Conn_01x02, J29 Conn_01x02, J30 Conn_01x05, J31 Conn_01x05, J32 Conn_01x02, J33 Conn_01x02, J34 Conn_01x02, J35 Conn_01x02, J36 Conn_01x02, J37 Conn_01x02, J38 Conn_01x05, J39 Conn_01x05, J4 Conn_01x02, J40 Conn_01x02, J41 Conn_01x02, J42 Conn_01x02, J43 Conn_01x02, J44 Conn_01x02, J45 Conn_01x02, J46 Conn_01x05, J47 Conn_01x05, J48 Conn_01x02, J49 Conn_01x02, J5 Conn_01x02, J50 Conn_01x02, J51 Conn_01x02, J52 Conn_01x02, J53 Conn_01x02, J54 Conn_01x05, J55 Conn_01x05, J56 Conn_01x02, J57 Conn_01x02, J58 Conn_01x02, J59 Conn_01x02, J6 Conn_01x05, J60 Conn_01x02, J61 Conn_01x02, J62 Conn_01x05, J63 Conn_01x05, J64 Conn_01x02, J65 Conn_01x02, J7 Conn_01x05, J8 Conn_01x02, J9 Conn_01x02

Commit message: Isolating module
Parts:
- removed J10, J11, J12, J13, J16, J17, J18, J19, J20, J21, J24, J25, J26, J27, J28, J29, J32, J33, J34, J35, J36, J37, J4, J40, J41, J42, J43, J44, J45, J48, J49, J50, J51, J52, J53, J56, J57, J58, J59, J60, J61, J64, J65, J8: Conn_01x02, symbol Connector_Generic:Conn_01x02
- removed J14, J15, J22, J23, J30, J31, J38, J39, J46, J47, J54, J55, J62, J63, J7: Conn_01x05, symbol Connector_Generic:Conn_01x05
- renumbered J5 to J1, J6 to J2, J9 to J3
Connections:
- net labels removed: +5V, -5V, GND
- wire segments 156 -> 0
- no-connect marks 4 -> 0
Other:
- note removed: "EMG Filter for Prosthetic Limb Control System"
- note removed: "Female\n2-pin\nheader"
- note removed: "Male Jumper header"

Commit message: Update pcb module
Parts:
- J1, J3: footprint (none) -> Connector_PinHeader_2.54mm:PinHeader_1x02_P2.54mm_Vertical
- J2: footprint (none) -> Connector_PinHeader_2.54mm:PinHeader_1x05_P2.54mm_Vertical
Changed lines of the file:
@@
 F 0 "J2" H 4725 1400 50  0000 L CNN
 F 1 "Conn_01x05" H 4725 1300 50  0000 L CNN
-F 2 "" H 4775 1000 50  0001 C CNN
+F 2 "Connector_PinHeader_2.54mm:PinHeader_1x05_P2.54mm_Vertical" H 4775 1000 50  0001 C CNN
 F 3 "~" H 4775 1000 50  0001 C CNN
 	1    4775 1000
@@
 F 0 "J1" H 3600 1000 50  0000 R CNN
 F 1 "Conn_01x02" H 3950 900 50  0000 R CNN
-F 2 "" H 3550 800 50  0001 C CNN
+F 2 "Connector_PinHeader_2.54mm:PinHeader_1x02_P2.54mm_Vertical" H 3550 800 50  0001 C CNN
 F 3 "~" H 3550 800 50  0001 C CNN
 	1    3550 800
@@
 F 0 "J3" H 3600 800 50  0000 R CNN
 F 1 "Conn_01x02" H 3950 900 50  0000 R CNN
-F 2 "" H 3550 1100 50  0001 C CNN
+F 2 "Connector_PinHeader_2.54mm:PinHeader_1x02_P2.54mm_Vertical" H 3550 1100 50  0001 C CNN
 F 3 "~" H 3550 1100 50  0001 C CNN
 	1    3550 1100

Commit message: fixed length
Changed lines of the file:
@@
 F4 "REF_A" I L 3750 900 50
 F5 "REF_B" I L 3750 1200 50
-F6 "OUT_A" I R 4575 800 50
-F7 "OUT_B" I R 4575 900 50
-F8 "+5V" I R 4575 1000 50
-F9 "-5V" I R 4575 1200 50
-F10 "GND" I R 4575 1100 50
+F6 "OUT_A" I R 4575 900 50
+F7 "OUT_B" I R 4575 1100 50
+F8 "+5V" I R 4575 1200 50
+F9 "-5V" I R 4575 800 50
+F10 "GND" I R 4575 1000 50
 $EndSheet
 $Comp

Commit message: Amplifier done
Changed lines of the file:
@@
 F6 "OUT_A" I R 4575 900 50
 F7 "OUT_B" I R 4575 1100 50
-F8 "+5V" I R 4575 1200 50
-F9 "-5V" I R 4575 800 50
+F8 "+5V" I R 4575 800 50
+F9 "-5V" I R 4575 1200 50
 F10 "GND" I R 4575 1000 50
 $EndSheet

Commit message: aligning pins to fit on motherboard
Changed lines of the file:
@@
 F1 "emg_module.sch" 50
 F2 "VIN_A" I L 3750 800 50
-F3 "VIN_B" I L 3750 1100 50
+F3 "VIN_B" I L 3750 1200 50
 F4 "REF_A" I L 3750 900 50
-F5 "REF_B" I L 3750 1200 50
+F5 "REF_B" I L 3750 1100 50
 F6 "OUT_A" I R 4575 900 50
 F7 "OUT_B" I R 4575 1100 50

Commit message: fixed shematic
Changed lines of the file:
@@
 F0 "emg_module" 50
 F1 "emg_module.sch" 50
-F2 "VIN_A" I L 3750 800 50
-F3 "VIN_B" I L 3750 1200 50
+F2 "+VIN_A" I L 3750 800 50
+F3 "-VIN_B" I L 3750 1200 50
 F4 "REF_A" I L 3750 900 50
 F5 "REF_B" I L 3750 1100 50
