File: hardware/kicad/emg-filter/emg-filter.sch (KiCad schematic (older format))
At the start: 62 parts, among them J10 Conn_01x02, J11 Conn_01x02, J12 Conn_01x02, J13 Conn_01x02, J14 Conn_01x05, J15 Conn_01x05, J16 Conn_01x02, J17 Conn_01x02, J18 Conn_01x02, J19 Conn_01x02, J20 Conn_01x02, J21 Conn_01x02, J22 Conn_01x05, J23 Conn_01x05, J24 Conn_01x02, J25 Conn_01x02, J26 Conn_01x02, J27 Conn_01x02, J28 Conn_01x02, J29 Conn_01x02, J30 Conn_01x05, J31 Conn_01x05, J32 Conn_01x02, J33 Conn_01x02, J34 Conn_01x02, J35 Conn_01x02, J36 Conn_01x02, J37 Conn_01x02, J38 Conn_01x05, J39 Conn_01x05, J4 Conn_01x02, J40 Conn_01x02, J41 Conn_01x02, J42 Conn_01x02, J43 Conn_01x02, J44 Conn_01x02, J45 Conn_01x02, J46 Conn_01x05, J47 Conn_01x05, J48 Conn_01x02, J49 Conn_01x02, J5 Conn_01x02, J50 Conn_01x02, J51 Conn_01x02, J52 Conn_01x02, J53 Conn_01x02, J54 Conn_01x05, J55 Conn_01x05, J56 Conn_01x02, J57 Conn_01x02, J58 Conn_01x02, J59 Conn_01x02, J6 Conn_01x05, J60 Conn_01x02, J61 Conn_01x02, J62 Conn_01x05, J63 Conn_01x05, J64 Conn_01x02, J65 Conn_01x02, J7 Conn_01x05, J8 Conn_01x02, J9 Conn_01x02

Commit message: Update wiring
Connections:
- wire segments 156 -> 160

Commit message: changed local lib path
Parts:
- removed J13, J17, J21, J25, J29, J33, J37, J41, J45, J49, J5, J53, J57, J61, J65, J9: Conn_01x02, symbol Connector_Generic:Conn_01x02
- removed J14, J22, J30, J39, J46, J55, J6, J62: Conn_01x05, symbol Connector_Generic:Conn_01x05
Other:
- note removed: "Male\n2-pin\nheader"

Commit message: update
Parts:
- renumbered J4 to J1, J19 to J10, J20 to J11, J23 to J12, J24 to J13, J26 to J14, J27 to J15, J28 to J16, J31 to J17, J32 to J18, J34 to J19, J7 to J2, J35 to J20, J36 to J21, J38 to J22, J40 to J23, J42 to J24, J43 to J25, J44 to J26, J47 to J27, J48 to J28, J50 to J29, J8 to J3, J51 to J30, J52 to J31, J54 to J32, J56 to J33, J58 to J34, J59 to J35, J60 to J36, J63 to J37, J64 to J38, J10 to J4, J11 to J5, J12 to J6, J15 to J7, J16 to J8, J18 to J9

Commit message: Update
Parts:
- removed J1, J10, J11, J13, J14, J15, J16, J18, J19, J20, J21, J23, J24, J25, J26, J28, J29, J3, J30, J31, J33, J34, J35, J36, J38, J4, J5, J6, J8, J9: Conn_01x02, symbol Connector_Generic:Conn_01x02
- removed J12, J17, J2, J22, J27, J32, J37, J7: Conn_01x05, symbol Connector_Generic:Conn_01x05
Connections:
- net labels removed: +5V, -5V, GND
- wire segments 160 -> 144
Other:
- note removed: "Female\n2-pin\nheader"
- note removed: "Male Jumper header"
