File: hardware/kicad/emg-filter/emg_module.sch (KiCad schematic (older format))
At the start: 0 parts

Commit message: Isolating module
Changed lines of the file:
@@
 $Descr A4 11693 8268
 encoding utf-8
-Sheet 3 51
+Sheet 2 7
 Title ""
 Date ""
@@
 AR Path="/61C38667/62542157" Ref="#PWR?"  Part="1"
 AR Path="/62542157" Ref="#PWR?"  Part="1"
-AR Path="/622DADD3/62542157" Ref="#PWR0159"  Part="1"
-AR Path="/62646A72/62542157" Ref="#PWR0190"  Part="1"
-AR Path="/62807237/62542157" Ref="#PWR0221"  Part="1"
-AR Path="/62807263/62542157" Ref="#PWR0252"  Part="1"
-AR Path="/6284E2B1/62542157" Ref="#PWR0283"  Part="1"
-AR Path="/6284E2DD/62542157" Ref="#PWR0314"  Part="1"
-AR Path="/6284E31C/62542157" Ref="#PWR0345"  Part="1"
-AR Path="/6284E336/62542157" Ref="#PWR0376"  Part="1"
-F 0 "#PWR0159" H 6675 3925 50  0001 C CNN
+AR Path="/622DADD3/62542157" Ref="#PWR05"  Part="1"
+AR Path="/62646A72/62542157" Ref="#PWR?"  Part="1"
+AR Path="/62807237/62542157" Ref="#PWR?"  Part="1"
+AR Path="/62807263/62542157" Ref="#PWR?"  Part="1"
+AR Path="/6284E2B1/62542157" Ref="#PWR?"  Part="1"
+AR Path="/6284E2DD/62542157" Ref="#PWR?"  Part="1"
+AR Path="/6284E31C/62542157" Ref="#PWR?"  Part="1"
+AR Path="/6284E336/62542157" Ref="#PWR?"  Part="1"
+F 0 "#PWR05" H 6675 3925 50  0001 C CNN
 F 1 "GND" H 6675 4025 50  0000 C CNN
 F 2 "" H 6675 4175 50  0001 C CNN
@@
 AR Path="/61C38667/6254215D" Ref="#PWR?"  Part="1"
 AR Path="/6254215D" Ref="#PWR?"  Part="1"
-AR Path="/622DADD3/6254215D" Ref="#PWR0160"  Part="1"
-AR Path="/62646A72/6254215D" Ref="#PWR0191"  Part="1"
-AR Path="/62807237/6254215D" Ref="#PWR0222"  Part="1"
-AR Path="/62807263/6254215D" Ref="#PWR0253"  Part="1"
-AR Path="/6284E2B1/6254215D" Ref="#PWR0284"  Part="1"
-AR Path="/6284E2DD/6254215D" Ref="#PWR0315"  Part="1"
-AR Path="/6284E31C/6254215D" Ref="#PWR0346"  Part="1"
-AR Path="/6284E336/6254215D" Ref="#PWR0377"  Part="1"
-F 0 "#PWR0160" H 6500 4025 50  0001 C CNN
+AR Path="/622DADD3/6254215D" Ref="#PWR04"  Part="1"
+AR Path="/62646A72/6254215D" Ref="#PWR?"  Part="1"
+AR Path="/62807237/6254215D" Ref="#PWR?"  Part="1"
+AR Path="/62807263/6254215D" Ref="#PWR?"  Part="1"
+AR Path="/6284E2B1/6254215D" Ref="#PWR?"  Part="1"
+AR Path="/6284E2DD/6254215D" Ref="#PWR?"  Part="1"
+AR Path="/6284E31C/6254215D" Ref="#PWR?"  Part="1"
+AR Path="/6284E336/6254215D" Ref="#PWR?"  Part="1"
+F 0 "#PWR04" H 6500 4025 50  0001 C CNN
 F 1 "+5V" H 6525 4325 50  0000 C CNN
 F 2 "" H 6500 4175 50  0001 C CNN
@@
 AR Path="/61C38667/62542163" Ref="#PWR?"  Part="1"
 AR Path="/62542163" Ref="#PWR?"  Part="1"
-AR Path="/622DADD3/62542163" Ref="#PWR0161"  Part="1"
-AR Path="/62646A72/62542163" Ref="#PWR0192"  Part="1"
-AR Path="/62807237/62542163" Ref="#PWR0223"  Part="1"
-AR Path="/62807263/62542163" Ref="#PWR0254"  Part="1"
-AR Path="/6284E2B1/62542163" Ref="#PWR0285"  Part="1"
-AR Path="/6284E2DD/62542163" Ref="#PWR0316"  Part="1"
-AR Path="/6284E31C/62542163" Ref="#PWR0347"  Part="1"
-AR Path="/6284E336/62542163" Ref="#PWR0378"  Part="1"
-F 0 "#PWR0161" H 6850 4275 50  0001 C CNN
+AR Path="/622DADD3/62542163" Ref="#PWR06"  Part="1"
+AR Path="/62646A72/62542163" Ref="#PWR?"  Part="1"
+AR Path="/62807237/62542163" Ref="#PWR?"  Part="1"
+AR Path="/62807263/62542163" Ref="#PWR?"  Part="1"
+AR Path="/6284E2B1/62542163" Ref="#PWR?"  Part="1"
+AR Path="/6284E2DD/62542163" Ref="#PWR?"  Part="1"
+AR Path="/6284E31C/62542163" Ref="#PWR?"  Part="1"
+AR Path="/6284E336/62542163" Ref="#PWR?"  Part="1"
+F 0 "#PWR06" H 6850 4275 50  0001 C CNN
 F 1 "-5V" H 6850 4325 50  0000 C CNN
 F 2 "" H 6850 4175 50  0001 C CNN
@@
 Text Notes 2825 3200 0    50   ~ 0
 Male 2-pin header
+$Comp
+L power:+5V #PWR?
+U 1 1 61F618C9
+P 2000 2575
+AR Path="/61C38667/61F618C9" Ref="#PWR?"  Part="1"
+AR Path="/61F618C9" Ref="#PWR?"  Part="1"
+AR Path="/622DADD3/61F618C9" Ref="#PWR01"  Part="1"
+AR Path="/62646A72/61F618C9" Ref="#PWR?"  Part="1"
+AR Path="/62807237/61F618C9" Ref="#PWR?"  Part="1"
+AR Path="/62807263/61F618C9" Ref="#PWR?"  Part="1"
+AR Path="/6284E2B1/61F618C9" Ref="#PWR?"  Part="1"
+AR Path="/6284E2DD/61F618C9" Ref="#PWR?"  Part="1"
+AR Path="/6284E31C/61F618C9" Ref="#PWR?"  Part="1"
+AR Path="/6284E336/61F618C9" Ref="#PWR?"  Part="1"
+F 0 "#PWR01" H 2000 2425 50  0001 C CNN
+F 1 "+5V" H 2025 2725 50  0000 C CNN
+F 2 "" H 2000 2575 50  0001 C CNN
+F 3 "" H 2000 2575 50  0001 C CNN
+	1    2000 2575
+	1    0    0    -1
+$EndComp
+$Comp
+L power:-5V #PWR?
+U 1 1 61F62396
+P 2900 2575
+AR Path="/61C38667/61F62396" Ref="#PWR?"  Part="1"
+AR Path="/61F62396" Ref="#PWR?"  Part="1"
+AR Path="/622DADD3/61F62396" Ref="#PWR03"  Part="1"
+AR Path="/62646A72/61F62396" Ref="#PWR?"  Part="1"
+AR Path="/62807237/61F62396" Ref="#PWR?"  Part="1"
+AR Path="/62807263/61F62396" Ref="#PWR?"  Part="1"
+AR Path="/6284E2B1/61F62396" Ref="#PWR?"  Part="1"
+AR Path="/6284E2DD/61F62396" Ref="#PWR?"  Part="1"
+AR Path="/6284E31C/61F62396" Ref="#PWR?"  Part="1"
+AR Path="/6284E336/61F62396" Ref="#PWR?"  Part="1"
+F 0 "#PWR03" H 2900 2675 50  0001 C CNN
+F 1 "-5V" H 2900 2725 50  0000 C CNN
+F 2 "" H 2900 2575 50  0001 C CNN
+F 3 "" H 2900 2575 50  0001 C CNN
+	1    2900 2575
+	1    0    0    -1
+$EndComp
+$Comp
+L power:PWR_FLAG #FLG01
+U 1 1 61F62BE9
+P 2000 2575
+F 0 "#FLG01" H 2000 2650 50  0001 C CNN
+F 1 "PWR_FLAG" H 2000 2748 50  0000 C CNN
+F 2 "" H 2000 2575 50  0001 C CNN
+F 3 "~" H 2000 2575 50  0001 C CNN
+	1    2000 2575
+	-1   0    0    1
+$EndComp
+$Comp
+L power:PWR_FLAG #FLG03
+U 1 1 61F6348C
+P 2900 2575
+F 0 "#FLG03" H 2900 2650 50  0001 C CNN
+F 1 "PWR_FLAG" H 2900 2748 50  0000 C CNN
+F 2 "" H 2900 2575 50  0001 C CNN
+F 3 "~" H 2900 2575 50  0001 C CNN
+	1    2900 2575
+	-1   0    0    1
+$EndComp
+$Comp
+L power:GND #PWR?
+U 1 1 61F63FE8
+P 2450 2575
+AR Path="/61C38667/61F63FE8" Ref="#PWR?"  Part="1"
+AR Path="/61F63FE8" Ref="#PWR?"  Part="1"
+AR Path="/622DADD3/61F63FE8" Ref="#PWR02"  Part="1"
+AR Path="/62646A72/61F63FE8" Ref="#PWR?"  Part="1"
+AR Path="/62807237/61F63FE8" Ref="#PWR?"  Part="1"
+AR Path="/62807263/61F63FE8" Ref="#PWR?"  Part="1"
+AR Path="/6284E2B1/61F63FE8" Ref="#PWR?"  Part="1"
+AR Path="/6284E2DD/61F63FE8" Ref="#PWR?"  Part="1"
+AR Path="/6284E31C/61F63FE8" Ref="#PWR?"  Part="1"
+AR Path="/6284E336/61F63FE8" Ref="#PWR?"  Part="1"
+F 0 "#PWR02" H 2450 2325 50  0001 C CNN
+F 1 "GND" H 2450 2425 50  0000 C CNN
+F 2 "" H 2450 2575 50  0001 C CNN
+F 3 "" H 2450 2575 50  0001 C CNN
+	1    2450 2575
+	-1   0    0    1
+$EndComp
+$Comp
+L power:PWR_FLAG #FLG02
+U 1 1 61F64527
+P 2450 2575
+F 0 "#FLG02" H 2450 2650 50  0001 C CNN
+F 1 "PWR_FLAG" H 2450 2748 50  0000 C CNN
+F 2 "" H 2450 2575 50  0001 C CNN
+F 3 "~" H 2450 2575 50  0001 C CNN
+	1    2450 2575
+	-1   0    0    1
+$EndComp
 $EndSCHEMATC

Commit message: fixed shematic
Changed lines of the file:
@@
-$EndSheet
-$Sheet
-S 1825 3525 700  525
-U 62542119
-F0 "sheet625420FC" 50
-F1 "input_ina.sch" 50
-F2 "+VIN_A_INA" I R 2525 3575 50
-F3 "REF_A_INA" I R 2525 3650 50
-F4 "-VIN_A_INA" I R 2525 3725 50
-F5 "+VIN_B_INA" I R 2525 3850 50
-F6 "REF_B_INA" I R 2525 3925 50
-F7 "-VIN_B_INA" I R 2525 4000 50
 $EndSheet
 $Sheet
@@
 F4 "REF_A_INA" I L 3325 3650 50
 F5 "REF_B_INA" I L 3325 3925 50
-F6 "-VIN_A_INA" I L 3325 3575 50
-F7 "+VIN_A_INA" I L 3325 3725 50
+F6 "-VIN_A_INA" I L 3325 3725 50
+F7 "+VIN_A_INA" I L 3325 3575 50
 F8 "+VIN_B_INA" I L 3325 3850 50
 F9 "-VIN_B_INA" I L 3325 4000 50
@@
 Wire Wire Line
 	6500 3950 6925 3950
-Text HLabel 2875 3525 1    50   Input ~ 0
-VIN_A
-Text HLabel 2875 4050 3    50   Input ~ 0
-VIN_B
 Text HLabel 2975 3525 1    50   Input ~ 0
 REF_A
@@
 F3 "RECT_AMP" I R 5600 3575 50
 $EndSheet
+Text HLabel 2875 4050 3    50   Input ~ 0
+-VIN_B
+Text HLabel 2875 3525 1    50   Input ~ 0
++VIN_A
+$Sheet
+S 1825 3525 700  525
+U 62542119
+F0 "sheet625420FC" 50
+F1 "input_ina.sch" 50
+F2 "+VIN_A_INA" I R 2525 3575 50
+F3 "REF_A_INA" I R 2525 3650 50
+F4 "-VIN_A_INA" I R 2525 3725 50
+F5 "+VIN_B_INA" I R 2525 3850 50
+F6 "REF_B_INA" I R 2525 3925 50
+F7 "-VIN_B_INA" I R 2525 4000 50
+$EndSheet
 $EndSCHEMATC
