File: hardware/kicad/emg-filter/emg_module.sch (KiCad schematic (older format))
At the start: 0 parts

Commit message: update
Changed lines of the file:
@@
 F4 "REF_A_INA" I L 3325 3650 50
 F5 "REF_B_INA" I L 3325 3925 50
-F6 "-VIN_A_INA" I L 3325 3575 50
-F7 "+VIN_A_INA" I L 3325 3725 50
+F6 "-VIN_A_INA" I L 3325 3725 50
+F7 "+VIN_A_INA" I L 3325 3575 50
 F8 "+VIN_B_INA" I L 3325 3850 50
 F9 "-VIN_B_INA" I L 3325 4000 50
@@
 AR Path="/61C38667/62542157" Ref="#PWR?"  Part="1"
 AR Path="/62542157" Ref="#PWR?"  Part="1"
-AR Path="/622DADD3/62542157" Ref="#PWR0159"  Part="1"
-AR Path="/62646A72/62542157" Ref="#PWR0190"  Part="1"
-AR Path="/62807237/62542157" Ref="#PWR0221"  Part="1"
-AR Path="/62807263/62542157" Ref="#PWR0252"  Part="1"
-AR Path="/6284E2B1/62542157" Ref="#PWR0283"  Part="1"
-AR Path="/6284E2DD/62542157" Ref="#PWR0314"  Part="1"
-AR Path="/6284E31C/62542157" Ref="#PWR0345"  Part="1"
-AR Path="/6284E336/62542157" Ref="#PWR0376"  Part="1"
-F 0 "#PWR0159" H 6675 3925 50  0001 C CNN
+AR Path="/622DADD3/62542157" Ref="#PWR036"  Part="1"
+AR Path="/62646A72/62542157" Ref="#PWR?"  Part="1"
+AR Path="/62807237/62542157" Ref="#PWR?"  Part="1"
+AR Path="/62807263/62542157" Ref="#PWR?"  Part="1"
+AR Path="/6284E2B1/62542157" Ref="#PWR?"  Part="1"
+AR Path="/6284E2DD/62542157" Ref="#PWR?"  Part="1"
+AR Path="/6284E31C/62542157" Ref="#PWR?"  Part="1"
+AR Path="/6284E336/62542157" Ref="#PWR?"  Part="1"
+AR Path="/6202BCF4/62542157" Ref="#PWR074"  Part="1"
+AR Path="/62039D68/62542157" Ref="#PWR0105"  Part="1"
+AR Path="/62039D86/62542157" Ref="#PWR0136"  Part="1"
+AR Path="/6204723A/62542157" Ref="#PWR0167"  Part="1"
+AR Path="/62047258/62542157" Ref="#PWR0198"  Part="1"
+AR Path="/62051D84/62542157" Ref="#PWR0229"  Part="1"
+AR Path="/62051DA2/62542157" Ref="#PWR0260"  Part="1"
+F 0 "#PWR0260" H 6675 3925 50  0001 C CNN
 F 1 "GND" H 6675 4025 50  0000 C CNN
 F 2 "" H 6675 4175 50  0001 C CNN
@@
 AR Path="/61C38667/6254215D" Ref="#PWR?"  Part="1"
 AR Path="/6254215D" Ref="#PWR?"  Part="1"
-AR Path="/622DADD3/6254215D" Ref="#PWR0160"  Part="1"
-AR Path="/62646A72/6254215D" Ref="#PWR0191"  Part="1"
-AR Path="/62807237/6254215D" Ref="#PWR0222"  Part="1"
-AR Path="/62807263/6254215D" Ref="#PWR0253"  Part="1"
-AR Path="/6284E2B1/6254215D" Ref="#PWR0284"  Part="1"
-AR Path="/6284E2DD/6254215D" Ref="#PWR0315"  Part="1"
-AR Path="/6284E31C/6254215D" Ref="#PWR0346"  Part="1"
-AR Path="/6284E336/6254215D" Ref="#PWR0377"  Part="1"
-F 0 "#PWR0160" H 6500 4025 50  0001 C CNN
+AR Path="/622DADD3/6254215D" Ref="#PWR035"  Part="1"
+AR Path="/62646A72/6254215D" Ref="#PWR?"  Part="1"
+AR Path="/62807237/6254215D" Ref="#PWR?"  Part="1"
+AR Path="/62807263/6254215D" Ref="#PWR?"  Part="1"
+AR Path="/6284E2B1/6254215D" Ref="#PWR?"  Part="1"
+AR Path="/6284E2DD/6254215D" Ref="#PWR?"  Part="1"
+AR Path="/6284E31C/6254215D" Ref="#PWR?"  Part="1"
+AR Path="/6284E336/6254215D" Ref="#PWR?"  Part="1"
+AR Path="/6202BCF4/6254215D" Ref="#PWR073"  Part="1"
+AR Path="/62039D68/6254215D" Ref="#PWR0104"  Part="1"
+AR Path="/62039D86/6254215D" Ref="#PWR0135"  Part="1"
+AR Path="/6204723A/6254215D" Ref="#PWR0166"  Part="1"
+AR Path="/62047258/6254215D" Ref="#PWR0197"  Part="1"
+AR Path="/62051D84/6254215D" Ref="#PWR0228"  Part="1"
+AR Path="/62051DA2/6254215D" Ref="#PWR0259"  Part="1"
+F 0 "#PWR0259" H 6500 4025 50  0001 C CNN
 F 1 "+5V" H 6525 4325 50  0000 C CNN
 F 2 "" H 6500 4175 50  0001 C CNN
@@
 AR Path="/61C38667/62542163" Ref="#PWR?"  Part="1"
 AR Path="/62542163" Ref="#PWR?"  Part="1"
-AR Path="/622DADD3/62542163" Ref="#PWR0161"  Part="1"
-AR Path="/62646A72/62542163" Ref="#PWR0192"  Part="1"
-AR Path="/62807237/62542163" Ref="#PWR0223"  Part="1"
-AR Path="/62807263/62542163" Ref="#PWR0254"  Part="1"
-AR Path="/6284E2B1/62542163" Ref="#PWR0285"  Part="1"
-AR Path="/6284E2DD/62542163" Ref="#PWR0316"  Part="1"
-AR Path="/6284E31C/62542163" Ref="#PWR0347"  Part="1"
-AR Path="/6284E336/62542163" Ref="#PWR0378"  Part="1"
-F 0 "#PWR0161" H 6850 4275 50  0001 C CNN
+AR Path="/622DADD3/62542163" Ref="#PWR037"  Part="1"
+AR Path="/62646A72/62542163" Ref="#PWR?"  Part="1"
+AR Path="/62807237/62542163" Ref="#PWR?"  Part="1"
+AR Path="/62807263/62542163" Ref="#PWR?"  Part="1"
+AR Path="/6284E2B1/62542163" Ref="#PWR?"  Part="1"
+AR Path="/6284E2DD/62542163" Ref="#PWR?"  Part="1"
+AR Path="/6284E31C/62542163" Ref="#PWR?"  Part="1"
+AR Path="/6284E336/62542163" Ref="#PWR?"  Part="1"
+AR Path="/6202BCF4/62542163" Ref="#PWR075"  Part="1"
+AR Path="/62039D68/62542163" Ref="#PWR0106"  Part="1"
+AR Path="/62039D86/62542163" Ref="#PWR0137"  Part="1"
+AR Path="/6204723A/62542163" Ref="#PWR0168"  Part="1"
+AR Path="/62047258/62542163" Ref="#PWR0199"  Part="1"
+AR Path="/62051D84/62542163" Ref="#PWR0230"  Part="1"
+AR Path="/62051DA2/62542163" Ref="#PWR0261"  Part="1"
+F 0 "#PWR0261" H 6850 4275 50  0001 C CNN
 F 1 "-5V" H 6850 4325 50  0000 C CNN
 F 2 "" H 6850 4175 50  0001 C CNN
